Commit message: remove converted urdf file (do not commit such files), fix EL_FLEX limits

File: urdf/dynaarm_parameters.urdf.xacro (robot description, xacro)
@@ -41,6 +41,6 @@
 	<xacro:property name="joint_3_origin_xyz" value="0.412 0 0" />
 	<xacro:property name="joint_3_origin_rpy" value="${J_PI} ${J_PI} 0" />
-	<xacro:property name="joint_3_lower_limit" value="0" />
-	<xacro:property name="joint_3_upper_limit" value="-${J_PI}" />
+	<xacro:property name="joint_3_lower_limit" value="-${J_PI}" />
+	<xacro:property name="joint_3_upper_limit" value="0.0" />
 	<xacro:property name="joint_4_name" value="FA_ROT" />
 	<xacro:property name="joint_4_type" value="revolute" />

Commit message: fixed the values to represent the real robot.

File: urdf/dynaarm_parameters.urdf.xacro (robot description, xacro)
@@ -33,7 +33,10 @@
 	<xacro:property name="joint_2_axis_xyz" value="0 0 -1" />
 	<xacro:property name="joint_2_origin_xyz" value="0 0 0.0" />
-	<xacro:property name="joint_2_origin_rpy" value="${J_PI/2} -${J_PI/2} 0" />
-	<xacro:property name="joint_2_lower_limit" value="${-J_PI/2 - 0.3}" />
-	<xacro:property name="joint_2_upper_limit" value="${J_PI/2 + 0.3}" />
+	<xacro:property name="joint_2_origin_rpy" value="${J_PI/2} 0 0" />
+	<!-- <xacro:property name="joint_2_origin_rpy" value="${J_PI/2} -${J_PI/2} 0" /> -->
+	<xacro:property name="joint_2_lower_limit" value="${-J_PI - 0.3}" />
+	<xacro:property name="joint_2_upper_limit" value="0.3" />
+	<!-- <xacro:property name="joint_2_lower_limit" value="${-J_PI/2 - 0.3}" />
+	<xacro:property name="joint_2_upper_limit" value="${J_PI/2 + 0.3}" /> -->
 	<xacro:property name="joint_3_name" value="EL_FLE" />
 	<xacro:property name="joint_3_type" value="revolute" />

Commit message: BUG: With Gazebo and moveit Need to set the upper limit a bit higher otherwise planning can't start.

File: urdf/dynaarm_parameters.urdf.xacro (robot description, xacro)
@@ -45,5 +45,5 @@
 	<xacro:property name="joint_3_origin_rpy" value="${J_PI} ${J_PI} 0" />
 	<xacro:property name="joint_3_lower_limit" value="-${J_PI}" />
-	<xacro:property name="joint_3_upper_limit" value="0.0" />
+	<xacro:property name="joint_3_upper_limit" value="0.05" />
 	<xacro:property name="joint_4_name" value="FA_ROT" />
 	<xacro:property name="joint_4_type" value="revolute" />
