Commit message: allow to configure drive config file path

File: urdf/dynaarm.ros2_control.xacro (robot description, xacro)
@@ -4,4 +4,5 @@
     <xacro:property name="initial_positions_filename" value="$(find duatic_ros2_description)/config/initial_positions.yaml"/>
     <xacro:property name="initial_positions" value="${xacro.load_yaml(initial_positions_filename)['initial_positions']}"/>
+    <xacro:property name="drive_config_file" value="$(find dynaarm_driver)/config/dynadrive.yaml"/>
     <ros2_control name="${name}" type="system">
       <xacro:if value="$(arg use_sim)">
@@ -16,4 +17,5 @@
           <param name="ethercat_bus">${ethercat_bus}</param>
           <param name="prefix">duatic</param>
+          <param name="drive_config_file">${drive_config_file}</param>
         </hardware>
       </xacro:unless>

Commit message: wire in mocked hardware mode

File: urdf/dynaarm.ros2_control.xacro (robot description, xacro)
@@ -1,5 +1,5 @@
 <?xml version="1.0"?>
 <robot xmlns:xacro="http://www.ros.org/wiki/xacro">
-  <xacro:macro name="dynaarm_ros2_control" params="name prefix use_sim ethercat_bus">
+  <xacro:macro name="dynaarm_ros2_control" params="name prefix use_sim use_gazebo ethercat_bus">
     <xacro:property name="initial_positions_filename" value="$(find duatic_ros2_description)/config/initial_positions.yaml"/>
     <xacro:property name="initial_positions" value="${xacro.load_yaml(initial_positions_filename)['initial_positions']}"/>
@@ -8,6 +8,10 @@
       <xacro:if value="$(arg use_sim)">
         <hardware>
-          <!-- <plugin>mock_components/GenericSystem</plugin> -->
-          <plugin>gz_ros2_control/GazeboSimSystem</plugin>
+            <xacro:unless value="$(arg use_gazebo)">
+              <plugin>mock_components/GenericSystem</plugin>
+            </xacro:unless>
+             <xacro:if value="$(arg use_gazebo)">
+              <plugin>gz_ros2_control/GazeboSimSystem</plugin>
+            </xacro:if>
         </hardware>
       </xacro:if>

File: urdf/dynaarm.xacro (robot description, xacro)
@@ -3,4 +3,5 @@
   <xacro:arg name="prefix" default="" />
   <xacro:arg name="use_sim" default="true" />
+  <xacro:arg name="use_gazebo" default="false" />
   <xacro:arg name="ethercat_bus" default="enp86s0" />
   <xacro:include filename="$(find duatic_ros2_description)/urdf/dynaarm.urdf.xacro" />
@@ -18,4 +19,5 @@
                               ethercat_bus="$(arg ethercat_bus)"
                               prefix="$(arg prefix)"
-                              use_sim="$(arg use_sim)" />
+                              use_sim="$(arg use_sim)"
+                              use_gazebo="$(arg use_gazebo)" />
 </robot>

Commit message: renamed duatic_ros2_description -> duatic_description

File: urdf/dynaarm.ros2_control.xacro (robot description, xacro)
@@ -2,5 +2,5 @@
 <robot xmlns:xacro="http://www.ros.org/wiki/xacro">
   <xacro:macro name="dynaarm_ros2_control" params="name prefix use_sim use_gazebo ethercat_bus">
-    <xacro:property name="initial_positions_filename" value="$(find duatic_ros2_description)/config/initial_positions.yaml"/>
+    <xacro:property name="initial_positions_filename" value="$(find duatic_description)/config/initial_positions.yaml"/>
     <xacro:property name="initial_positions" value="${xacro.load_yaml(initial_positions_filename)['initial_positions']}"/>
     <xacro:property name="drive_config_file" value="$(find dynaarm_driver)/config/dynadrive.yaml"/>

File: urdf/dynaarm.urdf.xacro (robot description, xacro)
@@ -2,5 +2,5 @@
 <robot xmlns:xacro="http://www.ros.org/wiki/xacro">
 	<xacro:macro name="dynaarm" params="parent prefix *origin">
-		<xacro:include filename="$(find duatic_ros2_description)/urdf/dynaarm_parameters.urdf.xacro"/>
+		<xacro:include filename="$(find duatic_description)/urdf/dynaarm_parameters.urdf.xacro"/>
 		<!-- World - Base -->
 		<joint name="${prefix}${joint_base_name}" type="${joint_base_type}">
@@ -17,5 +17,5 @@
 			<visual>
 				<geometry>
-					<mesh filename="file://$(find duatic_ros2_description)/meshes/100_base_mesh.dae" />
+					<mesh filename="file://$(find duatic_description)/meshes/100_base_mesh.dae" />
 				</geometry>
 				<material name="carbon_fiber">
@@ -25,5 +25,5 @@
 			<collision>
 				<geometry>
-					<mesh filename="file://$(find duatic_ros2_description)/meshes/100_base_mesh_col.dae" />
+					<mesh filename="file://$(find duatic_description)/meshes/100_base_mesh_col.dae" />
 				</geometry>
 			</collision>
@@ -38,5 +38,5 @@
 			<visual>
 				<geometry>
-					<mesh filename="file://$(find duatic_ros2_description)/meshes/101_shoulder_mesh.dae"/>
+					<mesh filename="file://$(find duatic_description)/meshes/101_shoulder_mesh.dae"/>
 				</geometry>
 				<material name="carbon_fiber">
@@ -46,5 +46,5 @@
 			<collision>
 				<geometry>
-					<mesh filename="file://$(find duatic_ros2_description)/meshes/101_shoulder_mesh_col.dae"/>
+					<mesh filename="file://$(find duatic_description)/meshes/101_shoulder_mesh_col.dae"/>
 				</geometry>
 			</collision>
@@ -59,5 +59,5 @@
 			<visual>
 				<geometry>
-					<mesh filename="file://$(find duatic_ros2_description)/meshes/102_upperarm_mesh.dae"/>
+					<mesh filename="file://$(find duatic_description)/meshes/102_upperarm_mesh.dae"/>
 				</geometry>
 				<material name="carbon_fiber">
@@ -67,5 +67,5 @@
 			<collision>
 				<geometry>
-					<mesh filename="file://$(find duatic_ros2_description)/meshes/102_upperarm_mesh_col.dae"/>
+					<mesh filename="file://$(find duatic_description)/meshes/102_upperarm_mesh_col.dae"/>
 				</geometry>
 			</collision>
@@ -80,5 +80,5 @@
 			<visual>
 				<geometry>
-					<mesh filename="file://$(find duatic_ros2_description)/meshes/103_elbow_mesh.dae"/>
+					<mesh filename="file://$(find duatic_description)/meshes/103_elbow_mesh.dae"/>
 				</geometry>
 				<material name="carbon_fiber">
@@ -88,5 +88,5 @@
 			<collision>
 				<geometry>
-					<mesh filename="file://$(find duatic_ros2_description)/meshes/103_elbow_mesh_col.dae"/>
+					<mesh filename="file://$(find duatic_description)/meshes/103_elbow_mesh_col.dae"/>
 				</geometry>
 			</collision>

File: urdf/dynaarm.xacro (robot description, xacro)
@@ -5,6 +5,6 @@
   <xacro:arg name="use_gazebo" default="false" />
   <xacro:arg name="ethercat_bus" default="enp86s0" />
-  <xacro:include filename="$(find duatic_ros2_description)/urdf/dynaarm.urdf.xacro" />
-  <xacro:include filename="$(find duatic_ros2_description)/urdf/dynaarm.ros2_control.xacro" />
+  <xacro:include filename="$(find duatic_description)/urdf/dynaarm.urdf.xacro" />
+  <xacro:include filename="$(find duatic_description)/urdf/dynaarm.ros2_control.xacro" />
   <!-- create world link and link it to the dynaarm base -->
   <link name="world"/>

Commit message: Modified the ros2_control limits.

File: urdf/dynaarm.ros2_control.xacro (robot description, xacro)
@@ -5,4 +5,5 @@
     <xacro:property name="initial_positions" value="${xacro.load_yaml(initial_positions_filename)['initial_positions']}"/>
     <xacro:property name="drive_config_file" value="$(find dynaarm_driver)/config/dynadrive.yaml"/>
+    <xacro:property name="J_PI" value="3.1415926535897931" />
     <ros2_control name="${name}" type="system">
       <xacro:if value="$(arg use_sim)">
@@ -27,6 +28,6 @@
         <param name="address">1</param>
         <command_interface name="position">
-          <param name="min">{-2*pi}</param>
-          <param name="max">{2*pi}</param>
+          <param name="min">"${-J_PI - J_PI/2}"</param>
+          <param name="max">"${J_PI + J_PI/2}"</param>
         </command_interface>
         <command_interface name="velocity">
@@ -51,6 +52,6 @@
         <param name="address">3</param>
         <command_interface name="position">
-          <param name="min">{-2*pi}</param>
-          <param name="max">{2*pi}</param>
+          <param name="min">"${-J_PI/2 - 0.3}"</param>
+          <param name="max">"${J_PI/2 + 0.3}"</param>
         </command_interface>
         <command_interface name="velocity">
@@ -75,6 +76,6 @@
         <param name="address">2</param>
         <command_interface name="position">
-          <param name="min">{-2*pi}</param>
-          <param name="max">{2*pi}</param>
+          <param name="min">"-${J_PI}"</param>
+          <param name="max">0.0</param>
         </command_interface>
         <command_interface name="velocity">
@@ -99,6 +100,6 @@
         <param name="address">4</param>
         <command_interface name="position">
-          <param name="min">{-2*pi}</param>
-          <param name="max">{2*pi}</param>
+          <param name="min">"${-J_PI - J_PI/2}"</param>
+          <param name="max">"${J_PI + J_PI/2}"</param>
         </command_interface>
         <command_interface name="velocity">

File: urdf/dynaarm.xacro (robot description, xacro)
@@ -2,5 +2,5 @@
   xmlns:xacro="http://www.ros.org/wiki/xacro">
   <xacro:arg name="prefix" default="" />
-  <xacro:arg name="use_sim" default="true" />
+  <xacro:arg name="use_sim" default="false" />
   <xacro:arg name="use_gazebo" default="false" />
   <xacro:arg name="ethercat_bus" default="enp86s0" />

File: urdf/dynaarm_parameters.urdf.xacro (robot description, xacro)
@@ -16,5 +16,5 @@
 	<xacro:property name="link01_mesh" value="shoulder_mesh" />
 	<xacro:property name="link02_mesh" value="upperarm_mesh" />
-  <xacro:property name="link03_mesh" value="elbow_mesh" />
+    <xacro:property name="link03_mesh" value="elbow_mesh" />
 	<xacro:property name="joint_base_name"	value="joint_base" />
 	<xacro:property name="joint_base_type" value="fixed" />

Commit message: refactored use_sim to use_fake

File: urdf/dynaarm.ros2_control.xacro (robot description, xacro)
@@ -1,5 +1,5 @@
 <?xml version="1.0"?>
 <robot xmlns:xacro="http://www.ros.org/wiki/xacro">
-  <xacro:macro name="dynaarm_ros2_control" params="name prefix use_sim use_gazebo ethercat_bus">
+  <xacro:macro name="dynaarm_ros2_control" params="name prefix use_fake use_gazebo ethercat_bus">
     <xacro:property name="initial_positions_filename" value="$(find duatic_description)/config/initial_positions.yaml"/>
     <xacro:property name="initial_positions" value="${xacro.load_yaml(initial_positions_filename)['initial_positions']}"/>
@@ -7,5 +7,5 @@
     <xacro:property name="J_PI" value="3.1415926535897931" />
     <ros2_control name="${name}" type="system">
-      <xacro:if value="$(arg use_sim)">
+      <xacro:if value="$(arg use_fake)">
         <hardware>
             <xacro:unless value="$(arg use_gazebo)">
@@ -17,5 +17,5 @@
         </hardware>
       </xacro:if>
-      <xacro:unless value="$(arg use_sim)">
+      <xacro:unless value="$(arg use_fake)">
         <hardware>
           <plugin>dynaarm_driver/DynaArmHardwareInterface</plugin>
@@ -122,5 +122,5 @@
       </joint>
     </ros2_control>
-    <xacro:if value="$(arg use_sim)">
+    <xacro:if value="$(arg use_fake)">
       <gazebo>
         <plugin filename="libgz_ros2_control-system.so" name="gz_ros2_control::GazeboSimROS2ControlPlugin">

File: urdf/dynaarm.xacro (robot description, xacro)
@@ -2,5 +2,5 @@
   xmlns:xacro="http://www.ros.org/wiki/xacro">
   <xacro:arg name="prefix" default="" />
-  <xacro:arg name="use_sim" default="false" />
+  <xacro:arg name="use_fake" default="true" />
   <xacro:arg name="use_gazebo" default="false" />
   <xacro:arg name="ethercat_bus" default="enp86s0" />
@@ -19,5 +19,5 @@
                               ethercat_bus="$(arg ethercat_bus)"
                               prefix="$(arg prefix)"
-                              use_sim="$(arg use_sim)"
+                              use_fake="$(arg use_fake)"
                               use_gazebo="$(arg use_gazebo)" />
 </robot>

Commit message: refactored duatic_description -> dynaarm_description

File: urdf/dynaarm.ros2_control.xacro (robot description, xacro)
@@ -2,5 +2,5 @@
 <robot xmlns:xacro="http://www.ros.org/wiki/xacro">
   <xacro:macro name="dynaarm_ros2_control" params="name prefix use_fake use_gazebo ethercat_bus">
-    <xacro:property name="initial_positions_filename" value="$(find duatic_description)/config/initial_positions.yaml"/>
+    <xacro:property name="initial_positions_filename" value="$(find dynaarm_description)/config/initial_positions.yaml"/>
     <xacro:property name="initial_positions" value="${xacro.load_yaml(initial_positions_filename)['initial_positions']}"/>
     <xacro:property name="drive_config_file" value="$(find dynaarm_driver)/config/dynadrive.yaml"/>

File: urdf/dynaarm.urdf.xacro (robot description, xacro)
@@ -2,5 +2,5 @@
 <robot xmlns:xacro="http://www.ros.org/wiki/xacro">
 	<xacro:macro name="dynaarm" params="parent prefix *origin">
-		<xacro:include filename="$(find duatic_description)/urdf/dynaarm_parameters.urdf.xacro"/>
+		<xacro:include filename="$(find dynaarm_description)/urdf/dynaarm_parameters.urdf.xacro"/>
 		<!-- World - Base -->
 		<joint name="${prefix}${joint_base_name}" type="${joint_base_type}">
@@ -17,5 +17,5 @@
 			<visual>
 				<geometry>
-					<mesh filename="file://$(find duatic_description)/meshes/100_base_mesh.dae" />
+					<mesh filename="file://$(find dynaarm_description)/meshes/100_base_mesh.dae" />
 				</geometry>
 				<material name="carbon_fiber">
@@ -25,5 +25,5 @@
 			<collision>
 				<geometry>
-					<mesh filename="file://$(find duatic_description)/meshes/100_base_mesh_col.dae" />
+					<mesh filename="file://$(find dynaarm_description)/meshes/100_base_mesh_col.dae" />
 				</geometry>
 			</collision>
@@ -38,5 +38,5 @@
 			<visual>
 				<geometry>
-					<mesh filename="file://$(find duatic_description)/meshes/101_shoulder_mesh.dae"/>
+					<mesh filename="file://$(find dynaarm_description)/meshes/101_shoulder_mesh.dae"/>
 				</geometry>
 				<material name="carbon_fiber">
@@ -46,5 +46,5 @@
 			<collision>
 				<geometry>
-					<mesh filename="file://$(find duatic_description)/meshes/101_shoulder_mesh_col.dae"/>
+					<mesh filename="file://$(find dynaarm_description)/meshes/101_shoulder_mesh_col.dae"/>
 				</geometry>
 			</collision>
@@ -59,5 +59,5 @@
 			<visual>
 				<geometry>
-					<mesh filename="file://$(find duatic_description)/meshes/102_upperarm_mesh.dae"/>
+					<mesh filename="file://$(find dynaarm_description)/meshes/102_upperarm_mesh.dae"/>
 				</geometry>
 				<material name="carbon_fiber">
@@ -67,5 +67,5 @@
 			<collision>
 				<geometry>
-					<mesh filename="file://$(find duatic_description)/meshes/102_upperarm_mesh_col.dae"/>
+					<mesh filename="file://$(find dynaarm_description)/meshes/102_upperarm_mesh_col.dae"/>
 				</geometry>
 			</collision>
@@ -80,5 +80,5 @@
 			<visual>
 				<geometry>
-					<mesh filename="file://$(find duatic_description)/meshes/103_elbow_mesh.dae"/>
+					<mesh filename="file://$(find dynaarm_description)/meshes/103_elbow_mesh.dae"/>
 				</geometry>
 				<material name="carbon_fiber">
@@ -88,5 +88,5 @@
 			<collision>
 				<geometry>
-					<mesh filename="file://$(find duatic_description)/meshes/103_elbow_mesh_col.dae"/>
+					<mesh filename="file://$(find dynaarm_description)/meshes/103_elbow_mesh_col.dae"/>
 				</geometry>
 			</collision>

File: urdf/dynaarm.xacro (robot description, xacro)
@@ -5,6 +5,6 @@
   <xacro:arg name="use_gazebo" default="false" />
   <xacro:arg name="ethercat_bus" default="enp86s0" />
-  <xacro:include filename="$(find duatic_description)/urdf/dynaarm.urdf.xacro" />
-  <xacro:include filename="$(find duatic_description)/urdf/dynaarm.ros2_control.xacro" />
+  <xacro:include filename="$(find dynaarm_description)/urdf/dynaarm.urdf.xacro" />
+  <xacro:include filename="$(find dynaarm_description)/urdf/dynaarm.ros2_control.xacro" />
   <!-- create world link and link it to the dynaarm base -->
   <link name="world"/>

Commit message: Removed the dependency to the dynaarm_driver package. Added a drive_config_file_path argument to forward the dynadrive config file.

File: urdf/dynaarm.ros2_control.xacro (robot description, xacro)
@@ -1,8 +1,7 @@
 <?xml version="1.0"?>
 <robot xmlns:xacro="http://www.ros.org/wiki/xacro">
-  <xacro:macro name="dynaarm_ros2_control" params="name prefix use_fake use_gazebo ethercat_bus">
+  <xacro:macro name="dynaarm_ros2_control" params="name prefix use_fake use_gazebo ethercat_bus drive_config_file_path">
     <xacro:property name="initial_positions_filename" value="$(find dynaarm_description)/config/initial_positions.yaml"/>
     <xacro:property name="initial_positions" value="${xacro.load_yaml(initial_positions_filename)['initial_positions']}"/>
-    <xacro:property name="drive_config_file" value="$(find dynaarm_driver)/config/dynadrive.yaml"/>
     <xacro:property name="J_PI" value="3.1415926535897931" />
     <ros2_control name="${name}" type="system">
@@ -22,5 +21,5 @@
           <param name="ethercat_bus">${ethercat_bus}</param>
           <param name="prefix">duatic</param>
-          <param name="drive_config_file">${drive_config_file}</param>
+          <param name="drive_config_file_path">${drive_config_file_path}</param>
         </hardware>
       </xacro:unless>

File: urdf/dynaarm.xacro (robot description, xacro)
@@ -5,4 +5,5 @@
   <xacro:arg name="use_gazebo" default="false" />
   <xacro:arg name="ethercat_bus" default="enp86s0" />
+  <xacro:arg name="drive_config_file_path" default="" />
   <xacro:include filename="$(find dynaarm_description)/urdf/dynaarm.urdf.xacro" />
   <xacro:include filename="$(find dynaarm_description)/urdf/dynaarm.ros2_control.xacro" />
@@ -20,4 +21,5 @@
                               prefix="$(arg prefix)"
                               use_fake="$(arg use_fake)"
-                              use_gazebo="$(arg use_gazebo)" />
+                              use_gazebo="$(arg use_gazebo)"
+                              drive_config_file_path="$(arg drive_config_file_path)"/>
 </robot>
