Commit message: Fixed also the dual xacro for the new dynaarm 0 position.

File: urdf/dynaarm_standalone_dual.urdf.xacro (robot description, xacro)
@@ -33,5 +33,5 @@
                 collision="$(arg collision)"
                 version="$(arg version)">
-    <origin xyz="0 0 0.085" rpy="0.0 0.0 0.0" />
+    <origin xyz="0 0 0" rpy="0.0 0.0 0.0" />
   </xacro:dynaarm>
   <!-- Note: for a real world application you would pass different parameters for both arms (e.g. different ethercat_bus)-->
@@ -44,5 +44,5 @@
                 collision="$(arg collision)"
                 version="$(arg version)">
-    <origin xyz="1.0 0 0.085" rpy="0.0 0.0 0.0" />
+    <origin xyz="1.0 0 0" rpy="0.0 0.0 0.0" />
   </xacro:dynaarm>
 </robot>
