Commit message: Added if query to the urdf creation to add cam stuff only for v2. This needs to be discussed how we work with these camera points for v1 / v2 / ...

File: urdf/dynaarm.urdf.xacro (robot description, xacro)
@@ -2,9 +2,22 @@
 <!--
 Copyright 2024 Duatic AG
-Redistribution and use in source and binary forms, with or without modification, are permitted provided that the following conditions are met:
-1. Redistributions of source code must retain the above copyright notice, this list of conditions and the following disclaimer.
-2. Redistributions in binary form must reproduce the above copyright notice, this list of conditions and the following disclaimer in the documentation and/or other materials provided with the distribution.
-3. Neither the name of the copyright holder nor the names of its contributors may be used to endorse or promote products derived from this software without specific prior written permission.
-THIS SOFTWARE IS PROVIDED BY THE COPYRIGHT HOLDERS AND CONTRIBUTORS “AS IS” AND ANY EXPRESS OR IMPLIED WARRANTIES, INCLUDING, BUT NOT LIMITED TO, THE IMPLIED WARRANTIES OF MERCHANTABILITY AND FITNESS FOR A PARTICULAR PURPOSE ARE DISCLAIMED. IN NO EVENT SHALL THE COPYRIGHT HOLDER OR CONTRIBUTORS BE LIABLE FOR ANY DIRECT, INDIRECT, INCIDENTAL, SPECIAL, EXEMPLARY, OR CONSEQUENTIAL DAMAGES (INCLUDING, BUT NOT LIMITED TO, PROCUREMENT OF SUBSTITUTE GOODS OR SERVICES; LOSS OF USE, DATA, OR PROFITS; OR BUSINESS INTERRUPTION) HOWEVER CAUSED AND ON ANY THEORY OF LIABILITY, WHETHER IN CONTRACT, STRICT LIABILITY, OR TORT (INCLUDING NEGLIGENCE OR OTHERWISE) ARISING IN ANY WAY OUT OF THE USE OF THIS SOFTWARE, EVEN IF ADVISED OF THE POSSIBILITY OF SUCH DAMAGE.
+Redistribution and use in source and binary forms, with or without modification, are permitted
+provided that the following conditions are met:
+1. Redistributions of source code must retain the above copyright notice, this list of conditions
+and the following disclaimer.
+2. Redistributions in binary form must reproduce the above copyright notice, this list of
+conditions and the following disclaimer in the documentation and/or other materials provided with
+the distribution.
+3. Neither the name of the copyright holder nor the names of its contributors may be used to
+endorse or promote products derived from this software without specific prior written permission.
+THIS SOFTWARE IS PROVIDED BY THE COPYRIGHT HOLDERS AND CONTRIBUTORS “AS IS” AND ANY EXPRESS OR
+IMPLIED WARRANTIES, INCLUDING, BUT NOT LIMITED TO, THE IMPLIED WARRANTIES OF MERCHANTABILITY AND
+FITNESS FOR A PARTICULAR PURPOSE ARE DISCLAIMED. IN NO EVENT SHALL THE COPYRIGHT HOLDER OR
+CONTRIBUTORS BE LIABLE FOR ANY DIRECT, INDIRECT, INCIDENTAL, SPECIAL, EXEMPLARY, OR CONSEQUENTIAL
+DAMAGES (INCLUDING, BUT NOT LIMITED TO, PROCUREMENT OF SUBSTITUTE GOODS OR SERVICES; LOSS OF USE,
+DATA, OR PROFITS; OR BUSINESS INTERRUPTION) HOWEVER CAUSED AND ON ANY THEORY OF LIABILITY, WHETHER
+IN CONTRACT, STRICT LIABILITY, OR TORT (INCLUDING NEGLIGENCE OR OTHERWISE) ARISING IN ANY WAY OUT
+OF
+THE USE OF THIS SOFTWARE, EVEN IF ADVISED OF THE POSSIBILITY OF SUCH DAMAGE.
 -->
 <robot name="dynaarm" xmlns:xacro="http://www.ros.org/wiki/xacro">
@@ -157,23 +170,25 @@
       </xacro:dynaarm_revolute_joint>
       <!--dynaarm_ELBOW_CAMERA_BASE-->
-      <link name="${link03_cam}">
-        <visual>
-          <origin rpy="0 0 0" xyz="0 0 0" />
-          <geometry>
-            <box size="0.001 0.001 0.001" />
-          </geometry>
-        </visual>
-        <inertial>
-          <origin rpy="0 0 0" xyz="0.0 0.0 0.0" />
-          <mass value="0.001" />
-          <inertia ixx="0.0000001" ixy="0.0" ixz="0.0" iyy="0.0000001" iyz="0.0" izz="0.0000001" />
-        </inertial>
-      </link>
-      <!-- Camera fixed on elbow -->
-      <xacro:dynaarm_joint_fixed joint_name="${joint_3_cam_name}"
-        parent="${link03}"
-        child="${link03_cam}">
-        <origin xyz="${joint_3_cam_origin_xyz}" rpy="${joint_3_cam_origin_rpy}" />
-      </xacro:dynaarm_joint_fixed>
+      <xacro:if value="${version == 'v2'}">
+        <link name="${link03_cam}">
+          <visual>
+            <origin rpy="0 0 0" xyz="0 0 0" />
+            <geometry>
+              <box size="0.001 0.001 0.001" />
+            </geometry>
+          </visual>
+          <inertial>
+            <origin rpy="0 0 0" xyz="0.0 0.0 0.0" />
+            <mass value="0.001" />
+            <inertia ixx="0.0000001" ixy="0.0" ixz="0.0" iyy="0.0000001" iyz="0.0" izz="0.0000001" />
+          </inertial>
+        </link>
+        <!-- Camera fixed on elbow -->
+        <xacro:dynaarm_joint_fixed joint_name="${joint_3_cam_name}"
+          parent="${link03}"
+          child="${link03_cam}">
+          <origin xyz="${joint_3_cam_origin_xyz}" rpy="${joint_3_cam_origin_rpy}" />
+        </xacro:dynaarm_joint_fixed>
+      </xacro:if>
       <!-- 3 Dof & Covers-->
       <xacro:if value="${covers}">
@@ -243,24 +258,26 @@
         <origin xyz="${joint_5_origin_xyz}" rpy="${joint_5_origin_rpy}" />
       </xacro:dynaarm_revolute_joint>
-      <!--dynaarm_WRIST_1_CAMERA_BASE-->
-      <link name="${link05_cam}">
-        <visual>
-          <origin rpy="0 0 0" xyz="0 0 0" />
-          <geometry>
-            <box size="0.001 0.001 0.001" />
-          </geometry>
-        </visual>
-        <inertial>
-          <origin rpy="0 0 0" xyz="0.0 0.0 0.0" />
-          <mass value="0.001" />
-          <inertia ixx="0.0000001" ixy="0.0" ixz="0.0" iyy="0.0000001" iyz="0.0" izz="0.0000001" />
-        </inertial>
-      </link>
-      <!-- Camera fixed on wrist1 -->
-      <xacro:dynaarm_joint_fixed joint_name="${joint_5_cam_name}"
-        parent="${link05}"
-        child="${link05_cam}">
-        <origin xyz="${joint_5_cam_origin_xyz}" rpy="${joint_5_cam_origin_rpy}" />
-      </xacro:dynaarm_joint_fixed>
+      <xacro:if value="${version == 'v2'}">
+        <!--dynaarm_WRIST_1_CAMERA_BASE-->
+        <link name="${link05_cam}">
+          <visual>
+            <origin rpy="0 0 0" xyz="0 0 0" />
+            <geometry>
+              <box size="0.001 0.001 0.001" />
+            </geometry>
+          </visual>
+          <inertial>
+            <origin rpy="0 0 0" xyz="0.0 0.0 0.0" />
+            <mass value="0.001" />
+            <inertia ixx="0.0000001" ixy="0.0" ixz="0.0" iyy="0.0000001" iyz="0.0" izz="0.0000001" />
+          </inertial>
+        </link>
+        <!-- Camera fixed on wrist1 -->
+        <xacro:dynaarm_joint_fixed joint_name="${joint_5_cam_name}"
+          parent="${link05}"
+          child="${link05_cam}">
+          <origin xyz="${joint_5_cam_origin_xyz}" rpy="${joint_5_cam_origin_rpy}" />
+        </xacro:dynaarm_joint_fixed>
+      </xacro:if>
       <!-- 5 Dof & Covers-->
       <xacro:if value="${covers}">

Commit message: Using now the macro way to generate the links for cameras.

File: urdf/dynaarm.urdf.xacro (robot description, xacro)
@@ -171,17 +171,6 @@
       <!--dynaarm_ELBOW_CAMERA_BASE-->
       <xacro:if value="${version == 'v2'}">
-        <link name="${link03_cam}">
-          <visual>
-            <origin rpy="0 0 0" xyz="0 0 0" />
-            <geometry>
-              <box size="0.001 0.001 0.001" />
-            </geometry>
-          </visual>
-          <inertial>
-            <origin rpy="0 0 0" xyz="0.0 0.0 0.0" />
-            <mass value="0.001" />
-            <inertia ixx="0.0000001" ixy="0.0" ixz="0.0" iyy="0.0000001" iyz="0.0" izz="0.0000001" />
-          </inertial>
-        </link>
+        <!-- Virtual elbow camera link -->
+        <xacro:virtual_link link_name="${link03_cam}" />
         <!-- Camera fixed on elbow -->
         <xacro:dynaarm_joint_fixed joint_name="${joint_3_cam_name}"
@@ -238,5 +227,5 @@
     <!-- 5 DoF -->
     <xacro:if value="${dof >= 5}">
-      <!-- dynaarm_WRIST_1 -->
+      <!-- WRIST_1 -->
       <xacro:dynaarm_link_w_collision link_name="${link05}" file_name="${link05_mesh}">
         <link_inertia>
@@ -247,5 +236,5 @@
         </link_collision>
       </xacro:dynaarm_link_w_collision>
-      <!-- WRIST_1 -->
+      <!-- WR_FLE -->
       <xacro:dynaarm_revolute_joint joint_name="${joint_5_name}" parent="${link04}"
         child="${link05}"
@@ -259,18 +248,6 @@
       </xacro:dynaarm_revolute_joint>
       <xacro:if value="${version == 'v2'}">
-        <!--dynaarm_WRIST_1_CAMERA_BASE-->
-        <link name="${link05_cam}">
-          <visual>
-            <origin rpy="0 0 0" xyz="0 0 0" />
-            <geometry>
-              <box size="0.001 0.001 0.001" />
-            </geometry>
-          </visual>
-          <inertial>
-            <origin rpy="0 0 0" xyz="0.0 0.0 0.0" />
-            <mass value="0.001" />
-            <inertia ixx="0.0000001" ixy="0.0" ixz="0.0" iyy="0.0000001" iyz="0.0" izz="0.0000001" />
-          </inertial>
-        </link>
+        <!-- Virtual wrist camera link -->
+        <xacro:virtual_link link_name="${link05_cam}" />
         <!-- Camera fixed on wrist1 -->
         <xacro:dynaarm_joint_fixed joint_name="${joint_5_cam_name}"
@@ -295,5 +272,5 @@
     <!-- 6 DoF -->
     <xacro:if value="${dof >= 6}">
-      <!-- dynaarm_WRIST_2 -->
+      <!-- WRIST_2 -->
       <xacro:dynaarm_link link_name="${link06}" file_name="${link06_mesh}">
         <link_inertia>
@@ -301,5 +278,5 @@
         </link_inertia>
       </xacro:dynaarm_link>
-      <!-- WRIST_2 -->
+      <!-- WR_ROT -->
       <xacro:dynaarm_revolute_joint joint_name="${joint_6_name}" parent="${link05}"
         child="${link06}"

Commit message: Added controller path as parameter

File: urdf/dynaarm.urdf.xacro (robot description, xacro)
@@ -26,5 +26,5 @@
   <!-- -->
   <xacro:macro name="dynaarm"
-    params="tf_prefix parent_link dof mode ethercat_bus start_in_freeze_mode:=false drive_parameter_folder:='' covers version *origin">
+    params="tf_prefix parent_link dof mode ethercat_bus controller_path start_in_freeze_mode:=false drive_parameter_folder:='' covers version *origin">
     <!--Allow the user to pass a custom folder for drive parameters-->
     <xacro:property name="default_drive_parameter_folder" value="$(find dynaarm_driver)/config/${version}" />
@@ -52,5 +52,5 @@
     <!-- Gazebo plugin -->
     <xacro:if value="${mode == 'sim'}">
-      <xacro:dynaarm_gazebo />
+      <xacro:dynaarm_gazebo controller_path="${controller_path}"/>
     </xacro:if>
     <!--ros2control-->
@@ -340,9 +340,9 @@
   <!-- DynaArm Gazebo-->
   <!-- -->
-  <xacro:macro name="dynaarm_gazebo">
+  <xacro:macro name="dynaarm_gazebo" params="controller_path">
     <gazebo>
       <plugin filename="libgz_ros2_control-system.so"
         name="gz_ros2_control::GazeboSimROS2ControlPlugin">
-        <parameters>$(find dynaarm_examples)/config/controllers.yaml</parameters>
+        <parameters>${controller_path}</parameters>
       </plugin>
     </gazebo>

Commit message: Removed an commented part as we don't need it there.

File: urdf/dynaarm.urdf.xacro (robot description, xacro)
@@ -336,14 +336,4 @@
           <origin xyz="${joint_ee_origin_xyz}" rpy="${joint_ee_origin_rpy}" />
       </xacro:dynaarm_joint_fixed>
-      <!-- Add x_kg weight to flange -->
-      <!-- <xacro:virtual_link link_name="${end_effector}_weight"
-          mass="0.2"
-          ixx="0.036" iyy="0.036" izz="0.002">
-      </xacro:virtual_link>
-      <xacro:dynaarm_joint_fixed joint_name="${end_effector}_weight_joint"
-          parent="${end_effector}"
-          child="${end_effector}_weight">
-          <origin xyz="0.0 0.0 0.02" rpy="0 0 0" />
-      </xacro:dynaarm_joint_fixed> -->
   </xacro:macro>
   <!-- -->

Commit message: feat: move gz_ros2_control plugin from template urdf to standalone urdfs

File: urdf/dynaarm.urdf.xacro (robot description, xacro)
@@ -26,5 +26,5 @@
   <!-- -->
   <xacro:macro name="dynaarm"
-    params="tf_prefix parent_link collision:='simple' dof mode ethercat_bus drive_order:='' start_in_freeze_mode:=false drive_parameter_folder:='' controller_path:='' covers version *origin">
+    params="tf_prefix parent_link collision:='simple' dof mode ethercat_bus drive_order:='' start_in_freeze_mode:=false drive_parameter_folder:='' covers version *origin">
     <!-- Allow the user to pass the drive order file -->
     <xacro:property name="default_drive_order_file" value="$(find dynaarm_description)/urdf/common/${version}/drive_order.yaml" />
@@ -54,8 +54,4 @@
     <xacro:dynaarm_main_body />
     <xacro:dynaarm_tool />
-    <!-- Gazebo plugin -->
-    <xacro:if value="${mode == 'sim'}">
-      <xacro:dynaarm_gazebo controller_path="${controller_path}"/>
-    </xacro:if>
     <!--ros2control-->
     <xacro:dynaarm_ros2_control tf_prefix="${tf_prefix}"
@@ -346,15 +342,3 @@
       </xacro:dynaarm_joint_fixed>
   </xacro:macro>
-  <!-- -->
-  <!-- DynaArm Gazebo-->
-  <!-- -->
-  <xacro:macro name="dynaarm_gazebo" params="controller_path">
-    <gazebo>
-      <plugin filename="libgz_ros2_control-system.so"
-        name="gz_ros2_control::GazeboSimROS2ControlPlugin">
-        <parameters>${controller_path}</parameters>
-        <update_rate>100</update_rate>
-      </plugin>
-    </gazebo>
-  </xacro:macro>
 </robot>

File: urdf/dynaarm_standalone.urdf.xacro (robot description, xacro)
@@ -22,4 +22,6 @@
   <!-- v1, v2, ... -->
   <xacro:arg name="version" default="baracuda12" />
+  <!-- Path to ros2_control controller config file -->
+  <xacro:arg name="controller_path" default="" />
   <xacro:include filename="$(find dynaarm_description)/urdf/dynaarm.urdf.xacro" />
   <link name="world" />
@@ -35,3 +37,11 @@
     <origin xyz="0 0 0" rpy="0.0 0.0 0.0" />
   </xacro:dynaarm>
+  <!-- DynaArm Gazebo Ros2 Control-->
+  <gazebo>
+    <plugin filename="libgz_ros2_control-system.so"
+      name="gz_ros2_control::GazeboSimROS2ControlPlugin">
+      <parameters>$(arg controller_path)</parameters>
+      <update_rate>100</update_rate>
+    </plugin>
+  </gazebo>
 </robot>

File: urdf/dynaarm_standalone_dual.urdf.xacro (robot description, xacro)
@@ -22,4 +22,6 @@
   <!-- v1, v2, ... -->
   <xacro:arg name="version" default="baracuda12" />
+  <!-- Path to ros2_control controller config file -->
+  <xacro:arg name="controller_path" default="" />
   <xacro:include filename="$(find dynaarm_description)/urdf/dynaarm.urdf.xacro" />
   <link name="world" />
@@ -46,3 +48,11 @@
     <origin xyz="1.0 0 0" rpy="0.0 0.0 0.0" />
   </xacro:dynaarm>
+  <!-- DynaArm Gazebo Ros2 Control-->
+  <gazebo>
+    <plugin filename="libgz_ros2_control-system.so"
+      name="gz_ros2_control::GazeboSimROS2ControlPlugin">
+      <parameters>$(arg controller_path)</parameters>
+      <update_rate>100</update_rate>
+    </plugin>
+  </gazebo>
 </robot>
