Commit message: refactor(urdf):changed base_link from world to base_link, updated integration of ros2control gz plugin

File: urdf/dynaarm_standalone.urdf.xacro (robot description, xacro)
@@ -25,8 +25,8 @@
   <xacro:arg name="controller_path" default="" />
   <xacro:include filename="$(find dynaarm_description)/urdf/dynaarm.urdf.xacro" />
-  <link name="world" />
+  <link name="base_link" />
   <!-- create an instance of the dynaarm xacro macro and fix its base, move it up such that it doesn't intersect with the ground -->
   <xacro:dynaarm tf_prefix="$(arg tf_prefix)"
-                parent_link="world"
+                parent_link="base_link"
                 dof="$(arg dof)"
                 collision="$(arg collision)"
@@ -37,11 +37,8 @@
     <origin xyz="0 0 0" rpy="0.0 0.0 0.0" />
   </xacro:dynaarm>
-  <!-- DynaArm Gazebo Ros2 Control-->
-  <gazebo>
-    <plugin filename="libgz_ros2_control-system.so"
-      name="gz_ros2_control::GazeboSimROS2ControlPlugin">
-      <parameters>$(arg controller_path)</parameters>
-      <update_rate>100</update_rate>
-    </plugin>
-  </gazebo>
+  <!-- Gazebo Ros2 Control -->
+  <xacro:include filename="$(find duatic_control)/urdf/plugins.urdf.xacro" />
+  <xacro:control namespace="$(arg namespace)">
+    <remapping>cmd_vel:=cmd_vel</remapping> <!-- TODO: This line only exists, because otherwise the xacro doesn't compile -->
+  </xacro:control>
 </robot>

File: urdf/dynaarm_standalone_dual.urdf.xacro (robot description, xacro)
@@ -25,8 +25,8 @@
   <xacro:arg name="controller_path" default="" />
   <xacro:include filename="$(find dynaarm_description)/urdf/dynaarm.urdf.xacro" />
-  <link name="world" />
+  <link name="base_link" />
   <!-- create two dynaarms and fix their bases, move them up such that they do not intersect with the ground -->
   <xacro:dynaarm tf_prefix="$(arg tf_prefix)_1/"
-                parent_link="world"
+                parent_link="base_link"
                 dof="$(arg dof)"
                 mode="$(arg mode)"
@@ -39,5 +39,5 @@
   <!-- Note: for a real world application you would pass different parameters for both arms (e.g. different ethercat_bus)-->
   <xacro:dynaarm tf_prefix="$(arg tf_prefix)_2/"
-                parent_link="world"
+                parent_link="base_link"
                 dof="$(arg dof)"
                 mode="$(arg mode)"
@@ -49,10 +49,8 @@
   </xacro:dynaarm>
   <!-- DynaArm Gazebo Ros2 Control-->
-  <gazebo>
-    <plugin filename="libgz_ros2_control-system.so"
-      name="gz_ros2_control::GazeboSimROS2ControlPlugin">
-      <parameters>$(arg controller_path)</parameters>
-      <update_rate>100</update_rate>
-    </plugin>
-  </gazebo>
+  <!-- Gazebo Ros2 Control -->
+  <xacro:include filename="$(find duatic_control)/urdf/plugins.urdf.xacro" />
+  <xacro:control namespace="$(arg namespace)">
+    <remapping>cmd_vel:=cmd_vel</remapping> <!-- TODO: This line only exists, because otherwise the xacro doesn't compile -->
+  </xacro:control>
 </robot>

Commit message: Refactor (#52)
* feat: move gz_ros2_control plugin from template urdf to standalone urdfs

* refactor(urdf):changed base_link from world to base_link, updated integration of ros2control gz plugin

* feat(rviz): updated config

* feat(config): added dynaarm.srdf

File: urdf/dynaarm_standalone.urdf.xacro (robot description, xacro)
@@ -22,9 +22,11 @@
   <!-- v1, v2, ... -->
   <xacro:arg name="version" default="baracuda12" />
+  <!-- Path to ros2_control controller config file -->
+  <xacro:arg name="controller_path" default="" />
   <xacro:include filename="$(find dynaarm_description)/urdf/dynaarm.urdf.xacro" />
-  <link name="world" />
+  <link name="base_link" />
   <!-- create an instance of the dynaarm xacro macro and fix its base, move it up such that it doesn't intersect with the ground -->
   <xacro:dynaarm tf_prefix="$(arg tf_prefix)"
-                parent_link="world"
+                parent_link="base_link"
                 dof="$(arg dof)"
                 collision="$(arg collision)"
@@ -35,3 +37,8 @@
     <origin xyz="0 0 0" rpy="0.0 0.0 0.0" />
   </xacro:dynaarm>
+  <!-- Gazebo Ros2 Control -->
+  <xacro:include filename="$(find duatic_control)/urdf/plugins.urdf.xacro" />
+  <xacro:control namespace="$(arg namespace)">
+    <remapping>cmd_vel:=cmd_vel</remapping> <!-- TODO: This line only exists, because otherwise the xacro doesn't compile -->
+  </xacro:control>
 </robot>

File: urdf/dynaarm_standalone_dual.urdf.xacro (robot description, xacro)
@@ -22,9 +22,11 @@
   <!-- v1, v2, ... -->
   <xacro:arg name="version" default="baracuda12" />
+  <!-- Path to ros2_control controller config file -->
+  <xacro:arg name="controller_path" default="" />
   <xacro:include filename="$(find dynaarm_description)/urdf/dynaarm.urdf.xacro" />
-  <link name="world" />
+  <link name="base_link" />
   <!-- create two dynaarms and fix their bases, move them up such that they do not intersect with the ground -->
   <xacro:dynaarm tf_prefix="$(arg tf_prefix)_1/"
-                parent_link="world"
+                parent_link="base_link"
                 dof="$(arg dof)"
                 mode="$(arg mode)"
@@ -37,5 +39,5 @@
   <!-- Note: for a real world application you would pass different parameters for both arms (e.g. different ethercat_bus)-->
   <xacro:dynaarm tf_prefix="$(arg tf_prefix)_2/"
-                parent_link="world"
+                parent_link="base_link"
                 dof="$(arg dof)"
                 mode="$(arg mode)"
@@ -46,3 +48,9 @@
     <origin xyz="1.0 0 0" rpy="0.0 0.0 0.0" />
   </xacro:dynaarm>
+  <!-- DynaArm Gazebo Ros2 Control-->
+  <!-- Gazebo Ros2 Control -->
+  <xacro:include filename="$(find duatic_control)/urdf/plugins.urdf.xacro" />
+  <xacro:control namespace="$(arg namespace)">
+    <remapping>cmd_vel:=cmd_vel</remapping> <!-- TODO: This line only exists, because otherwise the xacro doesn't compile -->
+  </xacro:control>
 </robot>
