Commit message: switched default to 6dof

File: dynaarm_description_common/resource/xacro/dynaarm_common.urdf.xacro (robot description, xacro)
@@ -73,6 +73,7 @@
             <inertial>
                 <origin xyz="0.0 0.0 0.0" rpy="0 0 0" />
-                <mass value="0.02" />
-                <inertia ixx="0.01" ixy="0.0" iyy="0.01" ixz="0.0" iyz="0.0" izz="0.01" />
+                <mass value="0.001" />
+                <inertia ixx="0.0000001" ixy="0.0" iyy="0.0000001" ixz="0.0" iyz="0.0"
+                    izz="0.0000001" />
             </inertial>
         </link>

File: dynaarm_description_common/resource/xacro/dynaarm_parameters.urdf.xacro (robot description, xacro)
@@ -82,5 +82,5 @@
         <xacro:property name="joint_ee_xyz" value="0.0 0.0 0.05" />
         <xacro:property name="joint_ee_origin_xyz" value="0.0 0.0 0.05" />
-        <xacro:property name="joint_ee_origin_4dof_xyz" value="0.0 0.0 0.25" />
+        <xacro:property name="joint_ee_origin_4dof_xyz" value="0.0 0.0 0.4" />
         <xacro:property name="joint_ee_origin_rpy" value="0.0 0.0 ${J_PI/2}" />
         <xacro:property name="joint_ee_origin_4dof_rpy" value="0.0 0.0 ${J_PI/2}" />

File: dynaarm_standalone_description/resource/xacro/dynaarm_standalone.urdf.xacro (robot description, xacro)
@@ -1,5 +1,5 @@
 <robot name="dynaarm" xmlns:xacro="http://www.ros.org/wiki/xacro">
   <!-- 4dof, 6dof -->
-  <xacro:arg name="dynaarm_dof_configuration_arg" default="4dof" />
+  <xacro:arg name="dynaarm_dof_configuration_arg" default="6dof" />
   <!-- real, mock, sim -->
   <xacro:arg name="hardware_interface_type_arg" default="mock" />
