Commit message: Integrating the next version robot.

File: xacro/common/dynaarm.ros2control.xacro (robot description, xacro)
@@ -45,10 +45,10 @@
       <xacro:dynaarm_ros2control_joint name="${tf_prefix}SH_ROT" address="1" />
       <xacro:dynaarm_ros2control_joint name="${tf_prefix}SH_FLE" address="2" />
-      <xacro:dynaarm_ros2control_joint name="${tf_prefix}EL_FLE" address="3" />
+      <!-- <xacro:dynaarm_ros2control_joint name="${tf_prefix}EL_FLE" address="3" />
       <xacro:dynaarm_ros2control_joint name="${tf_prefix}FA_ROT" address="4" />
       <xacro:if value="${dof == '6dof'}">
         <xacro:dynaarm_ros2control_joint name="${tf_prefix}WRIST_1" address="5" />
         <xacro:dynaarm_ros2control_joint name="${tf_prefix}WRIST_2" address="6" />
-      </xacro:if>
+      </xacro:if> -->
     </ros2_control>
   </xacro:macro>

File: xacro/dynaarm_standalone.urdf.xacro (robot description, xacro)
@@ -9,9 +9,12 @@
   <!-- Change to add covers to the arm -->
   <xacro:arg name="covers" default="false" />
+  <!-- v1, v2, ... -->
+  <xacro:arg name="version" default="v2" />
+  <xacro:property name="version" value="$(arg version)" />
   <xacro:property name="dof" value="$(arg dof)" />
   <xacro:property name="mode" value="$(arg mode)" />
   <xacro:property name="ethercat_bus" value="$(arg ethercat_bus)" />
   <xacro:property name="covers" value="$(arg covers)" />
-  <xacro:include filename="$(find dynaarm_description)/xacro/common/dynaarm_macro_${dof}.urdf.xacro" />
+  <xacro:include filename="$(find dynaarm_description)/xacro/${version}/dynaarm_macro_${dof}.urdf.xacro" />
   <link name="world" />
   <!-- create dynaarm and fix its base, move it up such that is doesn't intersect with the ground -->
