Commit message: Inserted the first collision mesh and change the collision origins

File: urdf/common/dynaarm_parameters_v2.urdf.xacro (robot description, xacro)
@@ -55,5 +55,5 @@
   <xacro:property name="joint_2_name" value="${tf_prefix}SH_FLE" />
   <xacro:property name="joint_2_joint_type" value="revolute" />
-  <xacro:property name="joint_2_axis_xyz" value="0 0 -1" />
+  <xacro:property name="joint_2_axis_xyz" value="0 0 1" />
   <xacro:property name="joint_2_origin_xyz" value="0 0 0.047" />
   <xacro:property name="joint_2_origin_rpy" value="${J_PI/2} ${-J_PI/2} 0" />
@@ -95,69 +95,69 @@
   <xacro:property name="joint_ee_origin_4dof_rpy" value="0.0 0.0 ${J_PI/2}" />
   <xacro:property name="joint_ee_rpy" value="0 0 0" />
-  <!-- Base Robot -->
+<!-- Base Robot -->
   <xacro:property name="base_inertial">
     <inertial>
-      <mass value="1.894" />
+      <mass value="2.00205474" />
       <origin
-        xyz="${0.008222641*mm_to_m} ${-0.310936808*mm_to_m} ${-36.738569268*mm_to_m}"
+        xyz="0.00347077 0.00328869 -0.0488212"
         rpy="0 0 0" />
-      <inertia ixx="${2767.258474185*mm2_to_m2}" iyy="${2895.160105441*mm2_to_m2}"
-        izz="${3138.952392041*mm2_to_m2}" ixy="${0.393414115*mm2_to_m2}"
-        ixz="${-0.149570272*mm2_to_m2}" iyz="${25.32409214*mm2_to_m2}" />
+      <inertia ixx="0.00403342" iyy="0.00417534"
+        izz="0.00460211" ixy="0.00040828"
+        ixz="-0.00018775" iyz="-0.0001821" />
     </inertial>
   </xacro:property>
   <xacro:property name="link01_inertial">
     <inertial>
-      <mass value="2.644" />
-      <origin xyz="0.0 0.0 ${-1.7336*mm_to_m}" rpy="0 0 0" />
-      <inertia ixx="${10301.21*mm2_to_m2}" iyy="${3016.50*mm2_to_m2}"
-        izz="${10099.04*mm2_to_m2}" ixy="${-50.85*mm2_to_m2}"
-        ixz="${0.0*mm2_to_m2}" iyz="${0.0*mm2_to_m2}" />
+      <mass value="2.73096676" />
+      <origin xyz="0.00001348 0.00013521 0.0430259" rpy="0 0 0" />
+      <inertia ixx="0.01291668" iyy="0.00874231"
+        izz="0.01243436" ixy="0.0000044"
+        ixz="-0.00000179" iyz="-0.00000203" />
     </inertial>
   </xacro:property>
   <xacro:property name="link02_inertial">
     <inertial>
-      <mass value="1.394" />
-      <origin xyz="${211.09*mm_to_m} ${0.022*mm_to_m} ${-0.317*mm_to_m}"
+      <mass value="1.72040464" />
+      <origin xyz="0.20391301 -0.00000528 -0.00015224"
         rpy="0 0 0" />
-      <inertia ixx="${1161.79*mm2_to_m2}" iyy="${46092.126*mm2_to_m2}"
-        izz="${46279.53*mm2_to_m2}" ixy="${-0.72*mm2_to_m2}"
-        ixz="${-140.45*mm2_to_m2}" iyz="${0.007*mm2_to_m2}" />
+      <inertia ixx="0.00155499" iyy="0.05067934"
+        izz="0.0507131" ixy="0.00000098"
+        ixz="0.00004108" iyz="-0.00000143" />
     </inertial>
   </xacro:property>
   <xacro:property name="link03_inertial">
     <inertial>
-      <mass value="1.1" />
-      <origin xyz="${6.8*mm_to_m} ${-84.8*mm_to_m} ${-0.6*mm_to_m}" rpy="0 0 0" />
-      <inertia ixx="${1384.3*mm2_to_m2}" iyy="${716.8*mm2_to_m2}"
-        izz="${1130.1*mm2_to_m2}" ixy="${-41.6*mm2_to_m2}"
-        ixz="${8.5*mm2_to_m2}" iyz="${-10.5*mm2_to_m2}" />
+      <mass value="0.82320237" />
+      <origin xyz="0.00383866 -0.07802638 -0.00026928" rpy="0 0 0" />
+      <inertia ixx="0.00107419" iyy="0.00087121"
+        izz="0.00113856" ixy="0.00004166"
+        ixz="-0.00000398" iyz="-0.0000119" />
     </inertial>
   </xacro:property>
   <xacro:property name="link04_inertial">
     <inertial>
-      <mass value="0.342" />
-      <origin xyz="0.0 0.0 0.2143" rpy="0 0 0" />
-      <inertia ixx="${7000*mm2_to_m2}" iyy="${7000*mm2_to_m2}"
-        izz="${6400*mm2_to_m2}" ixy="${0.0*mm2_to_m2}"
-        ixz="${0.0*mm2_to_m2}" iyz="${0.0*mm2_to_m2}" />
+      <mass value="1.15674546" />
+      <origin xyz="-0.00115165 0.00001056 0.30067314" rpy="0 0 0" />
+      <inertia ixx="0.03129519" iyy="0.03125954"
+        izz="0.00090392" ixy="0.00000151"
+        ixz="-0.00017171" iyz="0.00000159" />
     </inertial>
   </xacro:property>
   <xacro:property name="link05_inertial">
     <inertial>
-      <mass value="1.69" />
-      <origin xyz="0.047 0.0 0.029" rpy="0 0 0" />
-      <inertia ixx="${1672*mm2_to_m2}" iyy="${4985*mm2_to_m2}"
-        izz="${5210*mm2_to_m2}" ixy="${0*mm2_to_m2}"
-        ixz="${129.7*mm2_to_m2}" iyz="${-3.7*mm2_to_m2}" />
+      <mass value="0.75007482" />
+      <origin xyz="0.07972553 -0.00005038 0.02334747" rpy="0 0 0" />
+      <inertia ixx="0.00065953" iyy="0.00088282"
+        izz="0.00078106" ixy="0.00000076"
+        ixz="0.00011795" iyz="-0.00000079" />
     </inertial>
   </xacro:property>
   <xacro:property name="link06_inertial">
     <inertial>
-      <mass value="0.1" />
-      <origin xyz="0.0 0.0 0.0064" rpy="0 0 0" />
-      <inertia ixx="${115*mm2_to_m2}" iyy="${115*mm2_to_m2}"
-        izz="${115*mm2_to_m2}" ixy="${0.0*mm2_to_m2}" ixz="${0*mm2_to_m2}"
-        iyz="${0.0*mm2_to_m2}" />
+      <mass value="0.0478406" />
+      <origin xyz="0.00045711 0.00000557 0.00344945" rpy="0 0 0" />
+      <inertia ixx="0.00001366" iyy="0.00001419"
+        izz="0.00002702" ixy="0"
+        ixz="0.00000008" iyz="0" />
     </inertial>
   </xacro:property>
@@ -211,45 +211,61 @@
     </inertial>
   </xacro:property>
-  <!-- Collision properties -->
-  <xacro:property name="base_collision">
-    <collision>
-      <origin xyz="0 0 -0.04" rpy="0 0 0" />
-      <geometry>
-        <cylinder radius="0.06" length="0.08" />
-      </geometry>
-    </collision>
-  </xacro:property>
-  <xacro:property name="link01_collision">
-    <collision>
-      <origin xyz="0 0 0" rpy="1.57 0 0" />
-      <geometry>
-        <cylinder radius="0.05" length="0.24" />
-      </geometry>
-    </collision>
-  </xacro:property>
-  <xacro:property name="link02_collision">
-    <collision>
-      <origin xyz="0.25 0 0" rpy="1.57 0 1.57" />
-      <geometry>
-        <cylinder radius="0.05" length="0.4" />
-      </geometry>
-    </collision>
-  </xacro:property>
-  <xacro:property name="link03_collision">
-    <collision>
-      <origin xyz="0.185 -0.0935 0" rpy="0 1.57 0" />
-      <geometry>
-        <cylinder radius="0.047" length="0.46" />
-      </geometry>
-    </collision>
-  </xacro:property>
-  <xacro:property name="link05_collision">
-    <collision>
-      <origin xyz="${0.045} 0 0.03" rpy="0 ${J_PI/2} 0" />
-      <geometry>
-        <cylinder radius="0.055" length="0.18" />
-      </geometry>
-    </collision>
-  </xacro:property>
+<!-- Collision properties -->
+<xacro:property name="base_collision">
+  <collision>
+    <origin xyz="0 0 0" rpy="0 0 0" />
+    <geometry>
+      <mesh filename="package://dynaarm_description/meshes/collision_meshes/base_collision_mesh.STL" scale="1 1 1" />
+    </geometry>
+  </collision>
+</xacro:property>
+<xacro:property name="link01_collision">
+  <collision>
+    <origin xyz="0 0 0.0105" rpy="0 0 0" />
+    <geometry>
+      <cylinder radius="0.05" length="0.24" />
+    </geometry>
+  </collision>
+</xacro:property>
+<xacro:property name="link02_collision">
+  <collision>
+    <origin xyz="0 0 0.047" rpy="${J_PI/2} ${-J_PI/2} 0" />
+    <geometry>
+      <cylinder radius="0.05" length="0.4" />
+    </geometry>
+  </collision>
+</xacro:property>
+<xacro:property name="link03_collision">
+  <collision>
+    <origin xyz="0.4127 0 0" rpy="${J_PI} 0 0" />
+    <geometry>
+      <cylinder radius="0.047" length="0.46" />
+    </geometry>
+  </collision>
+</xacro:property>
+<xacro:property name="link04_collision">
+  <collision>
+    <origin xyz="0.0262 -0.0855 0" rpy="${J_PI/2} 0 ${J_PI/2}" />
+    <geometry>
+      <cylinder radius="0.05" length="0.2" />
+    </geometry>
+  </collision>
+</xacro:property>
+<xacro:property name="link05_collision">
+  <collision>
+    <origin xyz="0.0295 0 0.4207" rpy="0 ${-J_PI/2} 0" />
+    <geometry>
+      <cylinder radius="0.055" length="0.18" />
+    </geometry>
+  </collision>
+</xacro:property>
+<xacro:property name="link06_collision">
+  <collision>
+    <origin xyz="0.117 0.0 0.0295" rpy="${-J_PI/2} ${J_PI/2} ${-J_PI/2}" />
+    <geometry>
+      <cylinder radius="0.045" length="0.16" />
+    </geometry>
+  </collision>
+</xacro:property>
   <!-- set the ee_parent relative to the DoF -->
   <xacro:property name="ee_parent" value="${base}" />

Commit message: Added small sized dae file

File: urdf/common/dynaarm_parameters_v2.urdf.xacro (robot description, xacro)
@@ -17,5 +17,5 @@
   <xacro:if value="${covers}">
     <xacro:property name="base_mesh" value="base_mesh.STL" />
-    <xacro:property name="link01_mesh" value="shoulder_mesh.STL" />
+    <xacro:property name="link01_mesh" value="shoulderColor.dae" />
     <xacro:property name="link02_mesh" value="upperarm_mesh.STL" />
     <xacro:property name="link03_mesh" value="elbow_mesh.STL" />
@@ -24,5 +24,5 @@
     <xacro:property name="link06_mesh" value="wrist2_mesh.STL" />
     <xacro:property name="base_cover_mesh" value="base_mesh.STL" />
-    <xacro:property name="link01_cover_mesh" value="shoulder_mesh.STL" />
+    <xacro:property name="link01_cover_mesh" value="shoulderColor.dae" />
     <xacro:property name="link02_cover_mesh" value="upperarm_mesh.STL" />
     <xacro:property name="link03_cover_mesh" value="elbow_mesh.STL" />
@@ -33,5 +33,5 @@
   <xacro:unless value="${covers}">
     <xacro:property name="base_mesh" value="base_mesh.STL" />
-    <xacro:property name="link01_mesh" value="shoulder_mesh.STL" />
+    <xacro:property name="link01_mesh" value="shoulderColor.dae" />
     <xacro:property name="link02_mesh" value="upperarm_mesh.STL" />
     <xacro:property name="link03_mesh" value="elbow_mesh.STL" />

Commit message: Changes to add camera mounting point

File: urdf/common/dynaarm_parameters_v2.urdf.xacro (robot description, xacro)
@@ -10,4 +10,5 @@
   <xacro:property name="link02" value="${tf_prefix}UPPERARM" />
   <xacro:property name="link03" value="${tf_prefix}ELBOW" />
+  <xacro:property name="link03_cam" value="${tf_prefix}ELBOW_CAMERA_MOUNT" />
   <xacro:property name="link04" value="${tf_prefix}FOREARM" />
   <xacro:property name="link05" value="${tf_prefix}WRIST_1" />
@@ -20,4 +21,5 @@
     <xacro:property name="link02_mesh" value="upperarm_mesh.STL" />
     <xacro:property name="link03_mesh" value="elbow_mesh.STL" />
+    <xacro:property name="link03_cam_mesh" value=<box size="0.01 0.01 0.01"/>/>
     <xacro:property name="link04_mesh" value="forearm_mesh.STL" />
     <xacro:property name="link05_mesh" value="wrist1_mesh.STL" />
@@ -36,4 +38,5 @@
     <xacro:property name="link02_mesh" value="upperarm_mesh.STL" />
     <xacro:property name="link03_mesh" value="elbow_mesh.STL" />
+    <xacro:property name="link03_cam_mesh" value=<box size="0.01 0.01 0.01"/>/>
     <xacro:property name="link04_mesh" value="forearm_mesh.STL" />
     <xacro:property name="link05_mesh" value="wrist1_mesh.STL" />
@@ -67,4 +70,9 @@
   <xacro:property name="joint_3_lower_limit" value="-0.05" />
   <xacro:property name="joint_3_upper_limit" value="${J_PI}" />
+  <xacro:property name="joint_3_cam_name" value="${tf_prefix}EL_CAMERA" />
+  <xacro:property name="joint_3_cam_joint_type" value="fixed" />
+  <xacro:property name="joint_3_cam_axis_xyz" value="0 0 0" />
+  <xacro:property name="joint_3_cam_origin_xyz" value="0.0345 -0.1235 0" />
+  <xacro:property name="joint_3_cam_origin_rpy" value="0.0 0.0 0.0" />
   <xacro:property name="joint_4_name" value="${tf_prefix}FA_ROT" />
   <xacro:property name="joint_4_joint_type" value="revolute" />
@@ -162,4 +170,13 @@
     </inertial>
   </xacro:property>
+  <xacro:property name="link03_cam_inertial">
+    <inertial>
+      <mass value="1e-6" />
+      <origin xyz="0.0 0.0 0.0" rpy="0 0 0" />
+      <inertia ixx="1e-6" iyy="1e-6"
+        izz="1e-6" ixy="1e-6"
+        ixz="1e-6" iyz="1e-6" />
+    </inertial>
+  </xacro:property>
   <!-- Covers -->
   <xacro:property name="base_cover_inertial">

File: urdf/dynaarm.urdf.xacro (robot description, xacro)
@@ -147,4 +147,15 @@
         <origin xyz="${joint_3_origin_xyz}" rpy="${joint_3_origin_rpy}" />
       </xacro:dynaarm_revolute_joint>
+      <!--dynaarm_ELBOW_CAMERA_BASE-->
+      <xacro:dynaarm_link_w_collision link_name="${link03_cam}" file_name="${link03_cam_mesh}">
+        <link_inertia>
+          <xacro:insert_block name="link03_cam_inertial" />
+        </link_inertia>
+      <!-- Camera fixed on elbow -->
+        <xacro:dynaarm_joint_fixed joint_name="${joint_03_cam_name}"
+        parent="${link03}"
+          child="${link03_cam}">
+          <origin xyz="${joint_3_cam_origin_xyz}" rpy="${joint_3_cam_origin_rpy}" />
+        </xacro:dynaarm_joint_fixed>
       <!-- 3 Dof & Covers-->
       <xacro:if value="${covers}">

Commit message: Fixes to the camera mounting point

File: urdf/common/dynaarm_parameters_v2.urdf.xacro (robot description, xacro)
@@ -21,5 +21,4 @@
     <xacro:property name="link02_mesh" value="upperarm_mesh.STL" />
     <xacro:property name="link03_mesh" value="elbow_mesh.STL" />
-    <xacro:property name="link03_cam_mesh" value=<box size="0.01 0.01 0.01"/>/>
     <xacro:property name="link04_mesh" value="forearm_mesh.STL" />
     <xacro:property name="link05_mesh" value="wrist1_mesh.STL" />
@@ -38,5 +37,4 @@
     <xacro:property name="link02_mesh" value="upperarm_mesh.STL" />
     <xacro:property name="link03_mesh" value="elbow_mesh.STL" />
-    <xacro:property name="link03_cam_mesh" value=<box size="0.01 0.01 0.01"/>/>
     <xacro:property name="link04_mesh" value="forearm_mesh.STL" />
     <xacro:property name="link05_mesh" value="wrist1_mesh.STL" />
@@ -103,5 +101,5 @@
   <xacro:property name="joint_ee_origin_4dof_rpy" value="0.0 0.0 ${J_PI/2}" />
   <xacro:property name="joint_ee_rpy" value="0 0 0" />
-<!-- Base Robot -->
+  <!-- Base Robot -->
   <xacro:property name="base_inertial">
     <inertial>
@@ -228,61 +226,63 @@
     </inertial>
   </xacro:property>
-<!-- Collision properties -->
-<xacro:property name="base_collision">
-  <collision>
-    <origin xyz="0 0 0" rpy="0 0 0" />
-    <geometry>
-      <mesh filename="package://dynaarm_description/meshes/collision_meshes/base_collision_mesh.STL" scale="1 1 1" />
-    </geometry>
-  </collision>
-</xacro:property>
-<xacro:property name="link01_collision">
-  <collision>
-    <origin xyz="0 0 0.0105" rpy="0 0 0" />
-    <geometry>
-      <cylinder radius="0.05" length="0.24" />
-    </geometry>
-  </collision>
-</xacro:property>
-<xacro:property name="link02_collision">
-  <collision>
-    <origin xyz="0 0 0.047" rpy="${J_PI/2} ${-J_PI/2} 0" />
-    <geometry>
-      <cylinder radius="0.05" length="0.4" />
-    </geometry>
-  </collision>
-</xacro:property>
-<xacro:property name="link03_collision">
-  <collision>
-    <origin xyz="0.4127 0 0" rpy="${J_PI} 0 0" />
-    <geometry>
-      <cylinder radius="0.047" length="0.46" />
-    </geometry>
-  </collision>
-</xacro:property>
-<xacro:property name="link04_collision">
-  <collision>
-    <origin xyz="0.0262 -0.0855 0" rpy="${J_PI/2} 0 ${J_PI/2}" />
-    <geometry>
-      <cylinder radius="0.05" length="0.2" />
-    </geometry>
-  </collision>
-</xacro:property>
-<xacro:property name="link05_collision">
-  <collision>
-    <origin xyz="0.0295 0 0.4207" rpy="0 ${-J_PI/2} 0" />
-    <geometry>
-      <cylinder radius="0.055" length="0.18" />
-    </geometry>
-  </collision>
-</xacro:property>
-<xacro:property name="link06_collision">
-  <collision>
-    <origin xyz="0.117 0.0 0.0295" rpy="${-J_PI/2} ${J_PI/2} ${-J_PI/2}" />
-    <geometry>
-      <cylinder radius="0.045" length="0.16" />
-    </geometry>
-  </collision>
-</xacro:property>
+  <!-- Collision properties -->
+  <xacro:property name="base_collision">
+    <collision>
+      <origin xyz="0 0 0" rpy="0 0 0" />
+      <geometry>
+        <mesh
+          filename="package://dynaarm_description/meshes/collision_meshes/base_collision_mesh.STL"
+          scale="1 1 1" />
+      </geometry>
+    </collision>
+  </xacro:property>
+  <xacro:property name="link01_collision">
+    <collision>
+      <origin xyz="0 0 0.0105" rpy="0 0 0" />
+      <geometry>
+        <cylinder radius="0.05" length="0.24" />
+      </geometry>
+    </collision>
+  </xacro:property>
+  <xacro:property name="link02_collision">
+    <collision>
+      <origin xyz="0 0 0.047" rpy="${J_PI/2} ${-J_PI/2} 0" />
+      <geometry>
+        <cylinder radius="0.05" length="0.4" />
+      </geometry>
+    </collision>
+  </xacro:property>
+  <xacro:property name="link03_collision">
+    <collision>
+      <origin xyz="0.4127 0 0" rpy="${J_PI} 0 0" />
+      <geometry>
+        <cylinder radius="0.047" length="0.46" />
+      </geometry>
+    </collision>
+  </xacro:property>
+  <xacro:property name="link04_collision">
+    <collision>
+      <origin xyz="0.0262 -0.0855 0" rpy="${J_PI/2} 0 ${J_PI/2}" />
+      <geometry>
+        <cylinder radius="0.05" length="0.2" />
+      </geometry>
+    </collision>
+  </xacro:property>
+  <xacro:property name="link05_collision">
+    <collision>
+      <origin xyz="0.0295 0 0.4207" rpy="0 ${-J_PI/2} 0" />
+      <geometry>
+        <cylinder radius="0.055" length="0.18" />
+      </geometry>
+    </collision>
+  </xacro:property>
+  <xacro:property name="link06_collision">
+    <collision>
+      <origin xyz="0.117 0.0 0.0295" rpy="${-J_PI/2} ${J_PI/2} ${-J_PI/2}" />
+      <geometry>
+        <cylinder radius="0.045" length="0.16" />
+      </geometry>
+    </collision>
+  </xacro:property>
   <!-- set the ee_parent relative to the DoF -->
   <xacro:property name="ee_parent" value="${base}" />

File: urdf/dynaarm.urdf.xacro (robot description, xacro)
@@ -9,5 +9,6 @@
     <xacro:property name="ee_parent" value="${base}" />
     <xacro:include filename="$(find dynaarm_description)/urdf/common/dynaarm_common.urdf.xacro" />
-    <xacro:include filename="$(find dynaarm_description)/urdf/common/dynaarm_parameters_${version}.urdf.xacro" />
+    <xacro:include
+      filename="$(find dynaarm_description)/urdf/common/dynaarm_parameters_${version}.urdf.xacro" />
     <xacro:include filename="$(find dynaarm_description)/urdf/common/dynaarm.ros2control.xacro" />
     <xacro:dynaarm_joint_fixed joint_name="${joint_base_name}"
@@ -148,14 +149,23 @@
       </xacro:dynaarm_revolute_joint>
       <!--dynaarm_ELBOW_CAMERA_BASE-->
-      <xacro:dynaarm_link_w_collision link_name="${link03_cam}" file_name="${link03_cam_mesh}">
-        <link_inertia>
-          <xacro:insert_block name="link03_cam_inertial" />
-        </link_inertia>
+      <link name="${link03_cam}">
+        <visual>
+          <origin rpy="0 0 0" xyz="0 0 0" />
+          <geometry>
+            <box size="0.001 0.001 0.001" />
+          </geometry>
+        </visual>
+        <inertial>
+          <origin rpy="0 0 0" xyz="0.0 0.0 0.0" />
+          <mass value="0.001" />
+          <inertia ixx="0.0000001" ixy="0.0" ixz="0.0" iyy="0.0000001" iyz="0.0" izz="0.0000001" />
+        </inertial>
+      </link>
       <!-- Camera fixed on elbow -->
-        <xacro:dynaarm_joint_fixed joint_name="${joint_03_cam_name}"
+      <xacro:dynaarm_joint_fixed joint_name="${joint_3_cam_name}"
         parent="${link03}"
-          child="${link03_cam}">
-          <origin xyz="${joint_3_cam_origin_xyz}" rpy="${joint_3_cam_origin_rpy}" />
-        </xacro:dynaarm_joint_fixed>
+        child="${link03_cam}">
+        <origin xyz="${joint_3_cam_origin_xyz}" rpy="${joint_3_cam_origin_rpy}" />
+      </xacro:dynaarm_joint_fixed>
       <!-- 3 Dof & Covers-->
       <xacro:if value="${covers}">

Commit message: Added the second (wrist) camera mount to urdf

File: urdf/common/dynaarm_parameters_v2.urdf.xacro (robot description, xacro)
@@ -13,4 +13,5 @@
   <xacro:property name="link04" value="${tf_prefix}FOREARM" />
   <xacro:property name="link05" value="${tf_prefix}WRIST_1" />
+  <xacro:property name="link05_cam" value="${tf_prefix}WRIST_1_CAMERA_MOUNT" />
   <xacro:property name="link06" value="${tf_prefix}WRIST_2" />
   <xacro:property name="end_effector" value="${tf_prefix}END_EFFECTOR" />
@@ -87,4 +88,9 @@
   <xacro:property name="joint_5_lower_limit" value="${-J_PI/2}" />
   <xacro:property name="joint_5_upper_limit" value="${J_PI/2}" />
+  <xacro:property name="joint_5_cam_name" value="${tf_prefix}WRIST_1_CAMERA" />
+  <xacro:property name="joint_5_cam_joint_type" value="fixed" />
+  <xacro:property name="joint_5_cam_axis_xyz" value="0 0 0" />
+  <xacro:property name="joint_5_cam_origin_xyz" value="0.032 0 -0.017" />
+  <xacro:property name="joint_5_cam_origin_rpy" value="0.0 0.0 0.0" />
   <xacro:property name="joint_6_name" value="${tf_prefix}WRIST_2" />
   <xacro:property name="joint_6_joint_type" value="revolute" />
@@ -141,4 +147,13 @@
     </inertial>
   </xacro:property>
+  <xacro:property name="link03_cam_inertial">
+    <inertial>
+      <mass value="1e-6" />
+      <origin xyz="0.0 0.0 0.0" rpy="0 0 0" />
+      <inertia ixx="1e-6" iyy="1e-6"
+        izz="1e-6" ixy="1e-6"
+        ixz="1e-6" iyz="1e-6" />
+    </inertial>
+  </xacro:property>
   <xacro:property name="link04_inertial">
     <inertial>
@@ -159,4 +174,13 @@
     </inertial>
   </xacro:property>
+  <xacro:property name="link05_cam_inertial">
+    <inertial>
+      <mass value="1e-6" />
+      <origin xyz="0.0 0.0 0.0" rpy="0 0 0" />
+      <inertia ixx="1e-6" iyy="1e-6"
+        izz="1e-6" ixy="1e-6"
+        ixz="1e-6" iyz="1e-6" />
+    </inertial>
+  </xacro:property>
   <xacro:property name="link06_inertial">
     <inertial>
@@ -168,13 +192,4 @@
     </inertial>
   </xacro:property>
-  <xacro:property name="link03_cam_inertial">
-    <inertial>
-      <mass value="1e-6" />
-      <origin xyz="0.0 0.0 0.0" rpy="0 0 0" />
-      <inertia ixx="1e-6" iyy="1e-6"
-        izz="1e-6" ixy="1e-6"
-        ixz="1e-6" iyz="1e-6" />
-    </inertial>
-  </xacro:property>
   <!-- Covers -->
   <xacro:property name="base_cover_inertial">

File: urdf/dynaarm.urdf.xacro (robot description, xacro)
@@ -235,4 +235,24 @@
         <origin xyz="${joint_5_origin_xyz}" rpy="${joint_5_origin_rpy}" />
       </xacro:dynaarm_revolute_joint>
+      <!--dynaarm_WRIST_1_CAMERA_BASE-->
+      <link name="${link05_cam}">
+        <visual>
+          <origin rpy="0 0 0" xyz="0 0 0" />
+          <geometry>
+            <box size="0.001 0.001 0.001" />
+          </geometry>
+        </visual>
+        <inertial>
+          <origin rpy="0 0 0" xyz="0.0 0.0 0.0" />
+          <mass value="0.001" />
+          <inertia ixx="0.0000001" ixy="0.0" ixz="0.0" iyy="0.0000001" iyz="0.0" izz="0.0000001" />
+        </inertial>
+      </link>
+      <!-- Camera fixed on wrist1 -->
+      <xacro:dynaarm_joint_fixed joint_name="${joint_5_cam_name}"
+        parent="${link05}"
+        child="${link05_cam}">
+        <origin xyz="${joint_5_cam_origin_xyz}" rpy="${joint_5_cam_origin_rpy}" />
+      </xacro:dynaarm_joint_fixed>
       <!-- 5 Dof & Covers-->
       <xacro:if value="${covers}">
