Commit message: Added collision meshes and dae

File: urdf/common/dynaarm_parameters_v2.urdf.xacro (robot description, xacro)
@@ -39,27 +39,27 @@
   <!-- Meshes -->
   <xacro:if value="${covers}">
-    <xacro:property name="base_mesh" value="base_mesh.STL" />
+    <xacro:property name="base_mesh" value="base_mesh.dae" />
     <xacro:property name="link01_mesh" value="shoulder_mesh.dae" />
-    <xacro:property name="link02_mesh" value="upperarm_mesh.STL" />
-    <xacro:property name="link03_mesh" value="elbow_mesh.STL" />
-    <xacro:property name="link04_mesh" value="forearm_mesh.STL" />
-    <xacro:property name="link05_mesh" value="wrist1_mesh.STL" />
-    <xacro:property name="link06_mesh" value="wrist2_mesh.STL" />
-    <xacro:property name="base_cover_mesh" value="base_mesh.STL" />
+    <xacro:property name="link02_mesh" value="upperarm_mesh.dae" />
+    <xacro:property name="link03_mesh" value="elbow_mesh.dae" />
+    <xacro:property name="link04_mesh" value="forearm_mesh.dae" />
+    <xacro:property name="link05_mesh" value="wrist1_mesh.dae" />
+    <xacro:property name="link06_mesh" value="wrist2_mesh.dae" />
+    <xacro:property name="base_cover_mesh" value="base_mesh.dae" />
     <xacro:property name="link01_cover_mesh" value="shoulder_mesh.dae" />
-    <xacro:property name="link02_cover_mesh" value="upperarm_mesh.STL" />
-    <xacro:property name="link03_cover_mesh" value="elbow_mesh.STL" />
-    <xacro:property name="link04_cover_mesh" value="forearm_mesh.STL" />
-    <xacro:property name="link05_cover_mesh" value="wrist1_mesh.STL" />
-    <xacro:property name="link06_cover_mesh" value="wrist2_mesh.STL" />
+    <xacro:property name="link02_cover_mesh" value="upperarm_mesh.dae" />
+    <xacro:property name="link03_cover_mesh" value="elbow_mesh.dae" />
+    <xacro:property name="link04_cover_mesh" value="forearm_mesh.dae" />
+    <xacro:property name="link05_cover_mesh" value="wrist1_mesh.dae" />
+    <xacro:property name="link06_cover_mesh" value="wrist2_mesh.dae" />
   </xacro:if>
   <xacro:unless value="${covers}">
-    <xacro:property name="base_mesh" value="base_mesh.STL" />
+    <xacro:property name="base_mesh" value="base_mesh.dae" />
     <xacro:property name="link01_mesh" value="shoulder_mesh.dae" />
-    <xacro:property name="link02_mesh" value="upperarm_mesh.STL" />
-    <xacro:property name="link03_mesh" value="elbow_mesh.STL" />
-    <xacro:property name="link04_mesh" value="forearm_mesh.STL" />
-    <xacro:property name="link05_mesh" value="wrist1_mesh.STL" />
-    <xacro:property name="link06_mesh" value="wrist2_mesh.STL" />
+    <xacro:property name="link02_mesh" value="upperarm_mesh.dae" />
+    <xacro:property name="link03_mesh" value="elbow_mesh.dae" />
+    <xacro:property name="link04_mesh" value="forearm_mesh.dae" />
+    <xacro:property name="link05_mesh" value="wrist1_mesh.dae" />
+    <xacro:property name="link06_mesh" value="wrist2_mesh.dae" />
   </xacro:unless>
   <!-- Joint properties -->
@@ -268,5 +268,5 @@
       <geometry>
         <mesh
-          filename="package://dynaarm_description/meshes/collision_meshes/base_collision_mesh.STL"
+          filename="package://dynaarm_description/meshes/collision_meshes/base_collision_mesh.stl"
           scale="1 1 1" />
       </geometry>
@@ -275,7 +275,9 @@
   <xacro:property name="link01_collision">
     <collision>
-      <origin xyz="0 0 0.0105" rpy="0 0 0" />
-      <geometry>
-        <cylinder radius="0.05" length="0.24" />
+      <origin xyz="0 0 0" rpy="0 0 0" />
+      <geometry>
+        <mesh
+          filename="package://dynaarm_description/meshes/collision_meshes/shoulder_collision_mesh.stl"
+          scale="1 1 1" />
       </geometry>
     </collision>
@@ -283,7 +285,9 @@
   <xacro:property name="link02_collision">
     <collision>
-      <origin xyz="0 0 0.047" rpy="${J_PI/2} ${-J_PI/2} 0" />
-      <geometry>
-        <cylinder radius="0.05" length="0.4" />
+      <origin xyz="0 0 0" rpy="0 0 0" />
+      <geometry>
+        <mesh
+          filename="package://dynaarm_description/meshes/collision_meshes/upperarm_collision_mesh.stl"
+          scale="1 1 1" />
       </geometry>
     </collision>
@@ -291,7 +295,9 @@
   <xacro:property name="link03_collision">
     <collision>
-      <origin xyz="0.4127 0 0" rpy="${J_PI} 0 0" />
-      <geometry>
-        <cylinder radius="0.047" length="0.46" />
+      <origin xyz="0 0 0" rpy="0 0 0" />
+      <geometry>
+        <mesh
+          filename="package://dynaarm_description/meshes/collision_meshes/elbow_collision_mesh.stl"
+          scale="1 1 1" />
       </geometry>
     </collision>
@@ -299,7 +305,9 @@
   <xacro:property name="link04_collision">
     <collision>
-      <origin xyz="0.0262 -0.0855 0" rpy="${J_PI/2} 0 ${J_PI/2}" />
-      <geometry>
-        <cylinder radius="0.05" length="0.2" />
+      <origin xyz="0 0 0" rpy="0 0 0" />
+      <geometry>
+        <mesh
+          filename="package://dynaarm_description/meshes/collision_meshes/forearm_collision_mesh.stl"
+          scale="1 1 1" />
       </geometry>
     </collision>
@@ -307,7 +315,9 @@
   <xacro:property name="link05_collision">
     <collision>
-      <origin xyz="0.0295 0 0.4207" rpy="0 ${-J_PI/2} 0" />
-      <geometry>
-        <cylinder radius="0.055" length="0.18" />
+      <origin xyz="0 0 0" rpy="0 0 0" />
+      <geometry>
+        <mesh
+          filename="package://dynaarm_description/meshes/collision_meshes/wrist1_collision_mesh.stl"
+          scale="1 1 1" />
       </geometry>
     </collision>
@@ -315,7 +325,9 @@
   <xacro:property name="link06_collision">
     <collision>
-      <origin xyz="0.117 0.0 0.0295" rpy="${-J_PI/2} ${J_PI/2} ${-J_PI/2}" />
-      <geometry>
-        <cylinder radius="0.045" length="0.16" />
+      <origin xyz="0 0 0" rpy="0 0 0" />
+      <geometry>
+        <mesh
+          filename="package://dynaarm_description/meshes/collision_meshes/wrist2_collision_mesh.stl"
+          scale="1 1 1" />
       </geometry>
     </collision>

File: urdf/dynaarm.urdf.xacro (robot description, xacro)
@@ -196,9 +196,12 @@
     <xacro:if value="${dof >= 4}">
       <!-- dynaarm_FOREARM -->
-      <xacro:dynaarm_link link_name="${link04}" file_name="${link04_mesh}">
+      <xacro:dynaarm_link_w_collision link_name="${link04}" file_name="${link04_mesh}">
         <link_inertia>
           <xacro:insert_block name="link04_inertial" />
         </link_inertia>
-      </xacro:dynaarm_link>
+        <link_collision>
+          <xacro:insert_block name="link04_collision" />
+        </link_collision>
+      </xacro:dynaarm_link_w_collision>
       <!-- FA_ROT -->
       <xacro:dynaarm_revolute_joint joint_name="${joint_4_name}" parent="${link03}"
@@ -273,9 +276,12 @@
     <xacro:if value="${dof >= 6}">
       <!-- WRIST_2 -->
-      <xacro:dynaarm_link link_name="${link06}" file_name="${link06_mesh}">
+      <xacro:dynaarm_link_w_collision link_name="${link06}" file_name="${link06_mesh}">
         <link_inertia>
           <xacro:insert_block name="link06_inertial" />
         </link_inertia>
-      </xacro:dynaarm_link>
+        <link_collision>
+          <xacro:insert_block name="link06_collision" />
+        </link_collision>
+      </xacro:dynaarm_link_w_collision>
       <!-- WR_ROT -->
       <xacro:dynaarm_revolute_joint joint_name="${joint_6_name}" parent="${link05}"

Commit message: FIX!

File: urdf/common/dynaarm_parameters_v2.urdf.xacro (robot description, xacro)
@@ -87,5 +87,5 @@
   <xacro:property name="joint_3_axis_xyz" value="0 0 1" />
   <xacro:property name="joint_3_origin_xyz" value="0.4127 0 0" />
-  <xacro:property name="joint_3_origin_rpy" value="${J_PI} 0 0" />
+  <xacro:property name="joint_3_origin_rpy" value="0 0 0" />
   <xacro:property name="joint_3_lower_limit" value="-0.05" />
   <xacro:property name="joint_3_upper_limit" value="${J_PI}" />
