Commit message: trying to build a mergable version

File: urdf/common/dynaarm_parameters_v1.urdf.xacro (robot description, xacro)
@@ -82,5 +82,5 @@
   <xacro:property name="joint_4_lower_limit" value="${-J_PI - J_PI/2}" />
   <xacro:property name="joint_4_upper_limit" value="${J_PI + J_PI/2}" />
-  <xacro:property name="joint_5_name" value="${tf_prefix}WR_FLE" />
+  <xacro:property name="joint_5_name" value="${tf_prefix}WRIST_1" />
   <xacro:property name="joint_5_joint_type" value="revolute" />
   <xacro:property name="joint_5_axis_xyz" value="0 0 1" />
@@ -89,5 +89,5 @@
   <xacro:property name="joint_5_lower_limit" value="${-J_PI/2}" />
   <xacro:property name="joint_5_upper_limit" value="${J_PI/2}" />
-  <xacro:property name="joint_6_name" value="${tf_prefix}WR_ROT" />
+  <xacro:property name="joint_6_name" value="${tf_prefix}WRIST_2" />
   <xacro:property name="joint_6_joint_type" value="revolute" />
   <xacro:property name="joint_6_axis_xyz" value="0 0 1" />

File: urdf/common/dynaarm_parameters_v2.urdf.xacro (robot description, xacro)
@@ -18,6 +18,8 @@
   <xacro:property name="link02" value="${tf_prefix}UPPERARM" />
   <xacro:property name="link03" value="${tf_prefix}ELBOW" />
+  <xacro:property name="link03_cam" value="${tf_prefix}ELBOW_CAMERA_MOUNT" />
   <xacro:property name="link04" value="${tf_prefix}FOREARM" />
   <xacro:property name="link05" value="${tf_prefix}WRIST_1" />
+  <xacro:property name="link05_cam" value="${tf_prefix}WRIST_1_CAMERA_MOUNT" />
   <xacro:property name="link06" value="${tf_prefix}WRIST_2" />
   <xacro:property name="end_effector" value="${tf_prefix}END_EFFECTOR" />
@@ -25,5 +27,5 @@
   <xacro:if value="${covers}">
     <xacro:property name="base_mesh" value="base_mesh.STL" />
-    <xacro:property name="link01_mesh" value="shoulder_mesh.STL" />
+    <xacro:property name="link01_mesh" value="shoulderColor.dae" />
     <xacro:property name="link02_mesh" value="upperarm_mesh.STL" />
     <xacro:property name="link03_mesh" value="elbow_mesh.STL" />
@@ -31,15 +33,15 @@
     <xacro:property name="link05_mesh" value="wrist1_mesh.STL" />
     <xacro:property name="link06_mesh" value="wrist2_mesh.STL" />
-    <xacro:property name="base_cover_mesh" value="base_cover_mesh.STL" />
-    <xacro:property name="link01_cover_mesh" value="shoulder_cover_mesh.STL" />
-    <xacro:property name="link02_cover_mesh" value="upperarm_cover_mesh.STL" />
-    <xacro:property name="link03_cover_mesh" value="elbow_cover_mesh.STL" />
-    <xacro:property name="link04_cover_mesh" value="forearm_cover_mesh.STL" />
-    <xacro:property name="link05_cover_mesh" value="wrist_1_cover_mesh.STL" />
-    <xacro:property name="link06_cover_mesh" value="wrist_2_cover_mesh.STL" />
+    <xacro:property name="base_cover_mesh" value="base_mesh.STL" />
+    <xacro:property name="link01_cover_mesh" value="shoulderColor.dae" />
+    <xacro:property name="link02_cover_mesh" value="upperarm_mesh.STL" />
+    <xacro:property name="link03_cover_mesh" value="elbow_mesh.STL" />
+    <xacro:property name="link04_cover_mesh" value="forearm_mesh.STL" />
+    <xacro:property name="link05_cover_mesh" value="wrist1_mesh.STL" />
+    <xacro:property name="link06_cover_mesh" value="wrist2_mesh.STL" />
   </xacro:if>
   <xacro:unless value="${covers}">
     <xacro:property name="base_mesh" value="base_mesh.STL" />
-    <xacro:property name="link01_mesh" value="shoulder_mesh.STL" />
+    <xacro:property name="link01_mesh" value="shoulderColor.dae" />
     <xacro:property name="link02_mesh" value="upperarm_mesh.STL" />
     <xacro:property name="link03_mesh" value="elbow_mesh.STL" />
@@ -57,5 +59,5 @@
   <xacro:property name="joint_1_joint_type" value="revolute" />
   <xacro:property name="joint_1_axis_xyz" value="0 0 1" />
-  <xacro:property name="joint_1_origin_xyz" value="0 0 0.06" />
+  <xacro:property name="joint_1_origin_xyz" value="0 0 0.0105" />
   <xacro:property name="joint_1_origin_rpy" value="0 0 0" />
   <xacro:property name="joint_1_lower_limit" value="${-J_PI - J_PI/2}" />
@@ -63,6 +65,6 @@
   <xacro:property name="joint_2_name" value="${tf_prefix}SH_FLE" />
   <xacro:property name="joint_2_joint_type" value="revolute" />
-  <xacro:property name="joint_2_axis_xyz" value="0 0 -1" />
-  <xacro:property name="joint_2_origin_xyz" value="0 0 0.0" />
+  <xacro:property name="joint_2_axis_xyz" value="0 0 1" />
+  <xacro:property name="joint_2_origin_xyz" value="0 0 0.047" />
   <xacro:property name="joint_2_origin_rpy" value="${J_PI/2} ${-J_PI/2} 0" />
   <xacro:property name="joint_2_lower_limit" value="${-J_PI/2 - 0.3}" />
@@ -71,27 +73,37 @@
   <xacro:property name="joint_3_joint_type" value="revolute" />
   <xacro:property name="joint_3_axis_xyz" value="0 0 1" />
-  <xacro:property name="joint_3_origin_xyz" value="0.412 0 0" />
+  <xacro:property name="joint_3_origin_xyz" value="0.4127 0 0" />
   <xacro:property name="joint_3_origin_rpy" value="${J_PI} 0 0" />
   <xacro:property name="joint_3_lower_limit" value="-0.05" />
   <xacro:property name="joint_3_upper_limit" value="${J_PI}" />
+  <xacro:property name="joint_3_cam_name" value="${tf_prefix}EL_CAMERA" />
+  <xacro:property name="joint_3_cam_joint_type" value="fixed" />
+  <xacro:property name="joint_3_cam_axis_xyz" value="0 0 0" />
+  <xacro:property name="joint_3_cam_origin_xyz" value="0.0345 -0.1235 0" />
+  <xacro:property name="joint_3_cam_origin_rpy" value="0.0 0.0 0.0" />
   <xacro:property name="joint_4_name" value="${tf_prefix}FA_ROT" />
   <xacro:property name="joint_4_joint_type" value="revolute" />
   <xacro:property name="joint_4_axis_xyz" value="0 0 1" />
-  <xacro:property name="joint_4_origin_xyz" value="0.0325 -0.092 0" />
+  <xacro:property name="joint_4_origin_xyz" value="0.0262 -0.0855 0" />
   <xacro:property name="joint_4_origin_rpy" value="${J_PI/2} 0 ${J_PI/2}" />
   <xacro:property name="joint_4_lower_limit" value="${-J_PI - J_PI/2}" />
   <xacro:property name="joint_4_upper_limit" value="${J_PI + J_PI/2}" />
-  <xacro:property name="joint_5_name" value="${tf_prefix}WR_FLE" />
+  <xacro:property name="joint_5_name" value="${tf_prefix}WRIST_1" />
   <xacro:property name="joint_5_joint_type" value="revolute" />
   <xacro:property name="joint_5_axis_xyz" value="0 0 1" />
-  <xacro:property name="joint_5_origin_xyz" value="0.0 -0.03 0.4118" />
-  <xacro:property name="joint_5_origin_rpy" value="0 ${-J_PI/2} ${-J_PI/2}" />
+  <xacro:property name="joint_5_origin_xyz" value="0.0295 0 0.4207" />
+  <xacro:property name="joint_5_origin_rpy" value="0 ${-J_PI/2} 0" />
   <xacro:property name="joint_5_lower_limit" value="${-J_PI/2}" />
   <xacro:property name="joint_5_upper_limit" value="${J_PI/2}" />
-  <xacro:property name="joint_6_name" value="${tf_prefix}WR_ROT" />
+  <xacro:property name="joint_5_cam_name" value="${tf_prefix}WRIST_1_CAMERA" />
+  <xacro:property name="joint_5_cam_joint_type" value="fixed" />
+  <xacro:property name="joint_5_cam_axis_xyz" value="0 0 0" />
+  <xacro:property name="joint_5_cam_origin_xyz" value="0.032 0 -0.017" />
+  <xacro:property name="joint_5_cam_origin_rpy" value="0.0 0.0 0.0" />
+  <xacro:property name="joint_6_name" value="${tf_prefix}WRIST_2" />
   <xacro:property name="joint_6_joint_type" value="revolute" />
   <xacro:property name="joint_6_axis_xyz" value="0 0 1" />
-  <xacro:property name="joint_6_origin_xyz" value="0.12 0.0 0.03" />
-  <xacro:property name="joint_6_origin_rpy" value="${-J_PI/2} 0 ${-J_PI/2}" />
+  <xacro:property name="joint_6_origin_xyz" value="0.117 0.0 0.0295" />
+  <xacro:property name="joint_6_origin_rpy" value="${-J_PI/2} ${J_PI/2} ${-J_PI/2}" />
   <xacro:property name="joint_6_lower_limit" value="${-J_PI - J_PI/2}" />
   <xacro:property name="joint_6_upper_limit" value="${J_PI + J_PI/2}" />
@@ -106,49 +118,84 @@
   <xacro:property name="base_inertial">
     <inertial>
-      <mass value=" 2.00264891"/>
-      <origin rpy="0 0 0" xyz="0.00346973 0.00328767  -0.04882463"/>
-      <inertia ixx="0.00403356" ixy="0.00040829" ixz="-0.00018772" iyy="0.00417547" iyz="-0.00018208" izz="0.00460221"/>
+      <mass value="2.00205474" />
+      <origin
+        xyz="0.00347077 0.00328869 -0.0488212"
+        rpy="0 0 0" />
+      <inertia ixx="0.00403342" iyy="0.00417534"
+        izz="0.00460211" ixy="0.00040828"
+        ixz="-0.00018775" iyz="-0.0001821" />
     </inertial>
   </xacro:property>
   <xacro:property name="link01_inertial">
     <inertial>
-      <mass value="2.73096676"/>
-      <origin rpy="0 0 0" xyz="0.00001348 0.00013521 0.04302590"/>
-      <inertia ixx="0.01291668" ixy="0.00000440" ixz=" -0.00000179" iyy="0.00368667" iyz="-0.00001792" izz=" 0.01243431"/>
+      <mass value="2.73096676" />
+      <origin xyz="0.00001348 0.00013521 0.0430259" rpy="0 0 0" />
+      <inertia ixx="0.01291668" iyy="0.00874231"
+        izz="0.01243436" ixy="0.0000044"
+        ixz="-0.00000179" iyz="-0.00000203" />
     </inertial>
   </xacro:property>
   <xacro:property name="link02_inertial">
     <inertial>
-      <mass value="1.394"/>
-      <origin rpy="0 0 0" xyz="0.21109 2.2e-05 -0.000317"/>
-      <inertia ixx="0.00116179" ixy="-7.2e-07" ixz="-0.00014044999999999997" iyy="0.046092126" iyz="7e-09" izz="0.04627953"/>
+      <mass value="1.72040464" />
+      <origin xyz="0.20391301 -0.00000528 -0.00015224"
+        rpy="0 0 0" />
+      <inertia ixx="0.00155499" iyy="0.05067934"
+        izz="0.0507131" ixy="0.00000098"
+        ixz="0.00004108" iyz="-0.00000143" />
     </inertial>
   </xacro:property>
   <xacro:property name="link03_inertial">
     <inertial>
-      <mass value="1.1"/>
-      <origin rpy="0 0 0" xyz="0.0068 -0.0848 -0.0006"/>
-      <inertia ixx="0.0013843" ixy="-4.16e-05" ixz="8.5e-06" iyy="0.0007168" iyz="-1.05e-05" izz="0.0011300999999999998"/>
+      <mass value="0.82320237" />
+      <origin xyz="0.00383866 -0.07802638 -0.00026928" rpy="0 0 0" />
+      <inertia ixx="0.00107419" iyy="0.00087121"
+        izz="0.00113856" ixy="0.00004166"
+        ixz="-0.00000398" iyz="-0.0000119" />
+    </inertial>
+  </xacro:property>
+  <xacro:property name="link03_cam_inertial">
+    <inertial>
+      <mass value="1e-6" />
+      <origin xyz="0.0 0.0 0.0" rpy="0 0 0" />
+      <inertia ixx="1e-6" iyy="1e-6"
+        izz="1e-6" ixy="1e-6"
+        ixz="1e-6" iyz="1e-6" />
     </inertial>
   </xacro:property>
   <xacro:property name="link04_inertial">
     <inertial>
-      <mass value="0.342"/>
-      <origin rpy="0 0 0" xyz="0.0 0.0 0.2143"/>
-      <inertia ixx="0.006999999999999999" ixy="0.0" ixz="0.0" iyy="0.006999999999999999" iyz="0.0" izz="0.0063999999999999994"/>
+      <mass value="1.15674546" />
+      <origin xyz="-0.00115165 0.00001056 0.30067314" rpy="0 0 0" />
+      <inertia ixx="0.03129519" iyy="0.03125954"
+        izz="0.00090392" ixy="0.00000151"
+        ixz="-0.00017171" iyz="0.00000159" />
     </inertial>
   </xacro:property>
   <xacro:property name="link05_inertial">
     <inertial>
-      <mass value="1.69"/>
-      <origin rpy="0 0 0" xyz="0.047 0.0 0.029"/>
-      <inertia ixx="0.0016719999999999999" ixy="0.0" ixz="0.00012969999999999998" iyy="0.004985" iyz="-3.7e-06" izz="0.005209999999999999"/>
+      <mass value="0.75007482" />
+      <origin xyz="0.07972553 -0.00005038 0.02334747" rpy="0 0 0" />
+      <inertia ixx="0.00065953" iyy="0.00088282"
+        izz="0.00078106" ixy="0.00000076"
+        ixz="0.00011795" iyz="-0.00000079" />
+    </inertial>
+  </xacro:property>
+  <xacro:property name="link05_cam_inertial">
+    <inertial>
+      <mass value="1e-6" />
+      <origin xyz="0.0 0.0 0.0" rpy="0 0 0" />
+      <inertia ixx="1e-6" iyy="1e-6"
+        izz="1e-6" ixy="1e-6"
+        ixz="1e-6" iyz="1e-6" />
     </inertial>
   </xacro:property>
   <xacro:property name="link06_inertial">
     <inertial>
-      <mass value="0.1"/>
-      <origin rpy="0 0 0" xyz="0.0 0.0 0.0064"/>
-      <inertia ixx="0.00011499999999999999" ixy="0.0" ixz="0.0" iyy="0.00011499999999999999" iyz="0.0" izz="0.00011499999999999999"/>
+      <mass value="0.0478406" />
+      <origin xyz="0.00045711 0.00000557 0.00344945" rpy="0 0 0" />
+      <inertia ixx="0.00001366" iyy="0.00001419"
+        izz="0.00002702" ixy="0"
+        ixz="0.00000008" iyz="0" />
     </inertial>
   </xacro:property>
@@ -205,7 +252,9 @@
   <xacro:property name="base_collision">
     <collision>
-      <origin xyz="0 0 -0.04" rpy="0 0 0" />
-      <geometry>
-        <cylinder radius="0.06" length="0.08" />
+      <origin xyz="0 0 0" rpy="0 0 0" />
+      <geometry>
+        <mesh
+          filename="package://dynaarm_description/meshes/collision_meshes/base_collision_mesh.STL"
+          scale="1 1 1" />
       </geometry>
     </collision>
@@ -213,5 +262,5 @@
   <xacro:property name="link01_collision">
     <collision>
-      <origin xyz="0 0 0" rpy="1.57 0 0" />
+      <origin xyz="0 0 0.0105" rpy="0 0 0" />
       <geometry>
         <cylinder radius="0.05" length="0.24" />
@@ -221,5 +270,5 @@
   <xacro:property name="link02_collision">
     <collision>
-      <origin xyz="0.25 0 0" rpy="1.57 0 1.57" />
+      <origin xyz="0 0 0.047" rpy="${J_PI/2} ${-J_PI/2} 0" />
       <geometry>
         <cylinder radius="0.05" length="0.4" />
@@ -229,5 +278,5 @@
   <xacro:property name="link03_collision">
     <collision>
-      <origin xyz="0.185 -0.0935 0" rpy="0 1.57 0" />
+      <origin xyz="0.4127 0 0" rpy="${J_PI} 0 0" />
       <geometry>
         <cylinder radius="0.047" length="0.46" />
@@ -235,9 +284,25 @@
     </collision>
   </xacro:property>
+  <xacro:property name="link04_collision">
+    <collision>
+      <origin xyz="0.0262 -0.0855 0" rpy="${J_PI/2} 0 ${J_PI/2}" />
+      <geometry>
+        <cylinder radius="0.05" length="0.2" />
+      </geometry>
+    </collision>
+  </xacro:property>
   <xacro:property name="link05_collision">
     <collision>
-      <origin xyz="${0.045} 0 0.03" rpy="0 ${J_PI/2} 0" />
+      <origin xyz="0.0295 0 0.4207" rpy="0 ${-J_PI/2} 0" />
       <geometry>
         <cylinder radius="0.055" length="0.18" />
+      </geometry>
+    </collision>
+  </xacro:property>
+  <xacro:property name="link06_collision">
+    <collision>
+      <origin xyz="0.117 0.0 0.0295" rpy="${-J_PI/2} ${J_PI/2} ${-J_PI/2}" />
+      <geometry>
+        <cylinder radius="0.045" length="0.16" />
       </geometry>
     </collision>

File: urdf/dynaarm.urdf.xacro (robot description, xacro)
@@ -17,5 +17,6 @@
     <xacro:property name="ee_parent" value="${base}" />
     <xacro:include filename="$(find dynaarm_description)/urdf/common/dynaarm_common.urdf.xacro" />
-    <xacro:include filename="$(find dynaarm_description)/urdf/common/dynaarm_parameters_${version}.urdf.xacro" />
+    <xacro:include
+      filename="$(find dynaarm_description)/urdf/common/dynaarm_parameters_${version}.urdf.xacro" />
     <xacro:include filename="$(find dynaarm_description)/urdf/common/dynaarm.ros2control.xacro" />
     <xacro:dynaarm_joint_fixed joint_name="${joint_base_name}"
@@ -155,4 +156,24 @@
         <origin xyz="${joint_3_origin_xyz}" rpy="${joint_3_origin_rpy}" />
       </xacro:dynaarm_revolute_joint>
+      <!--dynaarm_ELBOW_CAMERA_BASE-->
+      <link name="${link03_cam}">
+        <visual>
+          <origin rpy="0 0 0" xyz="0 0 0" />
+          <geometry>
+            <box size="0.001 0.001 0.001" />
+          </geometry>
+        </visual>
+        <inertial>
+          <origin rpy="0 0 0" xyz="0.0 0.0 0.0" />
+          <mass value="0.001" />
+          <inertia ixx="0.0000001" ixy="0.0" ixz="0.0" iyy="0.0000001" iyz="0.0" izz="0.0000001" />
+        </inertial>
+      </link>
+      <!-- Camera fixed on elbow -->
+      <xacro:dynaarm_joint_fixed joint_name="${joint_3_cam_name}"
+        parent="${link03}"
+        child="${link03_cam}">
+        <origin xyz="${joint_3_cam_origin_xyz}" rpy="${joint_3_cam_origin_rpy}" />
+      </xacro:dynaarm_joint_fixed>
       <!-- 3 Dof & Covers-->
       <xacro:if value="${covers}">
@@ -222,4 +243,24 @@
         <origin xyz="${joint_5_origin_xyz}" rpy="${joint_5_origin_rpy}" />
       </xacro:dynaarm_revolute_joint>
+      <!--dynaarm_WRIST_1_CAMERA_BASE-->
+      <link name="${link05_cam}">
+        <visual>
+          <origin rpy="0 0 0" xyz="0 0 0" />
+          <geometry>
+            <box size="0.001 0.001 0.001" />
+          </geometry>
+        </visual>
+        <inertial>
+          <origin rpy="0 0 0" xyz="0.0 0.0 0.0" />
+          <mass value="0.001" />
+          <inertia ixx="0.0000001" ixy="0.0" ixz="0.0" iyy="0.0000001" iyz="0.0" izz="0.0000001" />
+        </inertial>
+      </link>
+      <!-- Camera fixed on wrist1 -->
+      <xacro:dynaarm_joint_fixed joint_name="${joint_5_cam_name}"
+        parent="${link05}"
+        child="${link05_cam}">
+        <origin xyz="${joint_5_cam_origin_xyz}" rpy="${joint_5_cam_origin_rpy}" />
+      </xacro:dynaarm_joint_fixed>
       <!-- 5 Dof & Covers-->
       <xacro:if value="${covers}">
@@ -274,5 +315,5 @@
       <plugin filename="libgz_ros2_control-system.so"
         name="gz_ros2_control::GazeboSimROS2ControlPlugin">
-        <parameters>$(find dynaarm_examples)/config/controllers.yaml</parameters>
+        <parameters>$(find dynaarm_driver)/config/controllers.yaml</parameters>
         <robotNamespace>dynaarm</robotNamespace>
         <robotDescription>dynaarm_description</robotDescription>

Commit message: rename and reposition endeffector joint

File: urdf/common/dynaarm_parameters_v1.urdf.xacro (robot description, xacro)
@@ -110,7 +110,7 @@
   <xacro:property name="joint_6_upper_limit" value="${J_PI + J_PI/2}" />
   <xacro:property name="joint_ee_name" value="${tf_prefix}flange_fix_joint" />
-  <xacro:property name="joint_ee_xyz" value="0.0 0.0 0.05" />
-  <xacro:property name="joint_ee_origin_xyz" value="0.0 0.0 0.05" />
-  <xacro:property name="joint_ee_origin_4dof_xyz" value="0.0 0.0 0.4" />
+  <xacro:property name="joint_ee_xyz" value="0.0 0.0 0.009" />
+  <xacro:property name="joint_ee_origin_xyz" value="0.0 0.0 0.009" />
+  <xacro:property name="joint_ee_origin_4dof_xyz" value="0.0 0.0 0.009" />
   <xacro:property name="joint_ee_origin_rpy" value="0.0 0.0 ${J_PI/2}" />
   <xacro:property name="joint_ee_origin_4dof_rpy" value="0.0 0.0 ${J_PI/2}" />

File: urdf/common/dynaarm_parameters_v2.urdf.xacro (robot description, xacro)
@@ -122,7 +122,7 @@
   <xacro:property name="joint_6_upper_limit" value="${J_PI + J_PI/2}" />
   <xacro:property name="joint_ee_name" value="${tf_prefix}flange_fix_joint" />
-  <xacro:property name="joint_ee_xyz" value="0.0 0.0 0.05" />
-  <xacro:property name="joint_ee_origin_xyz" value="0.0 0.0 0.05" />
-  <xacro:property name="joint_ee_origin_4dof_xyz" value="0.0 0.0 0.4" />
+  <xacro:property name="joint_ee_xyz" value="0.0 0.0 0.009" />
+  <xacro:property name="joint_ee_origin_xyz" value="0.0 0.0 0.009" />
+  <xacro:property name="joint_ee_origin_4dof_xyz" value="0.0 0.0 0.009" />
   <xacro:property name="joint_ee_origin_rpy" value="0.0 0.0 ${J_PI/2}" />
   <xacro:property name="joint_ee_origin_4dof_rpy" value="0.0 0.0 ${J_PI/2}" />
