Commit message: added final new line

File: urdf/common/dynaarm_common.urdf.xacro (robot description, xacro)
@@ -2,9 +2,22 @@
 <!--
 Copyright 2024 Duatic AG
-Redistribution and use in source and binary forms, with or without modification, are permitted provided that the following conditions are met:
-1. Redistributions of source code must retain the above copyright notice, this list of conditions and the following disclaimer.
-2. Redistributions in binary form must reproduce the above copyright notice, this list of conditions and the following disclaimer in the documentation and/or other materials provided with the distribution.
-3. Neither the name of the copyright holder nor the names of its contributors may be used to endorse or promote products derived from this software without specific prior written permission.
-THIS SOFTWARE IS PROVIDED BY THE COPYRIGHT HOLDERS AND CONTRIBUTORS “AS IS” AND ANY EXPRESS OR IMPLIED WARRANTIES, INCLUDING, BUT NOT LIMITED TO, THE IMPLIED WARRANTIES OF MERCHANTABILITY AND FITNESS FOR A PARTICULAR PURPOSE ARE DISCLAIMED. IN NO EVENT SHALL THE COPYRIGHT HOLDER OR CONTRIBUTORS BE LIABLE FOR ANY DIRECT, INDIRECT, INCIDENTAL, SPECIAL, EXEMPLARY, OR CONSEQUENTIAL DAMAGES (INCLUDING, BUT NOT LIMITED TO, PROCUREMENT OF SUBSTITUTE GOODS OR SERVICES; LOSS OF USE, DATA, OR PROFITS; OR BUSINESS INTERRUPTION) HOWEVER CAUSED AND ON ANY THEORY OF LIABILITY, WHETHER IN CONTRACT, STRICT LIABILITY, OR TORT (INCLUDING NEGLIGENCE OR OTHERWISE) ARISING IN ANY WAY OUT OF THE USE OF THIS SOFTWARE, EVEN IF ADVISED OF THE POSSIBILITY OF SUCH DAMAGE.
+Redistribution and use in source and binary forms, with or without modification, are permitted
+provided that the following conditions are met:
+1. Redistributions of source code must retain the above copyright notice, this list of conditions
+and the following disclaimer.
+2. Redistributions in binary form must reproduce the above copyright notice, this list of
+conditions and the following disclaimer in the documentation and/or other materials provided with
+the distribution.
+3. Neither the name of the copyright holder nor the names of its contributors may be used to
+endorse or promote products derived from this software without specific prior written permission.
+THIS SOFTWARE IS PROVIDED BY THE COPYRIGHT HOLDERS AND CONTRIBUTORS “AS IS” AND ANY EXPRESS OR
+IMPLIED WARRANTIES, INCLUDING, BUT NOT LIMITED TO, THE IMPLIED WARRANTIES OF MERCHANTABILITY AND
+FITNESS FOR A PARTICULAR PURPOSE ARE DISCLAIMED. IN NO EVENT SHALL THE COPYRIGHT HOLDER OR
+CONTRIBUTORS BE LIABLE FOR ANY DIRECT, INDIRECT, INCIDENTAL, SPECIAL, EXEMPLARY, OR CONSEQUENTIAL
+DAMAGES (INCLUDING, BUT NOT LIMITED TO, PROCUREMENT OF SUBSTITUTE GOODS OR SERVICES; LOSS OF USE,
+DATA, OR PROFITS; OR BUSINESS INTERRUPTION) HOWEVER CAUSED AND ON ANY THEORY OF LIABILITY, WHETHER
+IN CONTRACT, STRICT LIABILITY, OR TORT (INCLUDING NEGLIGENCE OR OTHERWISE) ARISING IN ANY WAY OUT
+OF
+THE USE OF THIS SOFTWARE, EVEN IF ADVISED OF THE POSSIBILITY OF SUCH DAMAGE.
 -->
 <robot xmlns:xacro="http://www.ros.org/wiki/xacro">
@@ -12,5 +25,6 @@
     <!-- DynaArm Base Link Macro -->
     <!-- -->
-    <xacro:macro name="dynaarm_baselink" params="link_name file_name **base_inertia **base_collision">
+    <xacro:macro name="dynaarm_baselink"
+        params="link_name file_name **base_inertia **base_collision">
         <link name="${link_name}">
             <visual>

File: urdf/common/dynaarm_parameters_v1.urdf.xacro (robot description, xacro)
@@ -1,9 +1,22 @@
 <!--
 Copyright 2024 Duatic AG
-Redistribution and use in source and binary forms, with or without modification, are permitted provided that the following conditions are met:
-1. Redistributions of source code must retain the above copyright notice, this list of conditions and the following disclaimer.
-2. Redistributions in binary form must reproduce the above copyright notice, this list of conditions and the following disclaimer in the documentation and/or other materials provided with the distribution.
-3. Neither the name of the copyright holder nor the names of its contributors may be used to endorse or promote products derived from this software without specific prior written permission.
-THIS SOFTWARE IS PROVIDED BY THE COPYRIGHT HOLDERS AND CONTRIBUTORS “AS IS” AND ANY EXPRESS OR IMPLIED WARRANTIES, INCLUDING, BUT NOT LIMITED TO, THE IMPLIED WARRANTIES OF MERCHANTABILITY AND FITNESS FOR A PARTICULAR PURPOSE ARE DISCLAIMED. IN NO EVENT SHALL THE COPYRIGHT HOLDER OR CONTRIBUTORS BE LIABLE FOR ANY DIRECT, INDIRECT, INCIDENTAL, SPECIAL, EXEMPLARY, OR CONSEQUENTIAL DAMAGES (INCLUDING, BUT NOT LIMITED TO, PROCUREMENT OF SUBSTITUTE GOODS OR SERVICES; LOSS OF USE, DATA, OR PROFITS; OR BUSINESS INTERRUPTION) HOWEVER CAUSED AND ON ANY THEORY OF LIABILITY, WHETHER IN CONTRACT, STRICT LIABILITY, OR TORT (INCLUDING NEGLIGENCE OR OTHERWISE) ARISING IN ANY WAY OUT OF THE USE OF THIS SOFTWARE, EVEN IF ADVISED OF THE POSSIBILITY OF SUCH DAMAGE.
+Redistribution and use in source and binary forms, with or without modification, are permitted
+provided that the following conditions are met:
+1. Redistributions of source code must retain the above copyright notice, this list of conditions
+and the following disclaimer.
+2. Redistributions in binary form must reproduce the above copyright notice, this list of
+conditions and the following disclaimer in the documentation and/or other materials provided with
+the distribution.
+3. Neither the name of the copyright holder nor the names of its contributors may be used to
+endorse or promote products derived from this software without specific prior written permission.
+THIS SOFTWARE IS PROVIDED BY THE COPYRIGHT HOLDERS AND CONTRIBUTORS “AS IS” AND ANY EXPRESS OR
+IMPLIED WARRANTIES, INCLUDING, BUT NOT LIMITED TO, THE IMPLIED WARRANTIES OF MERCHANTABILITY AND
+FITNESS FOR A PARTICULAR PURPOSE ARE DISCLAIMED. IN NO EVENT SHALL THE COPYRIGHT HOLDER OR
+CONTRIBUTORS BE LIABLE FOR ANY DIRECT, INDIRECT, INCIDENTAL, SPECIAL, EXEMPLARY, OR CONSEQUENTIAL
+DAMAGES (INCLUDING, BUT NOT LIMITED TO, PROCUREMENT OF SUBSTITUTE GOODS OR SERVICES; LOSS OF USE,
+DATA, OR PROFITS; OR BUSINESS INTERRUPTION) HOWEVER CAUSED AND ON ANY THEORY OF LIABILITY, WHETHER
+IN CONTRACT, STRICT LIABILITY, OR TORT (INCLUDING NEGLIGENCE OR OTHERWISE) ARISING IN ANY WAY OUT
+OF
+THE USE OF THIS SOFTWARE, EVEN IF ADVISED OF THE POSSIBILITY OF SUCH DAMAGE.
 -->
 <robot xmlns:xacro="http://www.ros.org/wiki/xacro">

Commit message: Fixing some inertias

File: urdf/common/dynaarm_common.urdf.xacro (robot description, xacro)
@@ -78,18 +78,23 @@
     <!-- DynaArm Virtual Link Macro -->
     <!-- -->
-    <xacro:macro name="virtual_link" params="link_name">
+    <xacro:macro name="virtual_link" params="link_name mass:=0.001 ixx:=0.0000001 iyy:=0.0000001 izz:=0.0000001">
         <link name="${link_name}">
             <visual>
                 <origin xyz="0 0 0" rpy="0 0 0" />
                 <geometry>
-                    <box size="0.001 0.001 0.001" />
+                    <box size="0.01 0.01 0.01" />
                 </geometry>
             </visual>
             <inertial>
                 <origin xyz="0.0 0.0 0.0" rpy="0 0 0" />
-                <mass value="0.001" />
-                <inertia ixx="0.0000001" ixy="0.0" iyy="0.0000001" ixz="0.0" iyz="0.0"
-                    izz="0.0000001" />
+                <mass value="${mass}" />
+                <inertia ixx="${ixx}" ixy="0.0" iyy="${iyy}" ixz="0.0" iyz="0.0" izz="${izz}" />
             </inertial>
+            <collision>
+                <origin xyz="0 0 0" rpy="0 0 0" />
+                <geometry>
+                    <box size="0.01 0.01 0.01" />
+                </geometry>
+            </collision>
         </link>
         <!-- Gazebo customization -->

File: urdf/dynaarm.urdf.xacro (robot description, xacro)
@@ -330,10 +330,20 @@
   <!-- -->
   <xacro:macro name="dynaarm_tool">
-    <xacro:virtual_link link_name="${end_effector}" />
-    <xacro:dynaarm_joint_fixed joint_name="${joint_ee_name}"
-      parent="${ee_parent}"
-      child="${end_effector}">
-      <origin xyz="${joint_ee_origin_xyz}" rpy="${joint_ee_origin_rpy}" />
-    </xacro:dynaarm_joint_fixed>
+      <xacro:virtual_link link_name="${end_effector}" />
+      <xacro:dynaarm_joint_fixed joint_name="${joint_ee_name}"
+          parent="${ee_parent}"
+          child="${end_effector}">
+          <origin xyz="${joint_ee_origin_xyz}" rpy="${joint_ee_origin_rpy}" />
+      </xacro:dynaarm_joint_fixed>
+      <!-- Add x_kg weight to flange -->
+      <!-- <xacro:virtual_link link_name="${end_effector}_weight"
+          mass="0.2"
+          ixx="0.036" iyy="0.036" izz="0.002">
+      </xacro:virtual_link>
+      <xacro:dynaarm_joint_fixed joint_name="${end_effector}_weight_joint"
+          parent="${end_effector}"
+          child="${end_effector}_weight">
+          <origin xyz="0.0 0.0 0.02" rpy="0 0 0" />
+      </xacro:dynaarm_joint_fixed> -->
   </xacro:macro>
   <!-- -->
