Commit message: Added the version arg to the view.launc file. Completely restructured the urdf stuff to dynamically be able to switch between 1-6 DoF and the versions without the need for multiple files.

File: urdf/common/dynaarm.ros2control.xacro (robot description, xacro)
@@ -43,12 +43,22 @@
         </xacro:if>
       </hardware>
-      <xacro:dynaarm_ros2control_joint name="${tf_prefix}SH_ROT" address="1" />
-      <xacro:dynaarm_ros2control_joint name="${tf_prefix}SH_FLE" address="2" />
-      <!-- <xacro:dynaarm_ros2control_joint name="${tf_prefix}EL_FLE" address="3" />
-      <xacro:dynaarm_ros2control_joint name="${tf_prefix}FA_ROT" address="4" />
-      <xacro:if value="${dof == '6dof'}">
+      <xacro:if value="${dof >= 1}">
+        <xacro:dynaarm_ros2control_joint name="${tf_prefix}SH_ROT" address="1" />
+      </xacro:if>
+      <xacro:if value="${dof >= 2}">
+        <xacro:dynaarm_ros2control_joint name="${tf_prefix}SH_FLE" address="2" />
+      </xacro:if>
+      <xacro:if value="${dof >= 3}">
+        <xacro:dynaarm_ros2control_joint name="${tf_prefix}EL_FLE" address="3" />
+      </xacro:if>
+      <xacro:if value="${dof >= 4}">
+        <xacro:dynaarm_ros2control_joint name="${tf_prefix}FA_ROT" address="4" />
+      </xacro:if>
+      <xacro:if value="${dof >= 5}">
         <xacro:dynaarm_ros2control_joint name="${tf_prefix}WRIST_1" address="5" />
+      </xacro:if>
+      <xacro:if value="${dof >= 6}">
         <xacro:dynaarm_ros2control_joint name="${tf_prefix}WRIST_2" address="6" />
-      </xacro:if> -->
+      </xacro:if>
     </ros2_control>
   </xacro:macro>

File: urdf/common/dynaarm_common.urdf.xacro (robot description, xacro)
@@ -4,16 +4,15 @@
     <!-- DynaArm Base Link Macro -->
     <!-- -->
-    <xacro:macro name="dynaarm_baselink"
-        params="link_name file_name **base_inertia  **base_collision">
+    <xacro:macro name="dynaarm_baselink" params="link_name file_name **base_inertia **base_collision">
         <link name="${link_name}">
             <visual>
                 <geometry>
                     <mesh
-                        filename="file://$(find dynaarm_description)/meshes/${version}/${file_name}.dae"
+                        filename="file://$(find dynaarm_description)/meshes/${version}/${file_name}"
                         scale="1.0 1.0 1.0" />
                 </geometry>
                 <material name="carbon_fiber">
-					<color rgba="0.792156862745098 0.819607843137255 0.933333333333333 1" />
-				</material>
+                    <color rgba="0.792156862745098 0.819607843137255 0.933333333333333 1" />
+                </material>
             </visual>
             <xacro:insert_block name="base_collision" />
@@ -25,10 +24,10 @@
     <!-- -->
     <xacro:macro name="dynaarm_link"
-        params="link_name file_name **link_inertia ">
+        params="link_name file_name **link_inertia">
         <link name="${link_name}">
             <visual>
                 <geometry>
                     <mesh
-                        filename="file://$(find dynaarm_description)/meshes/${version}/${file_name}.dae"
+                        filename="file://$(find dynaarm_description)/meshes/${version}/${file_name}"
                         scale="1.0 1.0 1.0" />
                 </geometry>
@@ -41,10 +40,10 @@
     <!-- -->
     <xacro:macro name="dynaarm_link_w_collision"
-        params="link_name file_name **link_inertia **link_collision ">
+        params="link_name file_name **link_inertia **link_collision">
         <link name="${link_name}">
             <visual>
                 <geometry>
                     <mesh
-                        filename="file://$(find dynaarm_description)/meshes/${version}/${file_name}.dae"
+                        filename="file://$(find dynaarm_description)/meshes/${version}/${file_name}"
                         scale="1.0 1.0 1.0" />
                 </geometry>
@@ -88,5 +87,14 @@
     <!-- -->
     <xacro:macro name="dynaarm_revolute_joint"
-        params="joint_name parent child joint_axis_xyz joint_origin_xyz joint_origin_rpy joint_lower_limit joint_upper_limit joint_limit_vel joint_limit_effort joint_type">
+        params="joint_name
+                parent
+                child
+                joint_axis_xyz
+                joint_lower_limit
+                joint_upper_limit
+                joint_limit_vel
+                joint_limit_effort
+                joint_type
+                *origin">
         <joint name="${joint_name}" type="${joint_type}">
             <parent link="${parent}" />
@@ -97,5 +105,5 @@
                 lower="${joint_lower_limit}" upper="${joint_upper_limit}" />
             <!-- limit effort also defines torque limit and freeze controller gains -->
-            <origin xyz="${joint_origin_xyz}" rpy="${joint_origin_rpy}" />
+            <xacro:insert_block name="origin" />
         </joint>
     </xacro:macro>
@@ -104,10 +112,10 @@
     <!-- -->
     <xacro:macro name="dynaarm_joint_fixed"
-        params="joint_name parent child joint_origin_xyz joint_origin_rpy">
+        params="joint_name parent child *origin">
         <joint name="${joint_name}" type="fixed">
             <parent link="${parent}" />
             <child link="${child}" />
-            <origin xyz="${joint_origin_xyz}" rpy="${joint_origin_rpy}" />
             <limit effort="2000" velocity="0" lower="0" upper="0" />
+            <xacro:insert_block name="origin" />
         </joint>
     </xacro:macro>

Commit message: Renamed Joint WRIST_1 -> WR_FLE and WRIST_2 -> WR_ROT to make it work with Gazebo.

File: urdf/common/dynaarm.ros2control.xacro (robot description, xacro)
@@ -64,8 +64,8 @@
       </xacro:if>
       <xacro:if value="${dof >= 5}">
-        <xacro:dynaarm_ros2control_joint name="${tf_prefix}WRIST_1" address="5" />
+        <xacro:dynaarm_ros2control_joint name="${tf_prefix}WR_FLE" address="5" />
       </xacro:if>
       <xacro:if value="${dof >= 6}">
-        <xacro:dynaarm_ros2control_joint name="${tf_prefix}WRIST_2" address="6" />
+        <xacro:dynaarm_ros2control_joint name="${tf_prefix}WR_ROT" address="6" />
       </xacro:if>
     </ros2_control>

File: urdf/common/dynaarm_parameters_v1.urdf.xacro (robot description, xacro)
@@ -82,5 +82,5 @@
   <xacro:property name="joint_4_lower_limit" value="${-J_PI - J_PI/2}" />
   <xacro:property name="joint_4_upper_limit" value="${J_PI + J_PI/2}" />
-  <xacro:property name="joint_5_name" value="${tf_prefix}WRIST_1" />
+  <xacro:property name="joint_5_name" value="${tf_prefix}WR_FLE" />
   <xacro:property name="joint_5_joint_type" value="revolute" />
   <xacro:property name="joint_5_axis_xyz" value="0 0 1" />
@@ -89,5 +89,5 @@
   <xacro:property name="joint_5_lower_limit" value="${-J_PI/2}" />
   <xacro:property name="joint_5_upper_limit" value="${J_PI/2}" />
-  <xacro:property name="joint_6_name" value="${tf_prefix}WRIST_2" />
+  <xacro:property name="joint_6_name" value="${tf_prefix}WR_ROT" />
   <xacro:property name="joint_6_joint_type" value="revolute" />
   <xacro:property name="joint_6_axis_xyz" value="0 0 1" />

File: urdf/common/dynaarm_parameters_v2.urdf.xacro (robot description, xacro)
@@ -82,5 +82,5 @@
   <xacro:property name="joint_4_lower_limit" value="${-J_PI - J_PI/2}" />
   <xacro:property name="joint_4_upper_limit" value="${J_PI + J_PI/2}" />
-  <xacro:property name="joint_5_name" value="${tf_prefix}WRIST_1" />
+  <xacro:property name="joint_5_name" value="${tf_prefix}WR_FLE" />
   <xacro:property name="joint_5_joint_type" value="revolute" />
   <xacro:property name="joint_5_axis_xyz" value="0 0 1" />
@@ -89,5 +89,5 @@
   <xacro:property name="joint_5_lower_limit" value="${-J_PI/2}" />
   <xacro:property name="joint_5_upper_limit" value="${J_PI/2}" />
-  <xacro:property name="joint_6_name" value="${tf_prefix}WRIST_2" />
+  <xacro:property name="joint_6_name" value="${tf_prefix}WR_ROT" />
   <xacro:property name="joint_6_joint_type" value="revolute" />
   <xacro:property name="joint_6_axis_xyz" value="0 0 1" />

File: urdf/dynaarm.urdf.xacro (robot description, xacro)
@@ -274,5 +274,5 @@
       <plugin filename="libgz_ros2_control-system.so"
         name="gz_ros2_control::GazeboSimROS2ControlPlugin">
-        <parameters>$(find dynaarm_driver)/config/controllers.yaml</parameters>
+        <parameters>$(find dynaarm_examples)/config/controllers.yaml</parameters>
         <robotNamespace>dynaarm</robotNamespace>
         <robotDescription>dynaarm_description</robotDescription>

Commit message: Implement different freeze mode behavior and fixed parameter passing + names

File: urdf/common/dynaarm.ros2control.xacro (robot description, xacro)
@@ -21,5 +21,4 @@
     <state_interface name="motor_temperature_coil_C" />
     <state_interface name="motor_bus_voltage" />
-    <state_interface name="command_freeze_mode" />
     <command_interface name="position" />
     <command_interface name="velocity" />
@@ -28,5 +27,4 @@
     <command_interface name="i_gain" />
     <command_interface name="d_gain" />
-    <command_interface name="command_freeze_mode" />
   </xacro:macro>
   <xacro:macro name="dynaarm_ros2control_joint" params="name address">
@@ -36,6 +34,6 @@
     </joint>
   </xacro:macro>
-  <xacro:macro name="dynaarm_ros2_control" params="tf_prefix">
-    <ros2_control name="DynaarmSystem" type="system">
+  <xacro:macro name="dynaarm_ros2_control" params="tf_prefix ethercat_bus start_in_freeze_mode">
+    <ros2_control name="${tf_prefix}DynaarmSystem" type="system">
       <hardware>
         <xacro:if value="${mode == 'sim'}">
@@ -49,4 +47,5 @@
           <param name="ethercat_bus">${ethercat_bus}</param>
           <param name="tf_prefix">${tf_prefix}</param>
+          <param name="start_in_freeze_mode">${start_in_freeze_mode}</param>
         </xacro:if>
       </hardware>
@@ -69,4 +68,7 @@
         <xacro:dynaarm_ros2control_joint name="${tf_prefix}WR_ROT" address="6" />
       </xacro:if>
+      <gpio name="${tf_prefix}DynaarmSystem">
+       <command_interface name="freeze_mode" />
+      </gpio>
     </ros2_control>
   </xacro:macro>

File: urdf/dynaarm.urdf.xacro (robot description, xacro)
@@ -26,5 +26,5 @@
   <!-- -->
   <xacro:macro name="dynaarm"
-    params="tf_prefix parent_link dof mode ethercat_bus covers version *origin">
+    params="tf_prefix parent_link dof mode ethercat_bus start_in_freeze_mode:=false covers version *origin">
     <!-- Set ee_parent based on the specified DoF -->
     <xacro:property name="ee_parent" value="${base}" />
@@ -46,5 +46,5 @@
     </xacro:if>
     <!--ros2control-->
-    <xacro:dynaarm_ros2_control tf_prefix="${tf_prefix}" />
+    <xacro:dynaarm_ros2_control tf_prefix="${tf_prefix}" ethercat_bus="${ethercat_bus}" start_in_freeze_mode="${start_in_freeze_mode}"  />
   </xacro:macro>
   <!-- -->

Commit message: rename joint and link names

File: urdf/common/dynaarm.ros2control.xacro (robot description, xacro)
@@ -51,20 +51,20 @@
       </hardware>
       <xacro:if value="${dof >= 1}">
-        <xacro:dynaarm_ros2control_joint name="${tf_prefix}SH_ROT" address="1" />
+        <xacro:dynaarm_ros2control_joint name="${tf_prefix}shoulder_rotation" address="1" />
       </xacro:if>
       <xacro:if value="${dof >= 2}">
-        <xacro:dynaarm_ros2control_joint name="${tf_prefix}SH_FLE" address="2" />
+        <xacro:dynaarm_ros2control_joint name="${tf_prefix}shoulder_flexion" address="2" />
       </xacro:if>
       <xacro:if value="${dof >= 3}">
-        <xacro:dynaarm_ros2control_joint name="${tf_prefix}EL_FLE" address="3" />
+        <xacro:dynaarm_ros2control_joint name="${tf_prefix}elbow_flexion" address="3" />
       </xacro:if>
       <xacro:if value="${dof >= 4}">
-        <xacro:dynaarm_ros2control_joint name="${tf_prefix}FA_ROT" address="4" />
+        <xacro:dynaarm_ros2control_joint name="${tf_prefix}forearm_rotation" address="4" />
       </xacro:if>
       <xacro:if value="${dof >= 5}">
-        <xacro:dynaarm_ros2control_joint name="${tf_prefix}WR_FLE" address="5" />
+        <xacro:dynaarm_ros2control_joint name="${tf_prefix}wrist_flexion" address="5" />
       </xacro:if>
       <xacro:if value="${dof >= 6}">
-        <xacro:dynaarm_ros2control_joint name="${tf_prefix}WR_ROT" address="6" />
+        <xacro:dynaarm_ros2control_joint name="${tf_prefix}wrist_rotation" address="6" />
       </xacro:if>
       <gpio name="${tf_prefix}DynaarmSystem">

File: urdf/common/dynaarm_parameters_v1.urdf.xacro (robot description, xacro)
@@ -28,11 +28,11 @@
   <!-- Links -->
   <xacro:property name="base" value="${tf_prefix}base" />
-  <xacro:property name="link01" value="${tf_prefix}SHOULDER" />
-  <xacro:property name="link02" value="${tf_prefix}UPPERARM" />
-  <xacro:property name="link03" value="${tf_prefix}ELBOW" />
-  <xacro:property name="link04" value="${tf_prefix}FOREARM" />
-  <xacro:property name="link05" value="${tf_prefix}WRIST_1" />
-  <xacro:property name="link06" value="${tf_prefix}WRIST_2" />
-  <xacro:property name="end_effector" value="${tf_prefix}END_EFFECTOR" />
+  <xacro:property name="link01" value="${tf_prefix}shoulder" />
+  <xacro:property name="link02" value="${tf_prefix}upperarm" />
+  <xacro:property name="link03" value="${tf_prefix}elbow" />
+  <xacro:property name="link04" value="${tf_prefix}forearm" />
+  <xacro:property name="link05" value="${tf_prefix}wrist_1" />
+  <xacro:property name="link06" value="${tf_prefix}wrist_2" />
+  <xacro:property name="end_effector" value="${tf_prefix}flange" />
   <!-- Meshes -->
   <xacro:if value="${covers}">
@@ -67,5 +67,5 @@
   <xacro:property name="joint_base_origin_xyz" value="0 0 0" />
   <xacro:property name="joint_base_origin_rpy" value="0 0 0" />
-  <xacro:property name="joint_1_name" value="${tf_prefix}SH_ROT" />
+  <xacro:property name="joint_1_name" value="${tf_prefix}shoulder_rotation" />
   <xacro:property name="joint_1_joint_type" value="revolute" />
   <xacro:property name="joint_1_axis_xyz" value="0 0 1" />
@@ -74,5 +74,5 @@
   <xacro:property name="joint_1_lower_limit" value="${-J_PI - J_PI/2}" />
   <xacro:property name="joint_1_upper_limit" value="${J_PI + J_PI/2}" />
-  <xacro:property name="joint_2_name" value="${tf_prefix}SH_FLE" />
+  <xacro:property name="joint_2_name" value="${tf_prefix}shoulder_flexion" />
   <xacro:property name="joint_2_joint_type" value="revolute" />
   <xacro:property name="joint_2_axis_xyz" value="0 0 -1" />
@@ -81,5 +81,5 @@
   <xacro:property name="joint_2_lower_limit" value="${-J_PI/2 - 0.3}" />
   <xacro:property name="joint_2_upper_limit" value="${J_PI/2 + 0.3}" />
-  <xacro:property name="joint_3_name" value="${tf_prefix}EL_FLE" />
+  <xacro:property name="joint_3_name" value="${tf_prefix}elbow_flexion" />
   <xacro:property name="joint_3_joint_type" value="revolute" />
   <xacro:property name="joint_3_axis_xyz" value="0 0 1" />
@@ -88,5 +88,5 @@
   <xacro:property name="joint_3_lower_limit" value="-0.05" />
   <xacro:property name="joint_3_upper_limit" value="${J_PI}" />
-  <xacro:property name="joint_4_name" value="${tf_prefix}FA_ROT" />
+  <xacro:property name="joint_4_name" value="${tf_prefix}forearm_rotation" />
   <xacro:property name="joint_4_joint_type" value="revolute" />
   <xacro:property name="joint_4_axis_xyz" value="0 0 1" />
@@ -95,5 +95,5 @@
   <xacro:property name="joint_4_lower_limit" value="${-J_PI - J_PI/2}" />
   <xacro:property name="joint_4_upper_limit" value="${J_PI + J_PI/2}" />
-  <xacro:property name="joint_5_name" value="${tf_prefix}WR_FLE" />
+  <xacro:property name="joint_5_name" value="${tf_prefix}wrist_flexion" />
   <xacro:property name="joint_5_joint_type" value="revolute" />
   <xacro:property name="joint_5_axis_xyz" value="0 0 1" />
@@ -102,5 +102,5 @@
   <xacro:property name="joint_5_lower_limit" value="${-J_PI/2}" />
   <xacro:property name="joint_5_upper_limit" value="${J_PI/2}" />
-  <xacro:property name="joint_6_name" value="${tf_prefix}WR_ROT" />
+  <xacro:property name="joint_6_name" value="${tf_prefix}wrist_rotation" />
   <xacro:property name="joint_6_joint_type" value="revolute" />
   <xacro:property name="joint_6_axis_xyz" value="0 0 1" />
@@ -109,5 +109,5 @@
   <xacro:property name="joint_6_lower_limit" value="${-J_PI - J_PI/2}" />
   <xacro:property name="joint_6_upper_limit" value="${J_PI + J_PI/2}" />
-  <xacro:property name="joint_ee_name" value="${tf_prefix}ee_fix_joint" />
+  <xacro:property name="joint_ee_name" value="${tf_prefix}flange_fix_joint" />
   <xacro:property name="joint_ee_xyz" value="0.0 0.0 0.05" />
   <xacro:property name="joint_ee_origin_xyz" value="0.0 0.0 0.05" />

File: urdf/common/dynaarm_parameters_v2.urdf.xacro (robot description, xacro)
@@ -28,13 +28,13 @@
   <!-- Links -->
   <xacro:property name="base" value="${tf_prefix}base" />
-  <xacro:property name="link01" value="${tf_prefix}SHOULDER" />
-  <xacro:property name="link02" value="${tf_prefix}UPPERARM" />
-  <xacro:property name="link03" value="${tf_prefix}ELBOW" />
-  <xacro:property name="link03_cam" value="${tf_prefix}ELBOW_CAMERA_MOUNT" />
-  <xacro:property name="link04" value="${tf_prefix}FOREARM" />
-  <xacro:property name="link05" value="${tf_prefix}WRIST_1" />
-  <xacro:property name="link05_cam" value="${tf_prefix}WRIST_1_CAMERA_MOUNT" />
-  <xacro:property name="link06" value="${tf_prefix}WRIST_2" />
-  <xacro:property name="end_effector" value="${tf_prefix}END_EFFECTOR" />
+  <xacro:property name="link01" value="${tf_prefix}shoulder" />
+  <xacro:property name="link02" value="${tf_prefix}upperarm" />
+  <xacro:property name="link03" value="${tf_prefix}elbow" />
+  <xacro:property name="link03_cam" value="${tf_prefix}elbow_camera_mount" />
+  <xacro:property name="link04" value="${tf_prefix}forearm" />
+  <xacro:property name="link05" value="${tf_prefix}wrist_1" />
+  <xacro:property name="link05_cam" value="${tf_prefix}wrist_1_camera_mount" />
+  <xacro:property name="link06" value="${tf_prefix}wrist_2" />
+  <xacro:property name="end_effector" value="${tf_prefix}flange" />
   <!-- Meshes -->
   <xacro:if value="${covers}">
@@ -69,5 +69,5 @@
   <xacro:property name="joint_base_origin_xyz" value="0 0 0" />
   <xacro:property name="joint_base_origin_rpy" value="0 0 0" />
-  <xacro:property name="joint_1_name" value="${tf_prefix}SH_ROT" />
+  <xacro:property name="joint_1_name" value="${tf_prefix}shoulder_rotation" />
   <xacro:property name="joint_1_joint_type" value="revolute" />
   <xacro:property name="joint_1_axis_xyz" value="0 0 1" />
@@ -76,5 +76,5 @@
   <xacro:property name="joint_1_lower_limit" value="${-J_PI - J_PI/2}" />
   <xacro:property name="joint_1_upper_limit" value="${J_PI + J_PI/2}" />
-  <xacro:property name="joint_2_name" value="${tf_prefix}SH_FLE" />
+  <xacro:property name="joint_2_name" value="${tf_prefix}shoulder_flexion" />
   <xacro:property name="joint_2_joint_type" value="revolute" />
   <xacro:property name="joint_2_axis_xyz" value="0 0 1" />
@@ -83,5 +83,5 @@
   <xacro:property name="joint_2_lower_limit" value="${-J_PI/2 - 0.3}" />
   <xacro:property name="joint_2_upper_limit" value="${J_PI/2 + 0.3}" />
-  <xacro:property name="joint_3_name" value="${tf_prefix}EL_FLE" />
+  <xacro:property name="joint_3_name" value="${tf_prefix}elbow_flexion" />
   <xacro:property name="joint_3_joint_type" value="revolute" />
   <xacro:property name="joint_3_axis_xyz" value="0 0 1" />
@@ -90,10 +90,10 @@
   <xacro:property name="joint_3_lower_limit" value="-0.05" />
   <xacro:property name="joint_3_upper_limit" value="${J_PI}" />
-  <xacro:property name="joint_3_cam_name" value="${tf_prefix}EL_CAMERA" />
+  <xacro:property name="joint_3_cam_name" value="${tf_prefix}elbow_camera" />
   <xacro:property name="joint_3_cam_joint_type" value="fixed" />
   <xacro:property name="joint_3_cam_axis_xyz" value="0 0 0" />
   <xacro:property name="joint_3_cam_origin_xyz" value="0.0345 -0.1235 0" />
   <xacro:property name="joint_3_cam_origin_rpy" value="0.0 0.0 0.0" />
-  <xacro:property name="joint_4_name" value="${tf_prefix}FA_ROT" />
+  <xacro:property name="joint_4_name" value="${tf_prefix}forearm_rotation" />
   <xacro:property name="joint_4_joint_type" value="revolute" />
   <xacro:property name="joint_4_axis_xyz" value="0 0 1" />
@@ -102,5 +102,5 @@
   <xacro:property name="joint_4_lower_limit" value="${-J_PI - J_PI/2}" />
   <xacro:property name="joint_4_upper_limit" value="${J_PI + J_PI/2}" />
-  <xacro:property name="joint_5_name" value="${tf_prefix}WR_FLE" />
+  <xacro:property name="joint_5_name" value="${tf_prefix}wrist_flexion" />
   <xacro:property name="joint_5_joint_type" value="revolute" />
   <xacro:property name="joint_5_axis_xyz" value="0 0 1" />
@@ -109,10 +109,10 @@
   <xacro:property name="joint_5_lower_limit" value="${-J_PI/2}" />
   <xacro:property name="joint_5_upper_limit" value="${J_PI/2}" />
-  <xacro:property name="joint_5_cam_name" value="${tf_prefix}WR_FLE_CAMERA" />
+  <xacro:property name="joint_5_cam_name" value="${tf_prefix}wrist_flexion_camera" />
   <xacro:property name="joint_5_cam_joint_type" value="fixed" />
   <xacro:property name="joint_5_cam_axis_xyz" value="0 0 0" />
   <xacro:property name="joint_5_cam_origin_xyz" value="0.032 0 -0.017" />
   <xacro:property name="joint_5_cam_origin_rpy" value="0.0 0.0 0.0" />
-  <xacro:property name="joint_6_name" value="${tf_prefix}WR_ROT" />
+  <xacro:property name="joint_6_name" value="${tf_prefix}wrist_rotation" />
   <xacro:property name="joint_6_joint_type" value="revolute" />
   <xacro:property name="joint_6_axis_xyz" value="0 0 1" />
@@ -121,5 +121,5 @@
   <xacro:property name="joint_6_lower_limit" value="${-J_PI - J_PI/2}" />
   <xacro:property name="joint_6_upper_limit" value="${J_PI + J_PI/2}" />
-  <xacro:property name="joint_ee_name" value="${tf_prefix}ee_fix_joint" />
+  <xacro:property name="joint_ee_name" value="${tf_prefix}flange_fix_joint" />
   <xacro:property name="joint_ee_xyz" value="0.0 0.0 0.05" />
   <xacro:property name="joint_ee_origin_xyz" value="0.0 0.0 0.05" />
