Commit message: added drive parameter folder argument to dynaarm macro

File: urdf/common/dynaarm.ros2control.xacro (robot description, xacro)
@@ -34,5 +34,5 @@
     </joint>
   </xacro:macro>
-  <xacro:macro name="dynaarm_ros2_control" params="tf_prefix ethercat_bus start_in_freeze_mode">
+  <xacro:macro name="dynaarm_ros2_control" params="tf_prefix ethercat_bus start_in_freeze_mode drive_parameter_folder">
     <ros2_control name="${tf_prefix}DynaarmSystem" type="system">
       <hardware>
@@ -48,4 +48,5 @@
           <param name="tf_prefix">${tf_prefix}</param>
           <param name="start_in_freeze_mode">${start_in_freeze_mode}</param>
+          <param name="drive_parameter_folder">${drive_parameter_folder}</param>
         </xacro:if>
       </hardware>

File: urdf/dynaarm.urdf.xacro (robot description, xacro)
@@ -26,5 +26,12 @@
   <!-- -->
   <xacro:macro name="dynaarm"
-    params="tf_prefix parent_link dof mode ethercat_bus start_in_freeze_mode:=false covers version *origin">
+    params="tf_prefix parent_link dof mode ethercat_bus start_in_freeze_mode:=false drive_parameter_folder:='' covers version *origin">
+    <xacro:property name="default_drive_parameter_folder" value="$(find dynaarm_driver)/config/${version}" />
+    <xacro:if value="${drive_parameter_folder == ''}">
+      <xacro:property name="drive_parameter_folder_internal" value="${default_drive_parameter_folder}" />
+    </xacro:if>
+    <xacro:unless value="${drive_parameter_folder == ''}">
+      <xacro:property name="drive_parameter_folder_internal" value="${drive_parameter_folder}" />
+    </xacro:unless>
     <!-- Set ee_parent based on the specified DoF -->
     <xacro:property name="ee_parent" value="${base}" />
@@ -46,5 +53,5 @@
     </xacro:if>
     <!--ros2control-->
-    <xacro:dynaarm_ros2_control tf_prefix="${tf_prefix}" ethercat_bus="${ethercat_bus}" start_in_freeze_mode="${start_in_freeze_mode}"  />
+    <xacro:dynaarm_ros2_control tf_prefix="${tf_prefix}" ethercat_bus="${ethercat_bus}" start_in_freeze_mode="${start_in_freeze_mode}"  drive_parameter_folder="${drive_parameter_folder_internal}" />
   </xacro:macro>
   <!-- -->

Commit message: better default parameter path handling

File: urdf/common/dynaarm.ros2control.xacro (robot description, xacro)
@@ -34,5 +34,5 @@
     </joint>
   </xacro:macro>
-  <xacro:macro name="dynaarm_ros2_control" params="tf_prefix ethercat_bus start_in_freeze_mode drive_parameter_folder">
+  <xacro:macro name="dynaarm_ros2_control" params="tf_prefix ethercat_bus start_in_freeze_mode drive_parameter_folder drive_parameter_folder_default">
     <ros2_control name="${tf_prefix}DynaarmSystem" type="system">
       <hardware>
@@ -49,4 +49,5 @@
           <param name="start_in_freeze_mode">${start_in_freeze_mode}</param>
           <param name="drive_parameter_folder">${drive_parameter_folder}</param>
+          <param name="drive_parameter_folder_default">${drive_parameter_folder_default}</param>
         </xacro:if>
       </hardware>

File: urdf/dynaarm.urdf.xacro (robot description, xacro)
@@ -53,5 +53,5 @@
     </xacro:if>
     <!--ros2control-->
-    <xacro:dynaarm_ros2_control tf_prefix="${tf_prefix}" ethercat_bus="${ethercat_bus}" start_in_freeze_mode="${start_in_freeze_mode}"  drive_parameter_folder="${drive_parameter_folder_internal}" />
+    <xacro:dynaarm_ros2_control tf_prefix="${tf_prefix}" ethercat_bus="${ethercat_bus}" start_in_freeze_mode="${start_in_freeze_mode}"  drive_parameter_folder="${drive_parameter_folder_internal}" drive_parameter_folder_default="${default_drive_parameter_folder}" />
   </xacro:macro>
   <!-- -->

Commit message: Add proper gazebo support

File: urdf/common/dynaarm.ros2control.xacro (robot description, xacro)
@@ -11,6 +11,6 @@
   <xacro:macro name="dynaarm_joint_ros2control_joint_interfaces">
     <state_interface name="position">
-        <!-- Slightly offset the initial position for the gazebo sim-->
-        <param name="initial_value">0.05</param>
+      <!-- Slightly offset the initial position for the gazebo sim-->
+      <param name="initial_value">0.05</param>
     </state_interface>
     <state_interface name="velocity" />
@@ -41,5 +41,9 @@
       <hardware>
         <xacro:if value="${mode == 'sim'}">
-          <plugin>gz_ros2_control/GazeboSimSystem</plugin>
+          <plugin>dynaarm_gz_ros2_control/GazeboSimSystem</plugin>
+          <param name="drive_parameter_folder">${drive_parameter_folder}</param>
+          <param name="drive_parameter_folder_default">${drive_parameter_folder_default}</param>
+          <param name="drive_mode">JointPositionVelocityTorquePidGains</param>
+          <use_force_commands>true</use_force_commands>
         </xacro:if>
         <xacro:if value="${mode == 'mock'}">
@@ -79,5 +83,5 @@
       </xacro:if>
       <gpio name="${tf_prefix}DynaarmSystem">
-       <command_interface name="freeze_mode" />
+        <command_interface name="freeze_mode" />
       </gpio>
     </ros2_control>

File: urdf/dynaarm.urdf.xacro (robot description, xacro)
@@ -330,10 +330,10 @@
   <!-- -->
   <xacro:macro name="dynaarm_tool">
-      <xacro:virtual_link link_name="${end_effector}" />
-      <xacro:dynaarm_joint_fixed joint_name="${joint_ee_name}"
-          parent="${ee_parent}"
-          child="${end_effector}">
-          <origin xyz="${joint_ee_origin_xyz}" rpy="${joint_ee_origin_rpy}" />
-      </xacro:dynaarm_joint_fixed>
+    <xacro:virtual_link link_name="${end_effector}" />
+    <xacro:dynaarm_joint_fixed joint_name="${joint_ee_name}"
+      parent="${ee_parent}"
+      child="${end_effector}">
+      <origin xyz="${joint_ee_origin_xyz}" rpy="${joint_ee_origin_rpy}" />
+    </xacro:dynaarm_joint_fixed>
   </xacro:macro>
   <!-- -->
@@ -342,8 +342,8 @@
   <xacro:macro name="dynaarm_gazebo" params="controller_path">
     <gazebo>
-      <plugin filename="libgz_ros2_control-system.so"
-        name="gz_ros2_control::GazeboSimROS2ControlPlugin">
+      <plugin filename="libdynaarm_gz_ros2_control-system.so"
+        name="dynaarm_gz_ros2_control::GazeboSimROS2ControlPlugin">
         <parameters>${controller_path}</parameters>
-        <update_rate>100</update_rate>
+        <pid_update_rate>1000</pid_update_rate>
       </plugin>
     </gazebo>

Commit message: Revert "Add proper gazebo support"
This reverts commit afd9097127cdf16fc4f4d5ccc5eb0934313a3127.

File: urdf/common/dynaarm.ros2control.xacro (robot description, xacro)
@@ -11,6 +11,6 @@
   <xacro:macro name="dynaarm_joint_ros2control_joint_interfaces">
     <state_interface name="position">
-      <!-- Slightly offset the initial position for the gazebo sim-->
-      <param name="initial_value">0.05</param>
+        <!-- Slightly offset the initial position for the gazebo sim-->
+        <param name="initial_value">0.05</param>
     </state_interface>
     <state_interface name="velocity" />
@@ -41,9 +41,5 @@
       <hardware>
         <xacro:if value="${mode == 'sim'}">
-          <plugin>dynaarm_gz_ros2_control/GazeboSimSystem</plugin>
-          <param name="drive_parameter_folder">${drive_parameter_folder}</param>
-          <param name="drive_parameter_folder_default">${drive_parameter_folder_default}</param>
-          <param name="drive_mode">JointPositionVelocityTorquePidGains</param>
-          <use_force_commands>true</use_force_commands>
+          <plugin>gz_ros2_control/GazeboSimSystem</plugin>
         </xacro:if>
         <xacro:if value="${mode == 'mock'}">
@@ -83,5 +79,5 @@
       </xacro:if>
       <gpio name="${tf_prefix}DynaarmSystem">
-        <command_interface name="freeze_mode" />
+       <command_interface name="freeze_mode" />
       </gpio>
     </ros2_control>

File: urdf/dynaarm.urdf.xacro (robot description, xacro)
@@ -330,10 +330,10 @@
   <!-- -->
   <xacro:macro name="dynaarm_tool">
-    <xacro:virtual_link link_name="${end_effector}" />
-    <xacro:dynaarm_joint_fixed joint_name="${joint_ee_name}"
-      parent="${ee_parent}"
-      child="${end_effector}">
-      <origin xyz="${joint_ee_origin_xyz}" rpy="${joint_ee_origin_rpy}" />
-    </xacro:dynaarm_joint_fixed>
+      <xacro:virtual_link link_name="${end_effector}" />
+      <xacro:dynaarm_joint_fixed joint_name="${joint_ee_name}"
+          parent="${ee_parent}"
+          child="${end_effector}">
+          <origin xyz="${joint_ee_origin_xyz}" rpy="${joint_ee_origin_rpy}" />
+      </xacro:dynaarm_joint_fixed>
   </xacro:macro>
   <!-- -->
@@ -342,8 +342,8 @@
   <xacro:macro name="dynaarm_gazebo" params="controller_path">
     <gazebo>
-      <plugin filename="libdynaarm_gz_ros2_control-system.so"
-        name="dynaarm_gz_ros2_control::GazeboSimROS2ControlPlugin">
+      <plugin filename="libgz_ros2_control-system.so"
+        name="gz_ros2_control::GazeboSimROS2ControlPlugin">
         <parameters>${controller_path}</parameters>
-        <pid_update_rate>1000</pid_update_rate>
+        <update_rate>100</update_rate>
       </plugin>
     </gazebo>

Commit message: Added setup for isaac-sim

File: urdf/common/dynaarm.ros2control.xacro (robot description, xacro)
@@ -31,13 +31,32 @@
     <command_interface name="d_gain" />
   </xacro:macro>
-  <xacro:macro name="dynaarm_ros2control_joint" params="name address">
+  <xacro:macro name="dynaarm_ros2control_joint" params="name address mode">
     <joint name="${name}">
-      <param name="address">${address}</param>
-      <xacro:dynaarm_joint_ros2control_joint_interfaces />
+      <xacro:if value="${mode != 'isaac'}">
+        <param name="address">${address}</param>
+        <xacro:dynaarm_joint_ros2control_joint_interfaces />
+      </xacro:if>
+      <xacro:if value="${mode == 'isaac'}">
+        <command_interface name="position" />
+        <command_interface name="velocity" />
+        <command_interface name="effort" />
+        <state_interface name="position">
+          <param name="initial_value">0.0</param>
+        </state_interface>
+        <state_interface name="velocity" />
+        <state_interface name="effort" />
+      </xacro:if>
     </joint>
   </xacro:macro>
-  <xacro:macro name="dynaarm_ros2_control" params="tf_prefix ethercat_bus start_in_freeze_mode drive_parameter_folder drive_parameter_folder_default ethercat_addresses">
+  <xacro:macro name="dynaarm_ros2_control" params="tf_prefix ethercat_bus start_in_freeze_mode drive_parameter_folder drive_parameter_folder_default ethercat_addresses mode">
     <ros2_control name="${tf_prefix}DynaarmSystem" type="system">
       <hardware>
+        <xacro:if value="${mode == 'isaac'}">
+          <plugin>joint_state_topic_hardware_interface/JointStateTopicSystem</plugin>
+          <param name="joint_states_topic">/isaac_joint_states</param>
+          <param name="joint_commands_topic">/isaac_joint_command</param>
+          <!-- Isaac wraps joint angles, this helps un-wrap them -->
+          <param name="sum_wrapped_joint_states">true</param>
+        </xacro:if>
         <xacro:if value="${mode == 'sim'}">
           <plugin>gz_ros2_control/GazeboSimSystem</plugin>
@@ -61,24 +80,26 @@
       </hardware>
       <xacro:if value="${dof >= 1}">
-        <xacro:dynaarm_ros2control_joint name="${tf_prefix}shoulder_rotation" address="${ethercat_addresses['shoulder_rotation']}" />
+        <xacro:dynaarm_ros2control_joint name="${tf_prefix}shoulder_rotation" address="${ethercat_addresses['shoulder_rotation']}" mode="${mode}" />
       </xacro:if>
       <xacro:if value="${dof >= 2}">
-        <xacro:dynaarm_ros2control_joint name="${tf_prefix}shoulder_flexion" address="${ethercat_addresses['shoulder_flexion']}" />
+        <xacro:dynaarm_ros2control_joint name="${tf_prefix}shoulder_flexion" address="${ethercat_addresses['shoulder_flexion']}" mode="${mode}" />
       </xacro:if>
       <xacro:if value="${dof >= 3}">
-        <xacro:dynaarm_ros2control_joint name="${tf_prefix}elbow_flexion" address="${ethercat_addresses['elbow_flexion']}" />
+        <xacro:dynaarm_ros2control_joint name="${tf_prefix}elbow_flexion" address="${ethercat_addresses['elbow_flexion']}" mode="${mode}" />
       </xacro:if>
       <xacro:if value="${dof >= 4}">
-        <xacro:dynaarm_ros2control_joint name="${tf_prefix}forearm_rotation" address="${ethercat_addresses['forearm_rotation']}" />
+        <xacro:dynaarm_ros2control_joint name="${tf_prefix}forearm_rotation" address="${ethercat_addresses['forearm_rotation']}" mode="${mode}" />
       </xacro:if>
       <xacro:if value="${dof >= 5}">
-        <xacro:dynaarm_ros2control_joint name="${tf_prefix}wrist_flexion" address="${ethercat_addresses['wrist_flexion']}" />
+        <xacro:dynaarm_ros2control_joint name="${tf_prefix}wrist_flexion" address="${ethercat_addresses['wrist_flexion']}" mode="${mode}" />
       </xacro:if>
       <xacro:if value="${dof >= 6}">
-        <xacro:dynaarm_ros2control_joint name="${tf_prefix}wrist_rotation" address="${ethercat_addresses['wrist_rotation']}" />
+        <xacro:dynaarm_ros2control_joint name="${tf_prefix}wrist_rotation" address="${ethercat_addresses['wrist_rotation']}" mode="${mode}" />
       </xacro:if>
-      <gpio name="${tf_prefix}DynaarmSystem">
-       <command_interface name="freeze_mode" />
-      </gpio>
+      <xacro:if value="${mode != 'isaac'}">
+        <gpio name="${tf_prefix}DynaarmSystem">
+          <command_interface name="freeze_mode" />
+        </gpio>
+      </xacro:if>
     </ros2_control>
   </xacro:macro>

File: urdf/dynaarm_standalone.urdf.xacro (robot description, xacro)
@@ -24,4 +24,5 @@
   <!-- Path to ros2_control controller config file -->
   <xacro:arg name="controller_path" default="" />
+  <xacro:arg name="namespace" default="dynaarm1" />
   <xacro:include filename="$(find dynaarm_description)/urdf/dynaarm.urdf.xacro" />
   <link name="base_link" />
