Commit message: Allow changing the ethercat address for different arm versions

File: urdf/common/arowana4/dynaarm_parameters.urdf.xacro (robot description, xacro)
@@ -21,4 +21,7 @@
 -->
 <robot xmlns:xacro="http://www.ros.org/wiki/xacro">
+  <xacro:property name="arm_version_name" value="arowana4"/>
+  <!-- Obtain the ethercat drive order (address order list)-->
+  <xacro:include filename="$(find dynaarm_description)/urdf/common/${arm_version_name}/drive_order.urdf.xacro"/>
   <xacro:property name="J_PI" value="3.14159265359" />
   <xacro:property name="baboon_peak_torque" value="40" />

File: urdf/common/baracuda12/dynaarm_parameters.urdf.xacro (robot description, xacro)
@@ -21,4 +21,7 @@
 -->
 <robot xmlns:xacro="http://www.ros.org/wiki/xacro">
+  <xacro:property name="arm_version_name" value="baracuda12"/>
+  <!-- Obtain the ethercat drive order (address order list)-->
+  <xacro:include filename="$(find dynaarm_description)/urdf/common/${arm_version_name}/drive_order.urdf.xacro"/>
   <xacro:property name="J_PI" value="3.14159265359" />
   <xacro:property name="baboon_peak_torque" value="40" />

File: urdf/common/dynaarm.ros2control.xacro (robot description, xacro)
@@ -34,5 +34,5 @@
     </joint>
   </xacro:macro>
-  <xacro:macro name="dynaarm_ros2_control" params="tf_prefix ethercat_bus start_in_freeze_mode drive_parameter_folder drive_parameter_folder_default">
+  <xacro:macro name="dynaarm_ros2_control" params="tf_prefix ethercat_bus start_in_freeze_mode drive_parameter_folder drive_parameter_folder_default ethercat_addresses">
     <ros2_control name="${tf_prefix}DynaarmSystem" type="system">
       <hardware>
@@ -53,20 +53,20 @@
       </hardware>
       <xacro:if value="${dof >= 1}">
-        <xacro:dynaarm_ros2control_joint name="${tf_prefix}shoulder_rotation" address="1" />
+        <xacro:dynaarm_ros2control_joint name="${tf_prefix}shoulder_rotation" address="${ethercat_addresses[0]}" />
       </xacro:if>
       <xacro:if value="${dof >= 2}">
-        <xacro:dynaarm_ros2control_joint name="${tf_prefix}shoulder_flexion" address="2" />
+        <xacro:dynaarm_ros2control_joint name="${tf_prefix}shoulder_flexion" address="${ethercat_addresses[1]}" />
       </xacro:if>
       <xacro:if value="${dof >= 3}">
-        <xacro:dynaarm_ros2control_joint name="${tf_prefix}elbow_flexion" address="3" />
+        <xacro:dynaarm_ros2control_joint name="${tf_prefix}elbow_flexion" address="${ethercat_addresses[2]}" />
       </xacro:if>
       <xacro:if value="${dof >= 4}">
-        <xacro:dynaarm_ros2control_joint name="${tf_prefix}forearm_rotation" address="4" />
+        <xacro:dynaarm_ros2control_joint name="${tf_prefix}forearm_rotation" address="${ethercat_addresses[3]}" />
       </xacro:if>
       <xacro:if value="${dof >= 5}">
-        <xacro:dynaarm_ros2control_joint name="${tf_prefix}wrist_flexion" address="5" />
+        <xacro:dynaarm_ros2control_joint name="${tf_prefix}wrist_flexion" address="${ethercat_addresses[4]}" />
       </xacro:if>
       <xacro:if value="${dof >= 6}">
-        <xacro:dynaarm_ros2control_joint name="${tf_prefix}wrist_rotation" address="6" />
+        <xacro:dynaarm_ros2control_joint name="${tf_prefix}wrist_rotation" address="${ethercat_addresses[5]}" />
       </xacro:if>
       <gpio name="${tf_prefix}DynaarmSystem">

File: urdf/dynaarm.urdf.xacro (robot description, xacro)
@@ -27,4 +27,5 @@
   <xacro:macro name="dynaarm"
     params="tf_prefix parent_link dof mode ethercat_bus start_in_freeze_mode:=false drive_parameter_folder:='' covers version *origin">
+    <!--Allow the user to pass a custom folder for drive parameters-->
     <xacro:property name="default_drive_parameter_folder" value="$(find dynaarm_driver)/config/${version}" />
     <xacro:if value="${drive_parameter_folder == ''}">
@@ -37,4 +38,5 @@
     <xacro:property name="ee_parent" value="${base}" />
     <xacro:include filename="$(find dynaarm_description)/urdf/common/dynaarm_common.urdf.xacro" />
+    <!-- Include the version specific information-->
     <xacro:include
       filename="$(find dynaarm_description)/urdf/common/${version}/dynaarm_parameters.urdf.xacro" />
@@ -53,5 +55,5 @@
     </xacro:if>
     <!--ros2control-->
-    <xacro:dynaarm_ros2_control tf_prefix="${tf_prefix}" ethercat_bus="${ethercat_bus}" start_in_freeze_mode="${start_in_freeze_mode}"  drive_parameter_folder="${drive_parameter_folder_internal}" drive_parameter_folder_default="${default_drive_parameter_folder}" />
+    <xacro:dynaarm_ros2_control tf_prefix="${tf_prefix}" ethercat_bus="${ethercat_bus}" start_in_freeze_mode="${start_in_freeze_mode}"  drive_parameter_folder="${drive_parameter_folder_internal}" drive_parameter_folder_default="${default_drive_parameter_folder}" ethercat_addresses="${ethercat_addresses}"/>
   </xacro:macro>
   <!-- -->

Commit message: rework patch

File: urdf/common/arowana4/dynaarm_parameters.urdf.xacro (robot description, xacro)
@@ -23,5 +23,6 @@
   <xacro:property name="arm_version_name" value="arowana4"/>
   <!-- Obtain the ethercat drive order (address order list)-->
-  <xacro:include filename="$(find dynaarm_description)/urdf/common/${arm_version_name}/drive_order.urdf.xacro"/>
+  <xacro:property name="drive_order_path" value="$(find dynaarm_description)/urdf/common/${arm_version_name}/drive_order.yaml"/>
+  <xacro:property name="ethercat_addresses" value="${xacro.load_yaml(drive_order_path)}"/>
   <xacro:property name="J_PI" value="3.14159265359" />
   <xacro:property name="baboon_peak_torque" value="40" />

File: urdf/common/baracuda12/dynaarm_parameters.urdf.xacro (robot description, xacro)
@@ -23,5 +23,6 @@
   <xacro:property name="arm_version_name" value="baracuda12"/>
   <!-- Obtain the ethercat drive order (address order list)-->
-  <xacro:include filename="$(find dynaarm_description)/urdf/common/${arm_version_name}/drive_order.urdf.xacro"/>
+  <xacro:property name="drive_order_path" value="$(find dynaarm_description)/urdf/common/${arm_version_name}/drive_order.yaml"/>
+  <xacro:property name="ethercat_addresses" value="${xacro.load_yaml(drive_order_path)}"/>
   <xacro:property name="J_PI" value="3.14159265359" />
   <xacro:property name="baboon_peak_torque" value="40" />

File: urdf/common/dynaarm.ros2control.xacro (robot description, xacro)
@@ -53,20 +53,20 @@
       </hardware>
       <xacro:if value="${dof >= 1}">
-        <xacro:dynaarm_ros2control_joint name="${tf_prefix}shoulder_rotation" address="${ethercat_addresses[0]}" />
+        <xacro:dynaarm_ros2control_joint name="${tf_prefix}shoulder_rotation" address="${ethercat_addresses['shoulder_rotation']}" />
       </xacro:if>
       <xacro:if value="${dof >= 2}">
-        <xacro:dynaarm_ros2control_joint name="${tf_prefix}shoulder_flexion" address="${ethercat_addresses[1]}" />
+        <xacro:dynaarm_ros2control_joint name="${tf_prefix}shoulder_flexion" address="${ethercat_addresses['shoulder_flexion']}" />
       </xacro:if>
       <xacro:if value="${dof >= 3}">
-        <xacro:dynaarm_ros2control_joint name="${tf_prefix}elbow_flexion" address="${ethercat_addresses[2]}" />
+        <xacro:dynaarm_ros2control_joint name="${tf_prefix}elbow_flexion" address="${ethercat_addresses['elbow_flexion']}" />
       </xacro:if>
       <xacro:if value="${dof >= 4}">
-        <xacro:dynaarm_ros2control_joint name="${tf_prefix}forearm_rotation" address="${ethercat_addresses[3]}" />
+        <xacro:dynaarm_ros2control_joint name="${tf_prefix}forearm_rotation" address="${ethercat_addresses['forearm_rotation']}" />
       </xacro:if>
       <xacro:if value="${dof >= 5}">
-        <xacro:dynaarm_ros2control_joint name="${tf_prefix}wrist_flexion" address="${ethercat_addresses[4]}" />
+        <xacro:dynaarm_ros2control_joint name="${tf_prefix}wrist_flexion" address="${ethercat_addresses['wrist_flexion']}" />
       </xacro:if>
       <xacro:if value="${dof >= 6}">
-        <xacro:dynaarm_ros2control_joint name="${tf_prefix}wrist_rotation" address="${ethercat_addresses[5]}" />
+        <xacro:dynaarm_ros2control_joint name="${tf_prefix}wrist_rotation" address="${ethercat_addresses['wrist_rotation']}" />
       </xacro:if>
       <gpio name="${tf_prefix}DynaarmSystem">

Commit message: Allow changing the ethercat address for different arm versions (#32)
* Allow changing the ethercat address for different arm versions
---------

Co-authored-by: Lennart Nachtigall <mail@firesurfer.de>

File: urdf/common/arowana4/dynaarm_parameters.urdf.xacro (robot description, xacro)
@@ -21,4 +21,8 @@
 -->
 <robot xmlns:xacro="http://www.ros.org/wiki/xacro">
+  <xacro:property name="arm_version_name" value="arowana4"/>
+  <!-- Obtain the ethercat drive order (address order list)-->
+  <xacro:property name="drive_order_path" value="$(find dynaarm_description)/urdf/common/${arm_version_name}/drive_order.yaml"/>
+  <xacro:property name="ethercat_addresses" value="${xacro.load_yaml(drive_order_path)}"/>
   <xacro:property name="J_PI" value="3.14159265359" />
   <xacro:property name="baboon_peak_torque" value="40" />

File: urdf/common/baracuda12/dynaarm_parameters.urdf.xacro (robot description, xacro)
@@ -21,4 +21,8 @@
 -->
 <robot xmlns:xacro="http://www.ros.org/wiki/xacro">
+  <xacro:property name="arm_version_name" value="baracuda12"/>
+  <!-- Obtain the ethercat drive order (address order list)-->
+  <xacro:property name="drive_order_path" value="$(find dynaarm_description)/urdf/common/${arm_version_name}/drive_order.yaml"/>
+  <xacro:property name="ethercat_addresses" value="${xacro.load_yaml(drive_order_path)}"/>
   <xacro:property name="J_PI" value="3.14159265359" />
   <xacro:property name="baboon_peak_torque" value="40" />

File: urdf/common/dynaarm.ros2control.xacro (robot description, xacro)
@@ -34,5 +34,5 @@
     </joint>
   </xacro:macro>
-  <xacro:macro name="dynaarm_ros2_control" params="tf_prefix ethercat_bus start_in_freeze_mode drive_parameter_folder drive_parameter_folder_default">
+  <xacro:macro name="dynaarm_ros2_control" params="tf_prefix ethercat_bus start_in_freeze_mode drive_parameter_folder drive_parameter_folder_default ethercat_addresses">
     <ros2_control name="${tf_prefix}DynaarmSystem" type="system">
       <hardware>
@@ -53,20 +53,20 @@
       </hardware>
       <xacro:if value="${dof >= 1}">
-        <xacro:dynaarm_ros2control_joint name="${tf_prefix}shoulder_rotation" address="1" />
+        <xacro:dynaarm_ros2control_joint name="${tf_prefix}shoulder_rotation" address="${ethercat_addresses['shoulder_rotation']}" />
       </xacro:if>
       <xacro:if value="${dof >= 2}">
-        <xacro:dynaarm_ros2control_joint name="${tf_prefix}shoulder_flexion" address="2" />
+        <xacro:dynaarm_ros2control_joint name="${tf_prefix}shoulder_flexion" address="${ethercat_addresses['shoulder_flexion']}" />
       </xacro:if>
       <xacro:if value="${dof >= 3}">
-        <xacro:dynaarm_ros2control_joint name="${tf_prefix}elbow_flexion" address="3" />
+        <xacro:dynaarm_ros2control_joint name="${tf_prefix}elbow_flexion" address="${ethercat_addresses['elbow_flexion']}" />
       </xacro:if>
       <xacro:if value="${dof >= 4}">
-        <xacro:dynaarm_ros2control_joint name="${tf_prefix}forearm_rotation" address="4" />
+        <xacro:dynaarm_ros2control_joint name="${tf_prefix}forearm_rotation" address="${ethercat_addresses['forearm_rotation']}" />
       </xacro:if>
       <xacro:if value="${dof >= 5}">
-        <xacro:dynaarm_ros2control_joint name="${tf_prefix}wrist_flexion" address="5" />
+        <xacro:dynaarm_ros2control_joint name="${tf_prefix}wrist_flexion" address="${ethercat_addresses['wrist_flexion']}" />
       </xacro:if>
       <xacro:if value="${dof >= 6}">
-        <xacro:dynaarm_ros2control_joint name="${tf_prefix}wrist_rotation" address="6" />
+        <xacro:dynaarm_ros2control_joint name="${tf_prefix}wrist_rotation" address="${ethercat_addresses['wrist_rotation']}" />
       </xacro:if>
       <gpio name="${tf_prefix}DynaarmSystem">

Commit message: Implemented a way to pass a drive order file to the dynaarm so the ethercat addresses can be loaded from there. Otherwise the default addresses will be loaded.

File: urdf/common/arowana4/dynaarm_parameters.urdf.xacro (robot description, xacro)
@@ -22,7 +22,10 @@
 <robot xmlns:xacro="http://www.ros.org/wiki/xacro">
   <xacro:property name="arm_version_name" value="arowana4"/>
-  <!-- Obtain the ethercat drive order (address order list)-->
-  <xacro:property name="drive_order_path" value="$(find dynaarm_description)/urdf/common/${arm_version_name}/drive_order.yaml"/>
-  <xacro:property name="ethercat_addresses" value="${xacro.load_yaml(drive_order_path)}"/>
+  <!--
+    Obtain the EtherCAT drive order (address order list).
+    The drive_order.yaml file is either loaded from the default location
+    in dynaarm.urdf.xacro or passed down from another launch file.
+  -->
+  <xacro:property name="ethercat_addresses" value="${xacro.load_yaml(drive_order_file)}"/>
   <xacro:property name="J_PI" value="3.14159265359" />
   <xacro:property name="baboon_peak_torque" value="40" />

File: urdf/common/baracuda12/dynaarm_parameters.urdf.xacro (robot description, xacro)
@@ -22,7 +22,10 @@
 <robot xmlns:xacro="http://www.ros.org/wiki/xacro">
   <xacro:property name="arm_version_name" value="baracuda12"/>
-  <!-- Obtain the ethercat drive order (address order list)-->
-  <xacro:property name="drive_order_path" value="$(find dynaarm_description)/urdf/common/${arm_version_name}/drive_order.yaml"/>
-  <xacro:property name="ethercat_addresses" value="${xacro.load_yaml(drive_order_path)}"/>
+  <!--
+    Obtain the EtherCAT drive order (address order list).
+    The drive_order.yaml file is either loaded from the default location
+    in dynaarm.urdf.xacro or passed down from another launch file.
+  -->
+  <xacro:property name="ethercat_addresses" value="${xacro.load_yaml(drive_order_file)}"/>
   <xacro:property name="J_PI" value="3.14159265359" />
   <xacro:property name="baboon_peak_torque" value="40" />

File: urdf/dynaarm.urdf.xacro (robot description, xacro)
@@ -26,5 +26,13 @@
   <!-- -->
   <xacro:macro name="dynaarm"
-    params="tf_prefix parent_link collision:='simple' dof mode ethercat_bus start_in_freeze_mode:=false drive_parameter_folder:='' controller_path:='' covers version *origin">
+    params="tf_prefix parent_link collision:='simple' dof mode ethercat_bus drive_order:='' start_in_freeze_mode:=false drive_parameter_folder:='' controller_path:='' covers version *origin">
+    <!-- Allow the user to pass the drive order file -->
+    <xacro:property name="default_drive_order_file" value="$(find dynaarm_description)/urdf/common/${version}/drive_order.yaml" />
+    <xacro:if value="${drive_order == ''}">
+      <xacro:property name="drive_order_file" value="${default_drive_order_file}" />
+    </xacro:if>
+    <xacro:unless value="${drive_order == ''}">
+      <xacro:property name="drive_order_file" value="${drive_order}" />
+    </xacro:unless>
     <!--Allow the user to pass a custom folder for drive parameters-->
     <xacro:property name="default_drive_parameter_folder" value="$(find dynaarm_driver)/config/${version}" />
@@ -39,6 +47,5 @@
     <xacro:include filename="$(find dynaarm_description)/urdf/common/dynaarm_common.urdf.xacro" />
     <!-- Include the version specific information-->
-    <xacro:include
-      filename="$(find dynaarm_description)/urdf/common/${version}/dynaarm_parameters.urdf.xacro" />
+    <xacro:include filename="$(find dynaarm_description)/urdf/common/${version}/dynaarm_parameters.urdf.xacro" />
     <xacro:include filename="$(find dynaarm_description)/urdf/common/dynaarm.ros2control.xacro" />
     <xacro:dynaarm_joint_fixed joint_name="${joint_base_name}"
@@ -55,5 +62,10 @@
     </xacro:if>
     <!--ros2control-->
-    <xacro:dynaarm_ros2_control tf_prefix="${tf_prefix}" ethercat_bus="${ethercat_bus}" start_in_freeze_mode="${start_in_freeze_mode}"  drive_parameter_folder="${drive_parameter_folder_internal}" drive_parameter_folder_default="${default_drive_parameter_folder}" ethercat_addresses="${ethercat_addresses}"/>
+    <xacro:dynaarm_ros2_control tf_prefix="${tf_prefix}"
+                                ethercat_bus="${ethercat_bus}"
+                                start_in_freeze_mode="${start_in_freeze_mode}"
+                                drive_parameter_folder="${drive_parameter_folder_internal}"
+                                drive_parameter_folder_default="${default_drive_parameter_folder}"
+                                ethercat_addresses="${ethercat_addresses}"/>
   </xacro:macro>
   <!-- -->

Commit message: Simplified the usage of the drive_order file for the ethercat_addresses.

File: urdf/common/arowana4/dynaarm_parameters.urdf.xacro (robot description, xacro)
@@ -22,10 +22,4 @@
 <robot xmlns:xacro="http://www.ros.org/wiki/xacro">
   <xacro:property name="arm_version_name" value="arowana4"/>
-  <!--
-    Obtain the EtherCAT drive order (address order list).
-    The drive_order.yaml file is either loaded from the default location
-    in dynaarm.urdf.xacro or passed down from another launch file.
-  -->
-  <xacro:property name="ethercat_addresses" value="${xacro.load_yaml(drive_order_file)}"/>
   <xacro:property name="J_PI" value="3.14159265359" />
   <xacro:property name="baboon_peak_torque" value="40" />

File: urdf/common/baracuda12/dynaarm_parameters.urdf.xacro (robot description, xacro)
@@ -22,10 +22,4 @@
 <robot xmlns:xacro="http://www.ros.org/wiki/xacro">
   <xacro:property name="arm_version_name" value="baracuda12"/>
-  <!--
-    Obtain the EtherCAT drive order (address order list).
-    The drive_order.yaml file is either loaded from the default location
-    in dynaarm.urdf.xacro or passed down from another launch file.
-  -->
-  <xacro:property name="ethercat_addresses" value="${xacro.load_yaml(drive_order_file)}"/>
   <xacro:property name="J_PI" value="3.14159265359" />
   <xacro:property name="baboon_peak_torque" value="40" />

File: urdf/dynaarm.urdf.xacro (robot description, xacro)
@@ -29,10 +29,7 @@
     <!-- Allow the user to pass the drive order file -->
     <xacro:property name="default_drive_order_file" value="$(find dynaarm_description)/urdf/common/${version}/drive_order.yaml" />
-    <xacro:if value="${drive_order == ''}">
-      <xacro:property name="drive_order_file" value="${default_drive_order_file}" />
-    </xacro:if>
-    <xacro:unless value="${drive_order == ''}">
-      <xacro:property name="drive_order_file" value="${drive_order}" />
-    </xacro:unless>
+    <xacro:property name="drive_order_file" value="${default_drive_order_file if drive_order == '' else drive_order}" />
+    <!-- Obtain the EtherCAT drive order (address order list) -->
+    <xacro:property name="ethercat_addresses" value="${xacro.load_yaml(drive_order_file)}"/>
     <!--Allow the user to pass a custom folder for drive parameters-->
     <xacro:property name="default_drive_parameter_folder" value="$(find dynaarm_driver)/config/${version}" />
