Commit message: Enabling the usage of an ethercat switch (#50)
* Implemented a way to pass a drive order file to the dynaarm so the ethercat addresses can be loaded from there. Otherwise the default addresses will be loaded.

* Pleased pre-commit

* Added minimal more information as a comment.

* Simplified the usage of the drive_order file for the ethercat_addresses.

* Pleased pre-commit

File: urdf/common/arowana4/dynaarm_parameters.urdf.xacro (robot description, xacro)
@@ -22,7 +22,4 @@
 <robot xmlns:xacro="http://www.ros.org/wiki/xacro">
   <xacro:property name="arm_version_name" value="arowana4"/>
-  <!-- Obtain the ethercat drive order (address order list)-->
-  <xacro:property name="drive_order_path" value="$(find dynaarm_description)/urdf/common/${arm_version_name}/drive_order.yaml"/>
-  <xacro:property name="ethercat_addresses" value="${xacro.load_yaml(drive_order_path)}"/>
   <xacro:property name="J_PI" value="3.14159265359" />
   <xacro:property name="baboon_peak_torque" value="40" />

File: urdf/common/baracuda12/dynaarm_parameters.urdf.xacro (robot description, xacro)
@@ -22,7 +22,4 @@
 <robot xmlns:xacro="http://www.ros.org/wiki/xacro">
   <xacro:property name="arm_version_name" value="baracuda12"/>
-  <!-- Obtain the ethercat drive order (address order list)-->
-  <xacro:property name="drive_order_path" value="$(find dynaarm_description)/urdf/common/${arm_version_name}/drive_order.yaml"/>
-  <xacro:property name="ethercat_addresses" value="${xacro.load_yaml(drive_order_path)}"/>
   <xacro:property name="J_PI" value="3.14159265359" />
   <xacro:property name="baboon_peak_torque" value="40" />

File: urdf/dynaarm.urdf.xacro (robot description, xacro)
@@ -26,5 +26,10 @@
   <!-- -->
   <xacro:macro name="dynaarm"
-    params="tf_prefix parent_link collision:='simple' dof mode ethercat_bus start_in_freeze_mode:=false drive_parameter_folder:='' controller_path:='' covers version *origin">
+    params="tf_prefix parent_link collision:='simple' dof mode ethercat_bus drive_order:='' start_in_freeze_mode:=false drive_parameter_folder:='' controller_path:='' covers version *origin">
+    <!-- Allow the user to pass the drive order file -->
+    <xacro:property name="default_drive_order_file" value="$(find dynaarm_description)/urdf/common/${version}/drive_order.yaml" />
+    <xacro:property name="drive_order_file" value="${default_drive_order_file if drive_order == '' else drive_order}" />
+    <!-- Obtain the EtherCAT drive order (address order list) -->
+    <xacro:property name="ethercat_addresses" value="${xacro.load_yaml(drive_order_file)}"/>
     <!--Allow the user to pass a custom folder for drive parameters-->
     <xacro:property name="default_drive_parameter_folder" value="$(find dynaarm_driver)/config/${version}" />
@@ -38,7 +43,6 @@
     <xacro:property name="ee_parent" value="${base}" />
     <xacro:include filename="$(find dynaarm_description)/urdf/common/dynaarm_common.urdf.xacro" />
-    <!-- Include the version specific information-->
-    <xacro:include
-      filename="$(find dynaarm_description)/urdf/common/${version}/dynaarm_parameters.urdf.xacro" />
+    <!-- Include the version specific information and also load the ethercat addresses from the drive file -->
+    <xacro:include filename="$(find dynaarm_description)/urdf/common/${version}/dynaarm_parameters.urdf.xacro" />
     <xacro:include filename="$(find dynaarm_description)/urdf/common/dynaarm.ros2control.xacro" />
     <xacro:dynaarm_joint_fixed joint_name="${joint_base_name}"
@@ -55,5 +59,10 @@
     </xacro:if>
     <!--ros2control-->
-    <xacro:dynaarm_ros2_control tf_prefix="${tf_prefix}" ethercat_bus="${ethercat_bus}" start_in_freeze_mode="${start_in_freeze_mode}"  drive_parameter_folder="${drive_parameter_folder_internal}" drive_parameter_folder_default="${default_drive_parameter_folder}" ethercat_addresses="${ethercat_addresses}"/>
+    <xacro:dynaarm_ros2_control tf_prefix="${tf_prefix}"
+                                ethercat_bus="${ethercat_bus}"
+                                start_in_freeze_mode="${start_in_freeze_mode}"
+                                drive_parameter_folder="${drive_parameter_folder_internal}"
+                                drive_parameter_folder_default="${default_drive_parameter_folder}"
+                                ethercat_addresses="${ethercat_addresses}"/>
   </xacro:macro>
   <!-- -->
