Commit message: increased the weight of the forearm after adding the longer tube.

File: urdf/common/baracuda12/dynaarm_parameters.urdf.xacro (robot description, xacro)
@@ -188,5 +188,6 @@
   <xacro:property name="link05_inertial">
     <inertial>
-      <mass value="0.75007482" />
+      <!-- <mass value="0.75007482" />  original value but doesn't work well - Needs investigation also regarding the other values, is this the forearm link?-->
+      <mass value="0.95007482" />
       <origin xyz="0.07972553 -0.00005038 0.02334747" rpy="0 0 0" />
       <inertia ixx="0.00065953" iyy="0.00088282"

Commit message: initial commit

File: urdf/common/baracuda12/dynaarm_parameters.urdf.xacro (robot description, xacro)
@@ -189,5 +189,5 @@
     <inertial>
       <!-- <mass value="0.75007482" />  original value but doesn't work well - Needs investigation also regarding the other values, is this the forearm link?-->
-      <mass value="0.95007482" />
+      <mass value="1.02007482" />
       <origin xyz="0.07972553 -0.00005038 0.02334747" rpy="0 0 0" />
       <inertia ixx="0.00065953" iyy="0.00088282"
@@ -207,7 +207,8 @@
   <xacro:property name="link06_inertial">
     <inertial>
-      <mass value="0.0478406" />
+    <!-- <mass value="0.0478406" />  original value but doesn't work well - Needs investigation also regarding the other values, is this the forearm link? <inertia ixx="0.00001366" iyy="0.00001419"-->
+      <mass value="0.0078406" />
       <origin xyz="0.00045711 0.00000557 0.00344945" rpy="0 0 0" />
-      <inertia ixx="0.00001366" iyy="0.00001419"
+      <inertia ixx="0.00000366" iyy="0.00000419"
         izz="0.00002702" ixy="0"
         ixz="0.00000008" iyz="0" />

Commit message: Modify the forearm orientation home to fit the new cable management.

File: urdf/common/baracuda12/dynaarm_parameters.urdf.xacro (robot description, xacro)
@@ -92,5 +92,5 @@
   <xacro:property name="joint_3_origin_xyz" value="0.4127 0 0" />
   <xacro:property name="joint_3_origin_rpy" value="0 0 0" />
-  <xacro:property name="joint_3_lower_limit" value="-0.05" />
+  <xacro:property name="joint_3_lower_limit" value="0.00" />
   <xacro:property name="joint_3_upper_limit" value="${J_PI}" />
   <xacro:property name="joint_3_cam_name" value="${tf_prefix}elbow_camera" />
@@ -103,5 +103,5 @@
   <xacro:property name="joint_4_axis_xyz" value="0 0 1" />
   <xacro:property name="joint_4_origin_xyz" value="0.0262 -0.0855 0" />
-  <xacro:property name="joint_4_origin_rpy" value="${J_PI/2} 0 ${J_PI/2}" />
+  <xacro:property name="joint_4_origin_rpy" value="${J_PI/2} ${J_PI/2} ${J_PI/2}" />
   <xacro:property name="joint_4_lower_limit" value="${-J_PI - J_PI/2}" />
   <xacro:property name="joint_4_upper_limit" value="${J_PI + J_PI/2}" />

Commit message: added correct limits

File: urdf/common/baracuda12/dynaarm_parameters.urdf.xacro (robot description, xacro)
@@ -78,6 +78,6 @@
   <xacro:property name="joint_1_origin_xyz" value="0 0 0.0105" />
   <xacro:property name="joint_1_origin_rpy" value="0 0 0" />
-  <xacro:property name="joint_1_lower_limit" value="${-J_PI - J_PI/2}" />
-  <xacro:property name="joint_1_upper_limit" value="${J_PI + J_PI/2}" />
+  <xacro:property name="joint_1_lower_limit" value="${-J_PI - J_PI/2 + 0.4}" />
+  <xacro:property name="joint_1_upper_limit" value="${J_PI + J_PI/2 - 0.4}" />
   <xacro:property name="joint_2_name" value="${tf_prefix}shoulder_flexion" />
   <xacro:property name="joint_2_joint_type" value="revolute" />
@@ -85,6 +85,6 @@
   <xacro:property name="joint_2_origin_xyz" value="0 0 0.047" />
   <xacro:property name="joint_2_origin_rpy" value="${J_PI/2} ${-J_PI/2} 0" />
-  <xacro:property name="joint_2_lower_limit" value="${-J_PI/2 - 0.3}" />
-  <xacro:property name="joint_2_upper_limit" value="${J_PI/2 + 0.3}" />
+  <xacro:property name="joint_2_lower_limit" value="${-J_PI/2 - 0.15}" />
+  <xacro:property name="joint_2_upper_limit" value="${J_PI/2 + 0.15}" />
   <xacro:property name="joint_3_name" value="${tf_prefix}elbow_flexion" />
   <xacro:property name="joint_3_joint_type" value="revolute" />
@@ -93,5 +93,5 @@
   <xacro:property name="joint_3_origin_rpy" value="0 0 0" />
   <xacro:property name="joint_3_lower_limit" value="0.00" />
-  <xacro:property name="joint_3_upper_limit" value="${J_PI}" />
+  <xacro:property name="joint_3_upper_limit" value="${J_PI - 0.05}" />
   <xacro:property name="joint_3_cam_name" value="${tf_prefix}elbow_camera" />
   <xacro:property name="joint_3_cam_joint_type" value="fixed" />
@@ -111,6 +111,6 @@
   <xacro:property name="joint_5_origin_xyz" value="0.0295 0 0.4207" />
   <xacro:property name="joint_5_origin_rpy" value="0 ${-J_PI/2} 0" />
-  <xacro:property name="joint_5_lower_limit" value="${-J_PI/2}" />
-  <xacro:property name="joint_5_upper_limit" value="${J_PI/2}" />
+  <xacro:property name="joint_5_lower_limit" value="${-J_PI/2 -0.25}" />
+  <xacro:property name="joint_5_upper_limit" value="${J_PI/2 + 0.25}" />
   <xacro:property name="joint_5_cam_name" value="${tf_prefix}wrist_flexion_camera" />
   <xacro:property name="joint_5_cam_joint_type" value="fixed" />

Commit message: Added the weight on the EE

File: urdf/common/baracuda12/dynaarm_parameters.urdf.xacro (robot description, xacro)
@@ -192,5 +192,5 @@
   <xacro:property name="link05_inertial">
     <inertial>
-      <!-- <mass value="0.75007482" />  original value but doesn't work well - Needs investigation also regarding the other values, is this the forearm link?-->
+      <!-- <mass value="0.75007482" />  original value but doesn't work well - Needs to include the cables inside the forearm tube?-->
       <mass value="0.95007482" />
       <origin xyz="0.07972553 -0.00005038 0.02334747" rpy="0 0 0" />
@@ -211,5 +211,6 @@
   <xacro:property name="link06_inertial">
     <inertial>
-      <mass value="0.0478406" />
+      <!-- <mass value="0.0478406" />  mass without the plastic EE handle -->
+      <mass value="0.1578406" />
       <origin xyz="0.00045711 0.00000557 0.00344945" rpy="0 0 0" />
       <inertia ixx="0.00001366" iyy="0.00001419"

Commit message: Adapterd the masses of the links for represent the real mass.

File: urdf/common/baracuda12/dynaarm_parameters.urdf.xacro (robot description, xacro)
@@ -144,4 +144,5 @@
     </inertial>
   </xacro:property>
+  <!-- Shoulder -->
   <xacro:property name="link01_inertial">
     <inertial>
@@ -153,7 +154,9 @@
     </inertial>
   </xacro:property>
+  <!-- Upper Arm -->
   <xacro:property name="link02_inertial">
     <inertial>
-      <mass value="1.72040464" />
+      <!-- Original - <mass value="1.72040464" /> -->
+      <mass value="2.12040464" />
       <origin xyz="0.20391301 -0.00000528 -0.00015224"
         rpy="0 0 0" />
@@ -163,4 +166,5 @@
     </inertial>
   </xacro:property>
+  <!-- Elbow -->
   <xacro:property name="link03_inertial">
     <inertial>
@@ -172,4 +176,5 @@
     </inertial>
   </xacro:property>
+  <!-- Camera Mounting Point 1 -->
   <xacro:property name="link03_cam_inertial">
     <inertial>
@@ -181,4 +186,5 @@
     </inertial>
   </xacro:property>
+  <!-- Forearm -->
   <xacro:property name="link04_inertial">
     <inertial>
@@ -190,8 +196,9 @@
     </inertial>
   </xacro:property>
+  <!-- wrist_1 -->
   <xacro:property name="link05_inertial">
     <inertial>
       <!-- <mass value="0.75007482" />  original value but doesn't work well - Needs to include the cables inside the forearm tube?-->
-      <mass value="0.95007482" />
+      <mass value="1.15007482" />
       <origin xyz="0.07972553 -0.00005038 0.02334747" rpy="0 0 0" />
       <inertia ixx="0.00065953" iyy="0.00088282"
@@ -200,4 +207,5 @@
     </inertial>
   </xacro:property>
+  <!-- Camera Mounting Point 2 -->
   <xacro:property name="link05_cam_inertial">
     <inertial>
@@ -209,8 +217,8 @@
     </inertial>
   </xacro:property>
+  <!-- Wrist 2 -->
   <xacro:property name="link06_inertial">
     <inertial>
-      <!-- <mass value="0.0478406" />  mass without the plastic EE handle -->
-      <mass value="0.1578406" />
+      <mass value="0.0478406" />
       <origin xyz="0.00045711 0.00000557 0.00344945" rpy="0 0 0" />
       <inertia ixx="0.00001366" iyy="0.00001419"

Commit message: Initial torso URDF in a working state.

File: urdf/common/baracuda12/dynaarm_parameters.urdf.xacro (robot description, xacro)
@@ -30,4 +30,6 @@
   <xacro:property name="mm2_to_m2" value="0.000001" />
   <xacro:property name="mm_to_m" value="0.001" />
+  <xacro:property name="distance_from_world_general_flange" value="0.001" />
+  <xacro:property name="distance_from_world_torso_flange" value="0.00096" />
   <!-- Links -->
   <xacro:property name="base" value="${tf_prefix}base" />

File: urdf/common/torso/torso_parameters.urdf.xacro (robot description, xacro)
@@ -40,13 +40,9 @@
   <xacro:property name="joint_tbase_origin_rpy" value="0 0 0" />
   <xacro:property name="joint_left_arm_name" value="${tf_prefix}left_arm_flange_fix_joint" />
-  <xacro:property name="joint_left_arm_origin_xyz" value="0.0 0.084464 0.55554" />
-  <xacro:property name="joint_left_arm_origin_rpy" value="0.0 2.3562 ${-J_PI}" />
-  <xacro:property name="joint_left_arm_xyz" value="0.0 0.084464 0.55554" />
-  <xacro:property name="joint_left_arm_rpy" value="0 0 0" />
+  <xacro:property name="joint_left_arm_origin_xyz" value="0.0 0.088 0.552" />
+  <xacro:property name="joint_left_arm_origin_rpy" value="2.3562 0.0 ${-J_PI}" />
   <xacro:property name="joint_right_arm_name" value="${tf_prefix}right_arm_flange_fix_joint" />
-  <xacro:property name="joint_right_arm_origin_xyz" value="0.0 -0.084464 0.55554" />
-  <xacro:property name="joint_right_arm_origin_rpy" value="0.0 2.3562 0.0" />
-  <xacro:property name="joint_right_arm_xyz" value="0.0 -0.084464 0.55554" />
-  <xacro:property name="joint_right_arm_rpy" value="0 0 0" />
+  <xacro:property name="joint_right_arm_origin_xyz" value="0.0 -0.088 0.552" />
+  <xacro:property name="joint_right_arm_origin_rpy" value="2.3562 0.0 0.0" />
   <!-- Base Robot -->
   <xacro:property name="tbase_inertial">

File: urdf/torso_standalone.urdf.xacro (robot description, xacro)
@@ -17,5 +17,6 @@
   </xacro:torso>
   <!-- Add two arms to torso -->
-  <xacro:dynaarm tf_prefix="$(arg tf_prefix)_arm1"
+  <xacro:dynaarm
+    tf_prefix="$(arg tf_prefix)_arm1"
     parent_link="left_arm_flange"
     dof="$(arg dof)"
@@ -24,5 +25,5 @@
     covers="$(arg covers)"
     version="$(arg dynaarm_version)">
-    <origin xyz="0.3 0.2 0.2" rpy="0 0 0" />
+    <origin xyz="0 0 0.095" rpy="0 0 0" />
   </xacro:dynaarm>
   <xacro:dynaarm tf_prefix="$(arg tf_prefix)_arm2"
@@ -33,5 +34,5 @@
     covers="$(arg covers)"
     version="$(arg dynaarm_version)">
-    <origin xyz="0.3 -0.2 0.2" rpy="0 0 0" />
+    <origin xyz="0 0 0.095" rpy="0 0 0" />
   </xacro:dynaarm>
 </robot>

Commit message: added simple collision model

File: urdf/common/baracuda12/dynaarm_parameters.urdf.xacro (robot description, xacro)
@@ -276,75 +276,136 @@
     </inertial>
   </xacro:property>
-  <!-- Collision properties -->
-  <xacro:property name="base_collision">
-    <collision>
-      <origin xyz="0 0 0" rpy="0 0 0" />
-      <geometry>
-        <mesh
-          filename="file://$(find dynaarm_description)/meshes/baracuda12/collision_meshes/base_collision_mesh.stl"
-          scale="1 1 1" />
-      </geometry>
-    </collision>
-  </xacro:property>
-  <xacro:property name="link01_collision">
-    <collision>
-      <origin xyz="0 0 0" rpy="0 0 0" />
-      <geometry>
-        <mesh
-          filename="file://$(find dynaarm_description)/meshes/baracuda12/collision_meshes/shoulder_collision_mesh.stl"
-          scale="1 1 1" />
-      </geometry>
-    </collision>
-  </xacro:property>
-  <xacro:property name="link02_collision">
-    <collision>
-      <origin xyz="0 0 0" rpy="0 0 0" />
-      <geometry>
-        <mesh
-          filename="file://$(find dynaarm_description)/meshes/baracuda12/collision_meshes/upperarm_collision_mesh.stl"
-          scale="1 1 1" />
-      </geometry>
-    </collision>
-  </xacro:property>
-  <xacro:property name="link03_collision">
-    <collision>
-      <origin xyz="0 0 0" rpy="0 0 0" />
-      <geometry>
-        <mesh
-          filename="file://$(find dynaarm_description)/meshes/baracuda12/collision_meshes/elbow_collision_mesh.stl"
-          scale="1 1 1" />
-      </geometry>
-    </collision>
-  </xacro:property>
-  <xacro:property name="link04_collision">
-    <collision>
-      <origin xyz="0 0 0" rpy="0 0 0" />
-      <geometry>
-        <mesh
-          filename="file://$(find dynaarm_description)/meshes/baracuda12/collision_meshes/forearm_collision_mesh.stl"
-          scale="1 1 1" />
-      </geometry>
-    </collision>
-  </xacro:property>
-  <xacro:property name="link05_collision">
-    <collision>
-      <origin xyz="0 0 0" rpy="0 0 0" />
-      <geometry>
-        <mesh
-          filename="file://$(find dynaarm_description)/meshes/baracuda12/collision_meshes/wrist1_collision_mesh.stl"
-          scale="1 1 1" />
-      </geometry>
-    </collision>
-  </xacro:property>
-  <xacro:property name="link06_collision">
-    <collision>
-      <origin xyz="0 0 0" rpy="0 0 0" />
-      <geometry>
-        <mesh
-          filename="file://$(find dynaarm_description)/meshes/baracuda12/collision_meshes/wrist2_collision_mesh.stl"
-          scale="1 1 1" />
-      </geometry>
-    </collision>
-  </xacro:property>
+ <xacro:if value="${collision == 'simple'}">
+    <!-- Collision properties -->
+    <xacro:property name="base_collision">
+        <collision>
+            <geometry>
+                <cylinder length='0.1' radius='0.05'/>
+            </geometry>
+            <origin xyz='0 0 0' rpy='0 0 0'/>
+        </collision>
+    </xacro:property>
+    <xacro:property name="link01_collision">
+          <collision>
+              <geometry>
+                  <cylinder length='0.25' radius='0.06'/>
+              </geometry>
+              <origin xyz='0 0 0.05' rpy='${J_PI/2} 0 0'/>
+          </collision>
+    </xacro:property>
+    <xacro:property name="link02_collision">
+          <collision>
+              <geometry>
+                  <cylinder length='0.4' radius='0.05'/>
+              </geometry>
+              <origin xyz='0.15 0 0' rpy='0 ${J_PI/2} 0'/>
+          </collision>
+    </xacro:property>
+    <xacro:property name="link03_collision">
+      <collision>
+          <geometry>
+              <cylinder length='0.2' radius='0.065'/>
+          </geometry>
+          <origin xyz='-0.01 -0.05 0' rpy='${J_PI/2} 0 0'/>
+      </collision>
+    </xacro:property>
+    <xacro:property name="link04_collision">
+      <collision>
+          <geometry>
+              <cylinder length='0.4' radius='0.04'/>
+          </geometry>
+          <origin xyz='0 0 0.2' rpy='0 0 0'/>
+      </collision>
+    </xacro:property>
+    <xacro:property name="link05_collision">
+      <collision>
+          <geometry>
+              <cylinder length='0.125' radius='0.05'/>
+          </geometry>
+          <origin xyz='0 0 0.025' rpy='0 0 ${J_PI/2}'/>
+      </collision>
+    </xacro:property>
+    <xacro:property name="link06_collision">
+      <collision>
+          <geometry>
+              <cylinder length='0.15' radius='0.052'/>
+          </geometry>
+          <origin xyz='0.005 0 -0.05' rpy='0 0 0'/>
+      </collision>
+    </xacro:property>
+  </xacro:if>
+  <xacro:if value="${collision == 'complex'}">
+    <!-- Collision properties -->
+    <xacro:property name="base_collision">
+      <collision>
+        <origin xyz="0 0 0" rpy="0 0 0" />
+        <geometry>
+          <mesh
+            filename="file://$(find dynaarm_description)/meshes/baracuda12/collision_meshes/base_collision_mesh.stl"
+            scale="1 1 1" />
+        </geometry>
+      </collision>
+    </xacro:property>
+    <xacro:property name="link01_collision">
+      <collision>
+        <origin xyz="0 0 0" rpy="0 0 0" />
+        <geometry>
+          <mesh
+            filename="file://$(find dynaarm_description)/meshes/baracuda12/collision_meshes/shoulder_collision_mesh.stl"
+            scale="1 1 1" />
+        </geometry>
+      </collision>
+    </xacro:property>
+    <xacro:property name="link02_collision">
+      <collision>
+        <origin xyz="0 0 0" rpy="0 0 0" />
+        <geometry>
+          <mesh
+            filename="file://$(find dynaarm_description)/meshes/baracuda12/collision_meshes/upperarm_collision_mesh.stl"
+            scale="1 1 1" />
+        </geometry>
+      </collision>
+    </xacro:property>
+    <xacro:property name="link03_collision">
+      <collision>
+        <origin xyz="0 0 0" rpy="0 0 0" />
+        <geometry>
+          <mesh
+            filename="file://$(find dynaarm_description)/meshes/baracuda12/collision_meshes/elbow_collision_mesh.stl"
+            scale="1 1 1" />
+        </geometry>
+      </collision>
+    </xacro:property>
+    <xacro:property name="link04_collision">
+      <collision>
+        <origin xyz="0 0 0" rpy="0 0 0" />
+        <geometry>
+          <mesh
+            filename="file://$(find dynaarm_description)/meshes/baracuda12/collision_meshes/forearm_collision_mesh.stl"
+            scale="1 1 1" />
+        </geometry>
+      </collision>
+    </xacro:property>
+    <xacro:property name="link05_collision">
+      <collision>
+        <origin xyz="0 0 0" rpy="0 0 0" />
+        <geometry>
+          <mesh
+            filename="file://$(find dynaarm_description)/meshes/baracuda12/collision_meshes/wrist1_collision_mesh.stl"
+            scale="1 1 1" />
+        </geometry>
+      </collision>
+    </xacro:property>
+    <xacro:property name="link06_collision">
+      <collision>
+        <origin xyz="0 0 0" rpy="0 0 0" />
+        <geometry>
+          <mesh
+            filename="file://$(find dynaarm_description)/meshes/baracuda12/collision_meshes/wrist2_collision_mesh.stl"
+            scale="1 1 1" />
+        </geometry>
+      </collision>
+    </xacro:property>
+  </xacro:if>
   <!-- set the ee_parent relative to the DoF -->
   <xacro:property name="ee_parent" value="${base}" />

File: urdf/dynaarm.urdf.xacro (robot description, xacro)
@@ -26,5 +26,5 @@
   <!-- -->
   <xacro:macro name="dynaarm"
-    params="tf_prefix parent_link dof mode ethercat_bus start_in_freeze_mode:=false drive_parameter_folder:='' controller_path:='' covers version *origin">
+    params="tf_prefix parent_link collision dof mode ethercat_bus start_in_freeze_mode:=false drive_parameter_folder:='' controller_path:='' covers version *origin">
     <!--Allow the user to pass a custom folder for drive parameters-->
     <xacro:property name="default_drive_parameter_folder" value="$(find dynaarm_driver)/config/${version}" />

Commit message: Modified the dynaarm simple collision model a bit for the last joint / link.

File: urdf/common/baracuda12/dynaarm_parameters.urdf.xacro (robot description, xacro)
@@ -329,7 +329,7 @@
       <collision>
           <geometry>
-              <cylinder length='0.15' radius='0.052'/>
+              <cylinder length='0.09' radius='0.052'/>
           </geometry>
-          <origin xyz='0.005 0 -0.05' rpy='0 0 0'/>
+          <origin xyz='0.005 0 -0.035' rpy='0 0 0'/>
       </collision>
     </xacro:property>

Commit message: Fixed the base location so that it is intuitively on the base flange when the location set to (0, 0, 0)

File: urdf/common/baracuda12/dynaarm_parameters.urdf.xacro (robot description, xacro)
@@ -76,5 +76,5 @@
   <xacro:property name="joint_1_joint_type" value="revolute" />
   <xacro:property name="joint_1_axis_xyz" value="0 0 1" />
-  <xacro:property name="joint_1_origin_xyz" value="0 0 0.0105" />
+  <xacro:property name="joint_1_origin_xyz" value="0 0 0.1105" />
   <xacro:property name="joint_1_origin_rpy" value="0 0 0" />
   <xacro:property name="joint_1_lower_limit" value="${-J_PI - J_PI/2 + 0.4}" />

File: urdf/dynaarm_standalone.urdf.xacro (robot description, xacro)
@@ -33,5 +33,5 @@
                 covers="$(arg covers)"
                 version="$(arg version)">
-    <origin xyz="0 0 0.085" rpy="0.0 0.0 0.0" />
+    <origin xyz="0 0 0" rpy="0.0 0.0 0.0" />
   </xacro:dynaarm>
 </robot>

Commit message: fix(urdf): updated base mass and inertia

File: urdf/common/baracuda12/dynaarm_parameters.urdf.xacro (robot description, xacro)
@@ -132,11 +132,11 @@
   <xacro:property name="base_inertial">
     <inertial>
-      <mass value="2.00205474" />
+      <mass value="1.94219788" />
       <origin
-        xyz="0.00347077 0.00328869 -0.0488212"
+        xyz="0.00243205 0.00250861 0.05299306"
         rpy="0 0 0" />
-      <inertia ixx="0.00403342" iyy="0.00417534"
-        izz="0.00460211" ixy="0.00040828"
-        ixz="-0.00018775" iyz="-0.0001821" />
+      <inertia ixx="0.00434815" iyy="0.00446542"
+        izz="0.00446174" ixy="0.00028867"
+        ixz="-0.00015925" iyz="-0.00015771" />
     </inertial>
   </xacro:property>
@@ -280,5 +280,5 @@
                 <cylinder length='0.1' radius='0.05'/>
             </geometry>
-            <origin xyz='0 0 0' rpy='0 0 0'/>
+            <origin xyz='0 0 0.05' rpy='0 0 0'/>
         </collision>
     </xacro:property>

Commit message: fix(urdf): updated shoulder and forearm mass, origin, and inertia

File: urdf/common/baracuda12/dynaarm_parameters.urdf.xacro (robot description, xacro)
@@ -144,9 +144,9 @@
   <xacro:property name="link01_inertial">
     <inertial>
-      <mass value="2.73096676" />
-      <origin xyz="0.00001348 0.00013521 0.0430259" rpy="0 0 0" />
-      <inertia ixx="0.01291668" iyy="0.00874231"
-        izz="0.01243436" ixy="0.0000044"
-        ixz="-0.00000179" iyz="-0.00000203" />
+      <mass value="2.825469" />
+      <origin xyz="0.000012 0.000480 0.039513" rpy="0 0 0" />
+      <inertia ixx="0.013069" iyy="0.004793"
+        izz="0.000046" ixy="0.000033"
+        ixz="-0.000002" iyz="-0.000046" />
     </inertial>
   </xacro:property>
@@ -186,9 +186,9 @@
   <xacro:property name="link04_inertial">
     <inertial>
-      <mass value="1.15674546" />
-      <origin xyz="-0.00115165 0.00001056 0.30067314" rpy="0 0 0" />
-      <inertia ixx="0.03129519" iyy="0.03125954"
-        izz="0.00090392" ixy="0.00000151"
-        ixz="-0.00017171" iyz="0.00000159" />
+      <mass value="1.237246" />
+      <origin xyz="-0.001568 0.000046 0.292163" rpy="0 0 0" />
+      <inertia ixx="0.033872" iyy="0.033868"
+        izz="0.001041" ixy="0.000002"
+        ixz="-0.000276" iyz="0.000018" />
     </inertial>
   </xacro:property>

Commit message: fix(urdf): added 100g to forearm mass

File: urdf/common/baracuda12/dynaarm_parameters.urdf.xacro (robot description, xacro)
@@ -186,5 +186,6 @@
   <xacro:property name="link04_inertial">
     <inertial>
-      <mass value="1.237246" />
+      <!-- The mass here is 100g more than the value in CAD, but through testing we found out that freedrive works better with the increased value (09.12.25 Antonis & Marc)-->
+      <mass value="1.337246" />
       <origin xyz="-0.001568 0.000046 0.292163" rpy="0 0 0" />
       <inertia ixx="0.033872" iyy="0.033868"
